File: KiCAD files/myDAQExpansionBoard/myDAQExpansionBoard.kicad_sch (KiCad schematic)
At the start: 0 parts

Commit message: schematic first revision
Parts:
- added C?: 1n, symbol Device:C
- added C? (x2): 100n, symbol Device:C
- added D? (x4): LED, symbol Device:LED
- added J1: OSTV7XX3151, symbol Connector_Generic:Conn_01x20
- added J? (x2): Screw_Terminal_01x02, symbol Connector:Screw_Terminal_01x02
- added JP? (x3): Jumper_3_Open, symbol Jumper:Jumper_3_Open
- added JP? (x8): Jumper_2_Open, symbol Jumper:Jumper_2_Open
- added R? (x4): 1k, symbol Device:R
- added R? (x6): 10k, symbol Device:R
- added R? (x7): 680, symbol Device:R
- added R?: R_Photo, symbol Device:R_Photo
- added R?: 1R, symbol Device:R
- added SW? (x2): SW_SPST, symbol Switch:SW_SPST
- added SW? (x2): SW_Push, symbol Switch:SW_Push
- added U?: ACS712xLCTR-05B, Package_SO:SOIC-8_3.9x4.9mm_P1.27mm, symbol Sensor_Current:ACS712xLCTR-05B
- added U?: 7447, symbol 74xx_IEEE:7447
- added U?: LM35-D, Package_SO:SOIC-8_3.9x4.9mm_P1.27mm, symbol Sensor_Temperature:LM35-D
- added U?: HDSP-7501, Display_7Segment:HDSP-A151, symbol Display_Character:HDSP-7501
Connections:
- new net: D?.1 (K), R?.1 (x4)
- new net: D?.2 (A), JP?.2 (B) (x4)
- new net: JP?.1 (A), R?.1 (x4)
- new net: JP?.1 (A), U?.7 (VIOUT)
- new net: JP?.3 (B), R?.1, R?.2
- new net: R?.2, U?.1 (IP+), U?.2 (IP+)
- new net: J?.1 (Pin_1), J?.2 (Pin_2), U?.3 (IP-), U?.4 (IP-)
- new net: C?.1, U?.6 (FILTER)
- new net: R?.1, U?.13 (a)
- new net: R?.2, U?.10 (A)
- new net: R?.1, U?.12 (b)
- new net: R?.2, U?.9 (B)
- new net: R?.1, U?.10 (d)
- new net: R?.1, U?.11 (c)
- new net: R?.1, U?.14 (g)
- new net: R?.1, U?.15 (f)
- new net: R?.2, U?.3 (~{LT}), U?.4 (~{BI}), U?.5 (~{RBI})
- new net: R?.1, U?.9 (e)
- new net: JP?.1 (A), U?.1 (Vout)
- new net: R?.2, U?.8 (C)
- new net: R?.2, U?.3 (G)
- new net: J?.1 (Pin_1), J?.2 (Pin_2), R?.1
- new net: JP?.2 (C), U?.1 (CA), U?.6 (CA)
- new net: R?.2, U?.5 (D)
- new net: R?.2, U?.2 (F)
- new net: R?.2, U?.4 (E)
- new net +15V: J1.1 (Pin_1)
- new net +5V: C?.1, C?.1, J1.20 (Pin_20), JP?.1 (A), JP?.2 (B), JP?.2 (B), JP?.2 (B), JP?.2 (B), R?.1, R?.1, U?.16 (VCC), U?.8 (+VS), U?.8 (VCC)
- new net -15V: J1.2 (Pin_2)
- new net AI0+: J1.7 (Pin_7), JP?.2 (C)
- new net AI1+: J1.9 (Pin_9), JP?.2 (C)
- new net AO0: J1.4 (Pin_4), JP?.3 (B)
- new net AO1: J1.5 (Pin_5)
- new net DIO0: J1.11 (Pin_11), JP?.1 (A), U?.7 (A)
- new net DIO1: J1.12 (Pin_12), JP?.1 (A), U?.1 (B)
- new net DIO2: J1.13 (Pin_13), JP?.1 (A), U?.2 (C)
- new net DIO3: J1.14 (Pin_14), JP?.1 (A)
- new net DIO4: J1.15 (Pin_15), R?.2, SW?.1
- new net DIO5: J1.16 (Pin_16), R?.2, SW?.1
- new net DIO6: J1.17 (Pin_17), R?.2, SW?.1 (A)
- new net DIO7: J1.18 (Pin_18), R?.2, SW?.1 (A)
- new net GND: C?.2, C?.2, C?.2, J1.10 (Pin_10), J1.19 (Pin_19), J1.3 (Pin_3), J1.6 (Pin_6), J1.8 (Pin_8), JP?.3 (B), R?.2, R?.2, R?.2, R?.2, R?.2, SW?.2, SW?.2, SW?.2 (B), SW?.2 (B), U?.4 (GND), U?.5 (GND), U?.8 (GND)
- no-connect marks 0 -> 2
Other:
- note added: "7SEGM"
- note added: "ACS712"
- note added: "LDR"
- note added: "LEDice"
- note added: "LM35"
- note added: "SKLOPKE"
- note added: "TIPKALA"
- note added: "TO-DO: DONE: - 2 tipkala i pritezni otpornici (2 jumpera za pull up) - DIO 4,5 - 2 sklopke i pritezni otpornici (2 jumpera za pull up) - DIO 6,7 - 4 LEDice - DIO 0,1,2,3 - IC 7447 za 7.segm zaslon - DIO 0,1,2 - LDR - AIO - LM35 - AI1 - shunt i priključnice - acs712, AI0"
- company: (none) -> TVZ
- title: (none) -> myDAQExpansionBoard

Commit message: Update myDAQExpansionBoard.kicad_sch
Connections:
- net DIO3: now also U?.6 (D)
- no-connect marks 2 -> 1
Changed lines of the file:
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@@
   )
   (no_connect (at 181.61 86.995))
-  (no_connect (at 127 75.565))
   (wire (pts (xy 108.585 49.53) (xy 111.125 49.53))
     (stroke (width 0) (type default) (color 0 0 0 0))
@@
     )
   )
+  (global_label "DIO3" (shape input) (at 127 75.565 180) (fields_autoplaced)
+    (effects (font (size 1.27 1.27)) (justify right))
+    (property "Intersheet References" "${INTERSHEET_REFS}" (id 0) (at 120.1721 75.4856 0)
+      (effects (font (size 1.27 1.27)) (justify right) hide)
+    )
+  )

Commit message: Update myDAQExpansionBoard.kicad_sch
Other:
- note added: "TO-DO: - zamijeniti 7447 s nekim drugim IC-om? (nema ga za kupiti) DONE: - 2 tipkala i pritezni otpornici (2 jumpera za pull up) - DIO 4,5 - 2 sklopke i pritezni otpornici (2 jumpera za pull up) - DIO 6,7 - 4 LEDice - DIO 0,1,2,3 - IC 7447 za 7.segm zaslon - DIO 0,1,2 - LDR - AIO - LM35 - AI1 - shunt i priključnice - acs712, AI0"
- note removed: "TO-DO: DONE: - 2 tipkala i pritezni otpornici (2 jumpera za pull up) - DIO 4,5 - 2 sklopke i pritezni otpornici (2 jumpera za pull up) - DIO 6,7 - 4 LEDice - DIO 0,1,2,3 - IC 7447 za 7.segm zaslon - DIO 0,1,2 - LDR - AIO - LM35 - AI1 - shunt i priključnice - acs712, AI0"
Changed lines of the file:
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@@
     (stroke (width 0) (type default) (color 0 0 0 0))
   )
-  (text "TO-DO:\n\nDONE:\n- 2 tipkala i pritezni otpornici (2 jumpera za pull up) - DIO 4,5\n- 2 sklopke i pritezni otpornici (2 jumpera za pull up) - DIO 6,7\n- 4 LEDice - DIO 0,1,2,3\n- IC 7447 za 7.segm zaslon - DIO 0,1,2\n- LDR - AIO\n- LM35 - AI1\n- shunt i priključnice\n- acs712, AI0"
+  (text "TO-DO:\n- zamijeniti 7447 s nekim drugim IC-om? (nema ga za kupiti)\n\nDONE:\n- 2 tipkala i pritezni otpornici (2 jumpera za pull up) - DIO 4,5\n- 2 sklopke i pritezni otpornici (2 jumpera za pull up) - DIO 6,7\n- 4 LEDice - DIO 0,1,2,3\n- IC 7447 za 7.segm zaslon - DIO 0,1,2\n- LDR - AIO\n- LM35 - AI1\n- shunt i priključnice\n- acs712, AI0"
     (at 19.05 172.085 0)
     (effects (font (size 1.27 1.27)) (justify left bottom))

Commit message: update
Parts:
- added C?: 100n, symbol Device:C
- added JP? (x2): Jumper_3_Open, symbol Jumper:Jumper_3_Open
- added U?: L293D, Package_DIP:DIP-16_W7.62mm, symbol Driver_Motor:L293D
Connections:
- net +5V: now also C?.1, JP?.3 (B), JP?.3 (B)
- net DIO0: now also U?.2 (1A)
- net DIO1: now also U?.7 (2A)
- net DIO2: now also U?.10 (3A)
- net DIO3: now also U?.15 (4A)
- net GND: now also C?.2, JP?.1 (A), JP?.1 (A)
- new net: JP?.2 (C), U?.1 (EN1,2)
- new net: JP?.2 (C), U?.9 (EN3,4)
Other:
- note added: "TO-DO: - zamijeniti 7447 s nekim drugim IC-om? (nema ga za kupiti) - L293D 2 digitalna izlaza, DIP s profi podnožjem DONE: - 2 tipkala i pritezni otpornici (2 jumpera za pull up) - DIO 4,5 - 2 sklopke i pritezni otpornici (2 jumpera za pull up) - DIO 6,7 - 4 LEDice - DIO 0,1,2,3 - IC 7447 za 7.segm zaslon - DIO 0,1,2 - LDR - AIO - LM35 - AI1 - shunt i priključnice - acs712, AI0"
- note removed: "TO-DO: - zamijeniti 7447 s nekim drugim IC-om? (nema ga za kupiti) DONE: - 2 tipkala i pritezni otpornici (2 jumpera za pull up) - DIO 4,5 - 2 sklopke i pritezni otpornici (2 jumpera za pull up) - DIO 6,7 - 4 LEDice - DIO 0,1,2,3 - IC 7447 za 7.segm zaslon - DIO 0,1,2 - LDR - AIO - LM35 - AI1 - shunt i priključnice - acs712, AI0"

Commit message: Update myDAQExpansionBoard.kicad_sch
Parts:
- removed U?: 7447, symbol 74xx_IEEE:7447
- added J2, J4: Screw_Terminal_01x02, symbol Connector:Screw_Terminal_01x02
- added JP14, JP15: Jumper_2_Open, symbol Jumper:Jumper_2_Open
- added U1: 74LS47, Package_DIP:DIP-16_W7.62mm, symbol 74xx:74LS47
- D1, D2, D3, D4: renamed from D?; footprint (none) -> LED_THT:LED_D5.0mm
- J1: footprint (none) -> Library:OSTV7XX3151
- gave numbers to parts that had none: 46
Connections:
- net +5V: now also U5.16 (VCC1), U1.16 (VCC)
- net DIO0: now also U1.7 (A)
- net DIO1: now also U1.1 (B)
- net DIO2: now also U1.2 (C)
- net DIO3: now also U1.6 (D)
- net GND: now also U5.12 (GND), U5.13 (GND), U5.4 (GND), U5.5 (GND), U1.8 (GND)
- net at U5.11 (3Y): now also J4.1 (Pin_1)
- net at U5.14 (4Y): now also J4.2 (Pin_2)
- net at U5.3 (1Y): now also J2.1 (Pin_1)
- net at U5.6 (2Y): now also J2.2 (Pin_2)
- net VDD: now reaches U5.8 (VCC2)
- net VDD: now also JP15.2 (B)
- net at R8.1: now also U1.13 (a)
- net at R9.1: now also U1.12 (b)
- net at R13.1: now also U1.10 (d)
- net at R11.1: now also U1.11 (c)
- net at R16.1: now also U1.14 (g)
- net at R15.1: now also U1.15 (f)
- net at R12.2: now also U1.3 (LT), U1.4 (BI), U1.5 (RBI)
- net at R14.1: now also U1.9 (e)
- net at J5.1 (Pin_1), J5.2 (Pin_2): now also JP14.1 (A), JP15.1 (A); no longer R17.1
- net +15V: no longer names the net of J1.1 (Pin_1)
- net -15V: no longer names the net of J1.2 (Pin_2)
- net AO1: no longer names the net of J1.5 (Pin_5)
- new net SHUNT: JP14.2 (B), R17.1
- no-connect marks 1 -> 4
Other:
- note added: "H-MOST"
- note added: "NAPAJANJE"
- note added: "TO-DO: DONE: - 2 tipkala i pritezni otpornici (2 jumpera za pull up) - DIO 4,5 - 2 sklopke i pritezni otpornici (2 jumpera za pull up) - DIO 6,7 - 4 LEDice - DIO 0,1,2,3 - IC 7447 za 7.segm zaslon - DIO 0,1,2 - LDR - AIO - LM35 - AI1 - shunt i priključnice - acs712, AI0 - L293D 4 digitalna izlaza, DIP s profi podnožjem - zamijeniti 7447 s nekim drugim IC-om"
- note removed: "TO-DO: - zamijeniti 7447 s nekim drugim IC-om? (nema ga za kupiti) - L293D 2 digitalna izlaza, DIP s profi podnožjem DONE: - 2 tipkala i pritezni otpornici (2 jumpera za pull up) - DIO 4,5 - 2 sklopke i pritezni otpornici (2 jumpera za pull up) - DIO 6,7 - 4 LEDice - DIO 0,1,2,3 - IC 7447 za 7.segm zaslon - DIO 0,1,2 - LDR - AIO - LM35 - AI1 - shunt i priključnice - acs712, AI0"
- moved on the sheet: C1, C2, C3, C4, D1, D2, D3, D4, J1, J3, J5, JP1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

Commit message: Update myDAQExpansionBoard.kicad_sch
Parts:
- added J2, J3: Conn_01x05_Male, Connector_PinHeader_2.54mm:PinHeader_1x05_P2.54mm_Vertical, symbol Connector:Conn_01x05_Male
- renumbered J2 to J4, J3 to J5, J4 to J6, J5 to J7
Connections:
- net +5V: now also J2.1 (Pin_1), J2.2 (Pin_2), J2.3 (Pin_3), J2.4 (Pin_4), J2.5 (Pin_5)
- net GND: now also J3.1 (Pin_1), J3.2 (Pin_2), J3.3 (Pin_3), J3.4 (Pin_4), J3.5 (Pin_5)
Other:
- note added: "TO-DO: - dodati dva kanala da mjerenje brzine DONE: - 2 tipkala i pritezni otpornici (2 jumpera za pull up) - DIO 4,5 - 2 sklopke i pritezni otpornici (2 jumpera za pull up) - DIO 6,7 - 4 LEDice - DIO 0,1,2,3 - IC za 7.segm zaslon - DIO 0,1,2 - LDR - AIO - LM35 - AI1 - shunt i priključnice - acs712, AI0 - L293D 4 digitalna izlaza, DIP s profi podnožjem - staviti 1x05 strip za GND - staviti 1x05 s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"
- note removed: "TO-DO: DONE: - 2 tipkala i pritezni otpornici (2 jumpera za pull up) - DIO 4,5 - 2 sklopke i pritezni otpornici (2 jumpera za pull up) - DIO 6,7 - 4 LEDice - DIO 0,1,2,3 - IC 7447 za 7.segm zaslon - DIO 0,1,2 - LDR - AIO - LM35 - AI1 - shunt i priključnice - acs712, AI0 - L293D 4 digitalna izlaza, DIP s profi podnožjem - zamijeniti 7447 s nekim drugim IC-om"

Commit message: Update myDAQExpansionBoard.kicad_sch
Parts:
- added J?: Conn_01x08_Male, symbol Connector:Conn_01x08_Male
Connections:
- net DIO0: now also J?.8 (Pin_8)
- net DIO1: now also J?.7 (Pin_7)
- net DIO2: now also J?.6 (Pin_6)
- net DIO3: now also J?.5 (Pin_5)
- net DIO4: now also J?.4 (Pin_4)
- net DIO5: now also J?.3 (Pin_3)
- net DIO6: now also J?.2 (Pin_2)
- net DIO7: now also J?.1 (Pin_1)
Changed lines of the file:
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@@
+    )
+  )
+  (global_label "DIO7" (shape input) (at 247.65 132.08 0) (fields_autoplaced)
+    (effects (font (size 1.27 1.27)) (justify left))
+    (property "Intersheet References" "${INTERSHEET_REFS}" (id 0) (at 254.4779 132.0006 0)
+      (effects (font (size 1.27 1.27)) (justify left) hide)
+    )
+  )
+  (global_label "DIO2" (shape input) (at 247.65 144.78 0) (fields_autoplaced)
+    (effects (font (size 1.27 1.27)) (justify left))
+    (property "Intersheet References" "${INTERSHEET_REFS}" (id 0) (at 254.4779 144.7006 0)
+      (effects (font (size 1.27 1.27)) (justify left) hide)
     )
   )
@@
     )
   )
+  (global_label "DIO0" (shape input) (at 247.65 149.86 0) (fields_autoplaced)
+    (effects (font (size 1.27 1.27)) (justify left))
+    (property "Intersheet References" "${INTERSHEET_REFS}" (id 0) (at 254.4779 149.7806 0)
+      (effects (font (size 1.27 1.27)) (justify left) hide)
+    )
+  )
   (global_label "DIO2" (shape input) (at 193.675 54.61 180) (fields_autoplaced)
     (effects (font (size 1.27 1.27)) (justify right))
@@
     )
   )
+  (global_label "DIO4" (shape input) (at 247.65 139.7 0) (fields_autoplaced)
+    (effects (font (size 1.27 1.27)) (justify left))
+    (property "Intersheet References" "${INTERSHEET_REFS}" (id 0) (at 254.4779 139.6206 0)
+      (effects (font (size 1.27 1.27)) (justify left) hide)
+    )
+  )
   (global_label "DIO4" (shape input) (at 31.75 55.88 0) (fields_autoplaced)
     (effects (font (size 1.27 1.27)) (justify left))
@@
     )
   )
+  (global_label "DIO1" (shape input) (at 247.65 147.32 0) (fields_autoplaced)
+    (effects (font (size 1.27 1.27)) (justify left))
+    (property "Intersheet References" "${INTERSHEET_REFS}" (id 0) (at 254.4779 147.2406 0)
+      (effects (font (size 1.27 1.27)) (justify left) hide)
+    )
+  )
   (global_label "DIO6" (shape input) (at 128.905 49.53 180) (fields_autoplaced)
     (effects (font (size 1.27 1.27)) (justify right))
@@
     )
   )
+  (global_label "DIO5" (shape input) (at 247.65 137.16 0) (fields_autoplaced)
+    (effects (font (size 1.27 1.27)) (justify left))
+    (property "Intersheet References" "${INTERSHEET_REFS}" (id 0) (at 254.4779 137.0806 0)
+      (effects (font (size 1.27 1.27)) (justify left) hide)
+    )
+  )
+  (global_label "DIO6" (shape input) (at 247.65 134.62 0) (fields_autoplaced)
+    (effects (font (size 1.27 1.27)) (justify left))
+    (property "Intersheet References" "${INTERSHEET_REFS}" (id 0) (at 254.4779 134.5406 0)
+      (effects (font (size 1.27 1.27)) (justify left) hide)
+    )
+  )
   (global_label "DIO2" (shape input) (at 83.82 76.835 180) (fields_autoplaced)
     (effects (font (size 1.27 1.27)) (justify right))
     (property "Intersheet References" "${INTERSHEET_REFS}" (id 0) (at 76.9921 76.7556 0)
       (effects (font (size 1.27 1.27)) (justify right) hide)
+    )
+  )
+  (global_label "DIO3" (shape input) (at 247.65 142.24 0) (fields_autoplaced)
+    (effects (font (size 1.27 1.27)) (justify left))
+    (property "Intersheet References" "${INTERSHEET_REFS}" (id 0) (at 254.4779 142.1606 0)
+      (effects (font (size 1.27 1.27)) (justify left) hide)
     )
   )
@@
     (pin "2")
   )
+  (symbol (lib_id "Connector:Conn_01x08_Male") (at 242.57 139.7 0) (unit 1)
+    (in_bom yes) (on_board yes) (fields_autoplaced)
+    (property "Reference" "J?" (id 0) (at 243.205 130.841 0))
+    (property "Value" "Conn_01x08_Male" (id 1) (at 243.205 130.8409 0)
+      (effects (font (size 1.27 1.27)) hide)
+    )
+    (property "Footprint" "" (id 2) (at 242.57 139.7 0)
+      (effects (font (size 1.27 1.27)) hide)
+    )
+    (property "Datasheet" "~" (id 3) (at 242.57 139.7 0)
+      (effects (font (size 1.27 1.27)) hide)
+    )
+    (pin "1")
+    (pin "2")
+    (pin "3")
+    (pin "4")
+    (pin "5")
+    (pin "6")
+    (pin "7")
+    (pin "8")
+  )
   (symbol (lib_id "Device:R") (at 122.555 88.265 90) (unit 1)
     (in_bom yes) (on_board yes)
@@
       (reference "J7") (unit 1) (value "Screw_Terminal_01x02") (footprint "")
     )
+    (path "/e978b021-68a3-493c-9c98-1e7ae8b7e007"
+      (reference "J?") (unit 1) (value "Conn_01x08_Male") (footprint "")
+    )
     (path "/79d1d2fe-44ad-4ea6-a4d2-2be9874caeed"

Commit message: Update myDAQExpansionBoard.kicad_sch
Parts:
- gave numbers to parts that had none: 1
- renumbered J7 to J8
Other:
- note added: "TO-DO: DONE: - 2 tipkala i pritezni otpornici (2 jumpera za pull up) - DIO 4,5 - 2 sklopke i pritezni otpornici (2 jumpera za pull up) - DIO 6,7 - 4 LEDice - DIO 0,1,2,3 - IC za 7.segm zaslon - DIO 0,1,2 - LDR - AIO - LM35 - AI1 - shunt i priključnice - acs712, AI0 - L293D 4 digitalna izlaza, DIP s profi podnožjem - staviti 1x05 strip za GND - staviti 1x05 strip za +5V"
- note removed: "TO-DO: - dodati dva kanala da mjerenje brzine DONE: - 2 tipkala i pritezni otpornici (2 jumpera za pull up) - DIO 4,5 - 2 sklopke i pritezni otpornici (2 jumpera za pull up) - DIO 6,7 - 4 LEDice - DIO 0,1,2,3 - IC za 7.segm zaslon - DIO 0,1,2 - LDR - AIO - LM35 - AI1 - shunt i priključnice - acs712, AI0 - L293D 4 digitalna izlaza, DIP s profi podnožjem - staviti 1x05 strip za GND - staviti 1x05 s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"
Changed lines of the file:
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@@
     (stroke (width 0) (type default) (color 0 0 0 0))
   )
-  (text "TO-DO:\n- dodati dva kanala da mjerenje brzine\n\n\nDONE:\n- 2 tipkala i pritezni otpornici (2 jumpera za pull up) - DIO 4,5\n- 2 sklopke i pritezni otpornici (2 jumpera za pull up) - DIO 6,7\n- 4 LEDice - DIO 0,1,2,3\n- IC za 7.segm zaslon - DIO 0,1,2\n- LDR - AIO\n- LM35 - AI1\n- shunt i priključnice\n- acs712, AI0\n- L293D 4 digitalna izlaza, DIP s profi podnožjem\n- staviti 1x05 strip za GND\n- staviti 1x05 strip za +5V"
+  (text "TO-DO:\n\nDONE:\n- 2 tipkala i pritezni otpornici (2 jumpera za pull up) - DIO 4,5\n- 2 sklopke i pritezni otpornici (2 jumpera za pull up) - DIO 6,7\n- 4 LEDice - DIO 0,1,2,3\n- IC za 7.segm zaslon - DIO 0,1,2\n- LDR - AIO\n- LM35 - AI1\n- shunt i priključnice\n- acs712, AI0\n- L293D 4 digitalna izlaza, DIP s profi podnožjem\n- staviti 1x05 strip za GND\n- staviti 1x05 strip za +5V"
     (at 103.505 191.77 0)
     (effects (font (size 1.27 1.27)) (justify left bottom))
@@
   (symbol (lib_id "Jumper:Jumper_2_Open") (at 131.445 29.21 90) (unit 1)
     (in_bom yes) (on_board yes) (fields_autoplaced)
-    (property "Reference" "JP4" (id 0) (at 132.588 28.3753 90)
+    (property "Reference" "JP4" (id 0) (at 132.588 29.6438 90)
       (effects (font (size 1.27 1.27)) (justify right))
     )
     (property "Value" "Jumper_2_Open" (id 1) (at 132.588 30.9122 90)
-      (effects (font (size 1.27 1.27)) (justify right))
+      (effects (font (size 1.27 1.27)) (justify right) hide)
     )
     (property "Footprint" "" (id 2) (at 131.445 29.21 0)
@@
   (symbol (lib_id "Jumper:Jumper_2_Open") (at 162.56 29.845 90) (unit 1)
     (in_bom yes) (on_board yes) (fields_autoplaced)
-    (property "Reference" "JP5" (id 0) (at 163.703 29.0103 90)
+    (property "Reference" "JP5" (id 0) (at 163.703 30.2788 90)
       (effects (font (size 1.27 1.27)) (justify right))
     )
     (property "Value" "Jumper_2_Open" (id 1) (at 163.703 31.5472 90)
-      (effects (font (size 1.27 1.27)) (justify right))
+      (effects (font (size 1.27 1.27)) (justify right) hide)
     )
     (property "Footprint" "" (id 2) (at 162.56 29.845 0)
@@
   (symbol (lib_id "Connector:Screw_Terminal_01x02") (at 27.94 179.07 180) (unit 1)
     (in_bom yes) (on_board yes)
-    (property "Reference" "J7" (id 0) (at 27.94 181.61 0))
+    (property "Reference" "J8" (id 0) (at 27.94 181.61 0))
     (property "Value" "Screw_Terminal_01x02" (id 1) (at 25.908 176.0978 0)
       (effects (font (size 1.27 1.27)) (justify left) hide)
@@
   (symbol (lib_id "Connector:Conn_01x08_Male") (at 242.57 139.7 0) (unit 1)
     (in_bom yes) (on_board yes) (fields_autoplaced)
-    (property "Reference" "J?" (id 0) (at 243.205 130.841 0))
+    (property "Reference" "J7" (id 0) (at 243.205 130.841 0))
     (property "Value" "Conn_01x08_Male" (id 1) (at 243.205 130.8409 0)
       (effects (font (size 1.27 1.27)) hide)
@@
       (reference "J6") (unit 1) (value "Screw_Terminal_01x02") (footprint "")
     )
+    (path "/e978b021-68a3-493c-9c98-1e7ae8b7e007"
+      (reference "J7") (unit 1) (value "Conn_01x08_Male") (footprint "")
+    )
     (path "/ac60c730-ffb0-4282-932b-c2355fa71946"
-      (reference "J7") (unit 1) (value "Screw_Terminal_01x02") (footprint "")
-    )
-    (path "/e978b021-68a3-493c-9c98-1e7ae8b7e007"
-      (reference "J?") (unit 1) (value "Conn_01x08_Male") (footprint "")
+      (reference "J8") (unit 1) (value "Screw_Terminal_01x02") (footprint "")
     )
     (path "/79d1d2fe-44ad-4ea6-a4d2-2be9874caeed"
