File: KiCAD files/myDAQExpansionBoard/myDAQExpansionBoard.kicad_sch (KiCad schematic)
At the start: 59 parts, among them J1 OSTV7XX3151, J2 Conn_01x05_Male, J3 Conn_01x05_Male, J4 Screw_Terminal_01x02, J5 Screw_Terminal_01x02, J6 Screw_Terminal_01x02, J7 Conn_01x08_Male, J8 Screw_Terminal_01x02, SW1 SW_Push, SW2 SW_Push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

Commit message: layout
Parts:
- C1, C2, C3: footprint (none) -> Capacitor_THT:C_Disc_D4.3mm_W1.9mm_P5.00mm
- C4: footprint (none) -> Capacitor_SMD:C_0603_1608Metric
- J4, J6: footprint (none) -> TerminalBlock_Phoenix:TerminalBlock_Phoenix_MKDS-1,5-2-5.08_1x02_P5.08mm_Horizontal
- J5, J8, JP1, JP14, JP15, JP2, JP3, JP4, JP5, JP6, JP7, JP8: footprint (none) -> Connector_PinHeader_2.54mm:PinHeader_1x02_P2.54mm_Vertical
- J7: footprint (none) -> Connector_PinHeader_2.54mm:PinHeader_1x08_P2.54mm_Vertical
- JP10, JP11, JP12, JP13, JP9: footprint (none) -> Connector_PinHeader_2.54mm:PinHeader_1x03_P2.54mm_Vertical
- R1, R10, R11, R12, R13, R14, R15, R16, R19, R2, R3, R4, R5, R6, R7, R8, R9: footprint (none) -> Resistor_THT:R_Axial_DIN0207_L6.3mm_D2.5mm_P10.16mm_Horizontal
- R17: footprint (none) -> Library:R_Axial_Power_L60.0mm_W14.0mm_P71.12mm
- R18: footprint (none) -> OptoDevice:R_LDR_7x6mm_P5.1mm_Vertical
- SW1, SW2: footprint (none) -> Library:SW_PUSH-12mm_Wuerth-430476085716
- SW3, SW4: footprint (none) -> Button_Switch_THT:SW_DIP_SPSTx01_Slide_9.78x4.72mm_W7.62mm_P2.54mm

Commit message: layout
Parts:
- C1, C2, C3: footprint Capacitor_THT:C_Disc_D4.3mm_W1.9mm_P5.00mm -> Capacitor_SMD:C_0603_1608Metric
- R1, R10, R11, R12, R13, R14, R15, R16, R19, R2, R3, R4, R5, R6, R7, R8, R9: footprint Resistor_THT:R_Axial_DIN0207_L6.3mm_D2.5mm_P10.16mm_Horizontal -> Resistor_SMD:R_0603_1608Metric
Connections:
- net GND: now also D1.1 (K), D2.1 (K), D3.1 (K), D4.1 (K); no longer R1.2, R10.2, R5.2, R7.2
- net at R7.1: now also JP7.2 (B); no longer D3.1 (K)
- net at R1.1: now also JP1.2 (B); no longer D1.1 (K)
- net at D1.2 (A): now also R1.2; no longer JP1.2 (B)
- net at D3.2 (A): now also R7.2; no longer JP7.2 (B)
- net at JP8.2 (B): now also R10.1; no longer D4.2 (A)
- net at JP6.2 (B): now also R5.1; no longer D2.2 (A)
- new net: D4.2 (A), R10.2
- new net: D2.2 (A), R5.2
Other:
- moved on the sheet: D1, D2, D3, D4, R1, R10, R5, R7

Commit message: update
Parts:
- added H1, H2, H3, H4: MountingHole_Pad, MountingHole:MountingHole_3.2mm_M3_Pad_Via, symbol Mechanical:MountingHole_Pad
- renumbered JP5 to JP1, JP1 to JP2, JP2 to JP3, JP3 to JP4, JP4 to JP5
Connections:
- net +5V: now also JP2.2 (B); no longer JP5.2 (B)
- net DIO0: now also JP5.1 (A); no longer JP2.1 (A)
- net at R2.1: now also JP1.1 (A); no longer JP3.1 (A)
- net at R3.1: now also JP2.1 (A); no longer JP4.1 (A)
- net at R4.1: now also JP3.1 (A); no longer JP5.1 (A)
- net at R1.1: now also JP5.2 (B); no longer JP2.2 (B)
- net at R6.1: now also JP4.1 (A); no longer JP1.1 (A)
- no-connect marks 4 -> 8
Other:
- note added: "SN74LS74 (6kn u electronic centru)"
- moved on the sheet: JP1, JP2, JP3, JP4, JP5

Commit message: update
Parts:
- added J9: Screw_Terminal_01x02, Connector_PinHeader_2.54mm:PinHeader_1x02_P2.54mm_Vertical, symbol Connector:Screw_Terminal_01x02
Connections:
- net GND: now also J9.1 (Pin_1), J9.2 (Pin_2)

Commit message: Update myDAQExpansionBoard.kicad_sch
Other:
- note added: "TO-DO: - debounce kondenzatori na tipkalima i možda sklopkama DONE: - 2 tipkala i pritezni otpornici (2 jumpera za pull up) - DIO 4,5 - 2 sklopke i pritezni otpornici (2 jumpera za pull up) - DIO 6,7 - 4 LEDice - DIO 0,1,2,3 - IC za 7.segm zaslon - DIO 0,1,2 - LDR - AIO - LM35 - AI1 - shunt i priključnice - acs712, AI0 - L293D 4 digitalna izlaza, DIP s profi podnožjem - staviti 1x05 strip za GND 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"
- note removed: "TO-DO: DONE: - 2 tipkala i pritezni otpornici (2 jumpera za pull up) - DIO 4,5 - 2 sklopke i pritezni otpornici (2 jumpera za pull up) - DIO 6,7 - 4 LEDice - DIO 0,1,2,3 - IC za 7.segm zaslon - DIO 0,1,2 - LDR - AIO - LM35 - AI1 - shunt i priključnice - acs712, AI0 - L293D 4 digitalna izlaza, DIP s profi podnožjem - staviti 1x05 strip za GND - staviti 1x05 strip za +5V"
Changed lines of the file:
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@@
     (stroke (width 0) (type default) (color 0 0 0 0))
   )
-  (text "TO-DO:\n\nDONE:\n- 2 tipkala i pritezni otpornici (2 jumpera za pull up) - DIO 4,5\n- 2 sklopke i pritezni otpornici (2 jumpera za pull up) - DIO 6,7\n- 4 LEDice - DIO 0,1,2,3\n- IC za 7.segm zaslon - DIO 0,1,2\n- LDR - AIO\n- LM35 - AI1\n- shunt i priključnice\n- acs712, AI0\n- L293D 4 digitalna izlaza, DIP s profi podnožjem\n- staviti 1x05 strip za GND\n- staviti 1x05 strip za +5V"
+  (text "TO-DO:\n- debounce kondenzatori na tipkalima i možda sklopkama\n\nDONE:\n- 2 tipkala i pritezni otpornici (2 jumpera za pull up) - DIO 4,5\n- 2 sklopke i pritezni otpornici (2 jumpera za pull up) - DIO 6,7\n- 4 LEDice - DIO 0,1,2,3\n- IC za 7.segm zaslon - DIO 0,1,2\n- LDR - AIO\n- LM35 - AI1\n- shunt i priključnice\n- acs712, AI0\n- L293D 4 digitalna izlaza, DIP s profi podnožjem\n- staviti 1x05 strip za GND\n- staviti 1x05 strip za +5V"
     (at 103.505 191.77 0)
     (effects (font (size 1.27 1.27)) (justify left bottom))

Commit message: update
Parts:
- removed U2: HDSP-7501, Display_7Segment:HDSP-A151, symbol Display_Character:HDSP-7501
- added U2: 7segm-symbol, Library:7segm-SA52, symbol Symbols:7segm-symbol
- SW1, SW2: footprint Library:SW_PUSH-12mm_Wuerth-430476085716 -> Library:Omron_B3F-12x12mm
Connections:
- net at R8.2: now also U2.7 (A)
- net at R9.2: now also U2.6 (B)
- net at R11.2: now also U2.4 (C)
- net at R16.2: now also U2.10 (G)
- net at JP9.2 (C): now also U2.8 (CA/CC)
- net at R13.2: now also U2.2 (D)
- net at R15.2: now also U2.9 (F)
- net at R14.2: now also U2.1 (E)
- no-connect marks 8 -> 9
Other:
- note added: "TO-DO: - debounce kondenzatori na tipkalima i možda sklopkama - odvojiti analogni i digitalni gnd - spst sklopke zamijeniti footprinte DONE: - 2 tipkala i pritezni otpornici (2 jumpera za pull up) - DIO 4,5 - 2 sklopke i pritezni otpornici (2 jumpera za pull up) - DIO 6,7 - 4 LEDice - DIO 0,1,2,3 - IC za 7.segm zaslon - DIO 0,1,2 - LDR - AIO - LM35 - AI1 - shunt i priključnice - acs712, AI0 - L29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"
- note removed: "TO-DO: - debounce kondenzatori na tipkalima i možda sklopkama DONE: - 2 tipkala i pritezni otpornici (2 jumpera za pull up) - DIO 4,5 - 2 sklopke i pritezni otpornici (2 jumpera za pull up) - DIO 6,7 - 4 LEDice - DIO 0,1,2,3 - IC za 7.segm zaslon - DIO 0,1,2 - LDR - AIO - LM35 - AI1 - shunt i priključnice - acs712, AI0 - L293D 4 digitalna izlaza, DIP s profi podnožjem - staviti 1x05 strip za GND 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"
Changed lines of the file:
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@@
   (junction (at 34.29 189.865) (diameter 0) (color 0 0 0 0)
   )
-  (junction (at 152.4 86.995) (diameter 0) (color 0 0 0 0)
-  )
   (junction (at 131.445 49.53) (diameter 0) (color 0 0 0 0)
   )
@@
   (junction (at 43.815 68.58) (diameter 0) (color 0 0 0 0)
   )
+  (no_connect (at 151.13 92.075))
   (no_connect (at 185.42 153.035))
   (no_connect (at 135.89 89.535))
@@
     (stroke (width 0) (type default) (color 0 0 0 0))
   )
+  (wire (pts (xy 152.4 94.615) (xy 151.13 94.615))
+    (stroke (width 0) (type default) (color 0 0 0 0))
+  )
   (wire (pts (xy 116.205 81.915) (xy 109.22 81.915))
     (stroke (width 0) (type default) (color 0 0 0 0))
@@
     (stroke (width 0) (type default) (color 0 0 0 0))
   )
-  (wire (pts (xy 152.4 83.185) (xy 152.4 86.995))
-    (stroke (width 0) (type default) (color 0 0 0 0))
-  )
   (wire (pts (xy 248.92 112.395) (xy 248.92 114.3))
     (stroke (width 0) (type default) (color 0 0 0 0))
@@
     (stroke (width 0) (type default) (color 0 0 0 0))
   )
-  (wire (pts (xy 152.4 89.535) (xy 152.4 86.995))
+  (wire (pts (xy 152.4 83.185) (xy 152.4 94.615))
     (stroke (width 0) (type default) (color 0 0 0 0))
   )
@@
     (stroke (width 0) (type default) (color 0 0 0 0))
   )
-  (wire (pts (xy 151.13 86.995) (xy 152.4 86.995))
-    (stroke (width 0) (type default) (color 0 0 0 0))
-  )
   (wire (pts (xy 98.425 22.225) (xy 98.425 23.495))
     (stroke (width 0) (type default) (color 0 0 0 0))
@@
     (stroke (width 0) (type default) (color 0 0 0 0))
   )
-  (wire (pts (xy 151.13 89.535) (xy 152.4 89.535))
-    (stroke (width 0) (type default) (color 0 0 0 0))
-  )
   (polyline (pts (xy 184.15 19.05) (xy 184.15 80.01))
     (stroke (width 0) (type default) (color 0 0 0 0))
@@
     (stroke (width 0) (type default) (color 0 0 0 0))
   )
-  (text "TO-DO:\n- debounce kondenzatori na tipkalima i možda sklopkama\n\nDONE:\n- 2 tipkala i pritezni otpornici (2 jumpera za pull up) - DIO 4,5\n- 2 sklopke i pritezni otpornici (2 jumpera za pull up) - DIO 6,7\n- 4 LEDice - DIO 0,1,2,3\n- IC za 7.segm zaslon - DIO 0,1,2\n- LDR - AIO\n- LM35 - AI1\n- shunt i priključnice\n- acs712, AI0\n- L293D 4 digitalna izlaza, DIP s profi podnožjem\n- staviti 1x05 strip za GND\n- staviti 1x05 strip za +5V"
-    (at 103.505 191.77 0)
+  (text "TO-DO:\n- debounce kondenzatori na tipkalima i možda sklopkama\n- odvojiti analogni i digitalni gnd\n- spst sklopke zamijeniti footprinte\n\nDONE:\n- 2 tipkala i pritezni otpornici (2 jumpera za pull up) - DIO 4,5\n- 2 sklopke i pritezni otpornici (2 jumpera za pull up) - DIO 6,7\n- 4 LEDice - DIO 0,1,2,3\n- IC za 7.segm zaslon - DIO 0,1,2\n- LDR - AIO\n- LM35 - AI1\n- shunt i priključnice\n- acs712, AI0\n- L293D 4 digitalna izlaza, DIP s profi podnožjem\n- staviti 1x05 strip za GND\n- staviti 1x05 strip za +5V"
+    (at 97.79 191.77 0)
     (effects (font (size 1.27 1.27)) (justify left bottom))
   )
@@
     (pin "9")
   )
+  (symbol (lib_id "Symbols:7segm-symbol") (at 143.51 81.915 0) (unit 1)
+    (in_bom yes) (on_board yes)
+    (property "Reference" "U2" (id 0) (at 139.7 67.945 0))
+    (property "Value" "7segm-symbol" (id 1) (at 143.51 98.425 0))
+    (property "Footprint" "Library:7segm-SA52" (id 2) (at 143.51 66.675 0)
+      (effects (font (size 1.27 1.27)) hide)
+    )
+    (property "Datasheet" "" (id 3) (at 143.51 66.675 0)
+      (effects (font (size 1.27 1.27)) hide)
+    )
+    (pin "1")
+    (pin "10")
+    (pin "2")
+    (pin "3")
+    (pin "4")
+    (pin "5")
+    (pin "6")
+    (pin "7")
+    (pin "8")
+    (pin "9")
+  )
   (symbol (lib_id "Device:LED") (at 224.155 54.61 180) (unit 1)
     (in_bom yes) (on_board yes) (fields_autoplaced)
@@
       (effects (font (size 1.27 1.27)) hide)
     )
-    (property "Footprint" "Library:SW_PUSH-12mm_Wuerth-430476085716" (id 2) (at 107.95 43.815 0)
+    (property "Footprint" "Library:Omron_B3F-12x12mm" (id 2) (at 107.95 43.815 0)
       (effects (font (size 1.27 1.27)) hide)
     )
@@
       (effects (font (size 1.27 1.27)) hide)
     )
-    (property "Footprint" "Library:SW_PUSH-12mm_Wuerth-430476085716" (id 2) (at 74.295 43.815 0)
+    (property "Footprint" "Library:Omron_B3F-12x12mm" (id 2) (at 74.295 43.815 0)
       (effects (font (size 1.27 1.27)) hide)
     )
@@
     (pin "1")
   )
-  (symbol (lib_id "Display_Character:HDSP-7501") (at 143.51 79.375 0) (unit 1)
-    (in_bom yes) (on_board yes) (fields_autoplaced)
-    (property "Reference" "U2" (id 0) (at 143.51 65.5122 0))
-    (property "Value" "HDSP-7501" (id 1) (at 143.51 65.5121 0)
-      (effects (font (size 1.27 1.27)) hide)
-    )
-    (property "Footprint" "Display_7Segment:HDSP-A151" (id 2) (at 143.51 93.345 0)
-      (effects (font (size 1.27 1.27)) hide)
-    )
-    (property "Datasheet" "https://docs.broadcom.com/docs/AV02-2553EN" (id 3) (at 130.81 65.405 0)
-      (effects (font (size 1.27 1.27)) hide)
-    )
-    (pin "1")
-    (pin "10")
-    (pin "2")
-    (pin "3")
-    (pin "4")
-    (pin "5")
-    (pin "6")
-    (pin "7")
-    (pin "8")
-    (pin "9")
-  )
   (symbol (lib_id "Device:C") (at 99.06 120.65 0) (unit 1)
     (in_bom yes) (on_board yes) (fields_autoplaced)
@@
     )
     (path "/90f2d58e-a255-450d-bc74-dbc1a747cc3e"
-      (reference "SW1") (unit 1) (value "SW_Push") (footprint "Library:SW_PUSH-12mm_Wuerth-430476085716")
+      (reference "SW1") (unit 1) (value "SW_Push") (footprint "Library:Omron_B3F-12x12mm")
     )
     (path "/62493830-d3bc-4a72-aaba-47cd882ea607"
-      (reference "SW2") (unit 1) (value "SW_Push") (footprint "Library:SW_PUSH-12mm_Wuerth-430476085716")
+      (reference "SW2") (unit 1) (value "SW_Push") (footprint "Library:Omron_B3F-12x12mm")
     )
     (path "/f29a92cb-91c3-4fb9-862c-dce8db47644e"
@@
       (reference "U1") (unit 1) (value "74LS47") (footprint "Package_DIP:DIP-16_W7.62mm")
     )
-    (path "/d638cae5-ce3b-465f-bf3c-765cde42189d"
-      (reference "U2") (unit 1) (value "HDSP-7501") (footprint "Display_7Segment:HDSP-A151")
+    (path "/14f40f3f-2684-4318-a5c7-b91006f6c589"
+      (reference "U2") (unit 1) (value "7segm-symbol") (footprint "Library:7segm-SA52")
     )
     (path "/20d266e3-011c-45d0-9f23-f4e509e2a6fc"
