File: KiCAD files/myDAQExpansionBoard/myDAQExpansionBoard.kicad_pcb (KiCad board)
At the start: 2 copper layers, 100 x 100 mm, 59 parts, among them J1 OSTV7XX3151, J2 Conn_01x05_Male, J3 Conn_01x05_Male, J4 Screw_Terminal_01x02, J5 Screw_Terminal_01x02, J6 Screw_Terminal_01x02, J7 Conn_01x08_Male, J8 Screw_Terminal_01x02, SW1 SW_Push, SW2 SW_Push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

Commit message: layout
Parts:
- C1, C2, C3: footprint Capacitor_THT:C_Disc_D4.3mm_W1.9mm_P5.00mm -> Capacitor_SMD:C_0603_1608Metric
- R1, R10, R11, R12, R13, R14, R15, R16, R19, R2, R3, R4, R5, R6, R7, R8, R9: footprint Resistor_THT:R_Axial_DIN0207_L6.3mm_D2.5mm_P10.16mm_Horizontal -> Resistor_SMD:R_0603_1608Metric
- moved U3 212.8 mm to (11.2, 101.8), turned to 90 degrees
- moved R18 198.3 mm to (24.7, 136.8)
- moved R17 120.0 mm to (11.2, 137.4), turned to 90 degrees
- moved JP7 110.4 mm to (153.6, 140.9)
- moved J4 110.4 mm to (92.1, 103.6), turned to 90 degrees
- moved SW1 106.1 mm to (40.5, 134.3)
- moved SW2 105.4 mm to (58.4, 134.3)
- moved SW3 103.6 mm to (82.0, 133.6), turned to -90 degrees
- moved JP1 94.0 mm to (137.6, 140.9)
- moved JP6 93.0 mm to (145.6, 140.9)
- moved D2 87.8 mm to (145.6, 157.5), turned to 90 degrees
- moved C3 87.5 mm to (73.8, 109.4)
- moved J2 80.1 mm to (92.0, 60.4)
- moved SW4 79.3 mm to (90.2, 133.6), turned to -90 degrees
- moved D4 74.0 mm to (161.6, 154.9), turned to -90 degrees
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Connections:
- D1 pad 1: Net-(D1-Pad1) -> GND
- D1 pad 2: Net-(D1-Pad2) -> Net-(R1-Pad2)
- D2 pad 1: Net-(D2-Pad1) -> GND
- D2 pad 2: Net-(D2-Pad2) -> Net-(R5-Pad2)
- D3 pad 1: Net-(D3-Pad1) -> GND
- D3 pad 2: Net-(D3-Pad2) -> Net-(R7-Pad2)
- D4 pad 1: Net-(D4-Pad1) -> GND
- D4 pad 2: Net-(D4-Pad2) -> Net-(R10-Pad2)
- JP1 pad 2: Net-(D1-Pad2) -> Net-(JP1-Pad2)
- JP6 pad 2: Net-(D2-Pad2) -> Net-(JP6-Pad2)
- JP7 pad 2: Net-(D3-Pad2) -> Net-(JP7-Pad2)
- JP8 pad 2: Net-(D4-Pad2) -> Net-(JP8-Pad2)
- R1 pad 1: Net-(D1-Pad1) -> Net-(JP1-Pad2)
- R1 pad 2: GND -> Net-(R1-Pad2)
- R10 pad 1: Net-(D4-Pad1) -> Net-(JP8-Pad2)
- R10 pad 2: GND -> Net-(R10-Pad2)
- R5 pad 1: Net-(D2-Pad1) -> Net-(JP6-Pad2)
- R5 pad 2: GND -> Net-(R5-Pad2)
- R7 pad 1: Net-(D3-Pad1) -> Net-(JP7-Pad2)
- R7 pad 2: GND -> Net-(R7-Pad2)

Commit message: update
Parts:
- added H1: MountingHole_Pad, MountingHole:MountingHole_3.2mm_M3_Pad_Via, F.Cu at (135.1, 50.6)
- added H2: MountingHole_Pad, MountingHole:MountingHole_3.2mm_M3_Pad_Via, F.Cu at (135.1, 140.6)
- added H3: MountingHole_Pad, MountingHole:MountingHole_3.2mm_M3_Pad_Via, F.Cu at (45.1, 140.6)
- added H4: MountingHole_Pad, MountingHole:MountingHole_3.2mm_M3_Pad_Via, F.Cu at (45.1, 50.6)
- moved U3 165.7 mm to (175.8, 120.6), turned to -90 degrees
- moved U4 155.1 mm to (49.0, 96.4), turned to -90 degrees
- moved JP6 81.3 mm to (226.7, 146.9)
- moved JP7 81.3 mm to (234.7, 146.9)
- moved JP8 81.3 mm to (242.7, 146.7)
- moved R1 81.2 mm to (218.7, 154.6)
- moved R10 81.2 mm to (242.7, 154.6)
- moved R5 81.2 mm to (226.7, 154.6)
- moved R7 81.2 mm to (234.7, 154.6)
- moved D1 81.2 mm to (218.6, 162.5)
- moved D2 81.2 mm to (226.6, 162.5)
- moved D3 81.2 mm to (234.6, 159.9)
- moved D4 81.2 mm to (242.6, 159.9)
- moved JP11 74.9 mm to (65.3, 61.5), turned to 180 degrees
- moved JP1 73.3 mm to (206.1, 114.8)
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Connections:
- JP1 pad 1: DIO0 -> Net-(JP1-Pad1)
- JP1 pad 2: Net-(JP1-Pad2) -> +5V
- JP3 pad 1: Net-(JP3-Pad1) -> Net-(R4-Pad1)
- JP4 pad 1: Net-(JP4-Pad1) -> Net-(R6-Pad1)
- JP5 pad 1: Net-(JP5-Pad1) -> DIO0
- JP5 pad 2: +5V -> Net-(R1-Pad1)
- R1 pad 1: Net-(JP1-Pad2) -> Net-(R1-Pad1)
- R2 pad 1: Net-(JP2-Pad1) -> Net-(JP1-Pad1)
- R3 pad 1: Net-(JP3-Pad1) -> Net-(JP2-Pad1)
- R4 pad 1: Net-(JP4-Pad1) -> Net-(R4-Pad1)
- R6 pad 1: Net-(JP5-Pad1) -> Net-(R6-Pad1)
Routing:
- net Net-(JP11-Pad1): track 0.00 -> 40.9 mm
- net AI1+: track 0.00 -> 26.9 mm
- net +5V: track 0.00 -> 17.5 mm
- net DIO7: track 0.00 -> 9.19 mm
- net DIO0: track 0.00 -> 9.18 mm
- net DIO6: track 0.00 -> 8.62 mm
- net DIO1: track 0.00 -> 8.57 mm
- net DIO5: track 0.00 -> 8.17 mm
- net DIO2: track 0.00 -> 8.09 mm
- net DIO4: track 0.00 -> 7.61 mm
- net DIO3: track 0.00 -> 7.52 mm
- net AO0: track 0.00 -> 7.35 mm
- net unconnected-(J1-Pad2): track 0.00 -> 2.54 mm
- net unconnected-(J1-Pad5): track 0.00 -> 2.54 mm
- net unconnected-(J1-Pad1): track 0.00 -> 2.54 mm
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Other:
- outline, holes or cut-outs redrawn
- board text added: "5V"
- board text added: "DIO0"
- board text added: "DIO1"
- board text added: "DIO2"
- board text added: "DIO3"
- board text added: "DIO4"
- board text added: "DIO5"
- board text added: "DIO6"
- board text added: "DIO7"
- board text added: "GND"

Commit message: update
Parts:
- added J9: Screw_Terminal_01x02, Connector_PinHeader_2.54mm:PinHeader_1x02_P2.54mm_Vertical, F.Cu at (173.4, 73.9)
Changed lines of the file:
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@@
   (net 65 "unconnected-(H4-Pad1)")
   (net 66 "Net-(JP1-Pad1)")
-  (net 67 "Net-(R4-Pad1)")
-  (net 68 "Net-(R6-Pad1)")
-  (net 69 "Net-(R1-Pad1)")
+  (net 67 "Net-(JP3-Pad1)")
+  (net 68 "Net-(JP4-Pad1)")
+  (net 69 "Net-(JP5-Pad2)")
   (footprint "Resistor_SMD:R_0603_1608Metric" (layer "F.Cu")
     (at 103.0325 179)
@@
       (net 17 "DIO0") (pinfunction "A") (pintype "passive"))
     (pad "2" thru_hole oval (at 0 2.54) (size 1.7 1.7) (drill 1) (layers *.Cu *.Mask)
-      (net 69 "Net-(R1-Pad1)") (pinfunction "B") (pintype "passive"))
+      (net 69 "Net-(JP5-Pad2)") (pinfunction "B") (pintype "passive"))
     (model "${KICAD6_3DMODEL_DIR}/Connector_PinHeader_2.54mm.3dshapes/PinHeader_1x02_P2.54mm_Vertical.wrl"
       (offset (xyz 0 0 0))
@@
       (net 40 "Net-(R8-Pad2)") (pintype "passive"))
     (model "${KICAD6_3DMODEL_DIR}/Resistor_SMD.3dshapes/R_0603_1608Metric.wrl"
+      (offset (xyz 0 0 0))
+      (scale (xyz 1 1 1))
+      (rotate (xyz 0 0 0))
+    )
+  )
+  (footprint "Connector_PinHeader_2.54mm:PinHeader_1x02_P2.54mm_Vertical" (layer "F.Cu")
+    (at 173.4 73.9)
+    (descr "Through hole straight pin header, 1x02, 2.54mm pitch, single row")
+    (tags "Through hole pin header THT 1x02 2.54mm single row")
+    (property "Sheetfile" "myDAQExpansionBoard.kicad_sch")
+    (property "Sheetname" "")
+    (attr through_hole)
+    (fp_text reference "J9" (at 0 -2.33) (layer "F.SilkS")
+      (effects (font (size 1 1) (thickness 0.15)))
+    )
+    (fp_text value "Screw_Terminal_01x02" (at 0 4.87) (layer "F.Fab")
+      (effects (font (size 1 1) (thickness 0.15)))
+    )
+    (fp_text user "${REFERENCE}" (at 0 1.27 90) (layer "F.Fab")
+      (effects (font (size 1 1) (thickness 0.15)))
+    )
+    (fp_line (start -1.33 0) (end -1.33 -1.33) (layer "F.SilkS") (width 0.12))
+    (fp_line (start -1.33 -1.33) (end 0 -1.33) (layer "F.SilkS") (width 0.12))
+    (fp_line (start -1.33 3.87) (end 1.33 3.87) (layer "F.SilkS") (width 0.12))
+    (fp_line (start 1.33 1.27) (end 1.33 3.87) (layer "F.SilkS") (width 0.12))
+    (fp_line (start -1.33 1.27) (end 1.33 1.27) (layer "F.SilkS") (width 0.12))
+    (fp_line (start -1.33 1.27) (end -1.33 3.87) (layer "F.SilkS") (width 0.12))
+    (fp_line (start 1.8 -1.8) (end -1.8 -1.8) (layer "F.CrtYd") (width 0.05))
+    (fp_line (start -1.8 4.35) (end 1.8 4.35) (layer "F.CrtYd") (width 0.05))
+    (fp_line (start -1.8 -1.8) (end -1.8 4.35) (layer "F.CrtYd") (width 0.05))
+    (fp_line (start 1.8 4.35) (end 1.8 -1.8) (layer "F.CrtYd") (width 0.05))
+    (fp_line (start -1.27 -0.635) (end -0.635 -1.27) (layer "F.Fab") (width 0.1))
+    (fp_line (start 1.27 3.81) (end -1.27 3.81) (layer "F.Fab") (width 0.1))
+    (fp_line (start 1.27 -1.27) (end 1.27 3.81) (layer "F.Fab") (width 0.1))
+    (fp_line (start -0.635 -1.27) (end 1.27 -1.27) (layer "F.Fab") (width 0.1))
+    (fp_line (start -1.27 3.81) (end -1.27 -0.635) (layer "F.Fab") (width 0.1))
+    (pad "1" thru_hole rect (at 0 0) (size 1.7 1.7) (drill 1) (layers *.Cu *.Mask)
+      (net 2 "GND") (pinfunction "Pin_1") (pintype "passive"))
+    (pad "2" thru_hole oval (at 0 2.54) (size 1.7 1.7) (drill 1) (layers *.Cu *.Mask)
+      (net 2 "GND") (pinfunction "Pin_2") (pintype "passive"))
+    (model "${KICAD6_3DMODEL_DIR}/Connector_PinHeader_2.54mm.3dshapes/PinHeader_1x02_P2.54mm_Vertical.wrl"
       (offset (xyz 0 0 0))
       (scale (xyz 1 1 1))
@@
     (fp_line (start -0.635 -1.27) (end 1.27 -1.27) (layer "F.Fab") (width 0.1))
     (pad "1" thru_hole rect (at 0 0) (size 1.7 1.7) (drill 1) (layers *.Cu *.Mask)
-      (net 67 "Net-(R4-Pad1)") (pinfunction "A") (pintype "passive"))
+      (net 67 "Net-(JP3-Pad1)") (pinfunction "A") (pintype "passive"))
     (pad "2" thru_hole oval (at 0 2.54) (size 1.7 1.7) (drill 1) (layers *.Cu *.Mask)
       (net 1 "+5V") (pinfunction "B") (pintype "passive"))
@@
     (fp_line (start -0.8 -0.4125) (end 0.8 -0.4125) (layer "F.Fab") (width 0.1))
     (pad "1" smd roundrect (at -0.825 0 270) (size 0.8 0.95) (layers "F.Cu" "F.Paste" "F.Mask") (roundrect_rratio 0.25)
-      (net 69 "Net-(R1-Pad1)") (pintype "passive"))
+      (net 69 "Net-(JP5-Pad2)") (pintype "passive"))
     (pad "2" smd roundrect (at 0.825 0 270) (size 0.8 0.95) (layers "F.Cu" "F.Paste" "F.Mask") (roundrect_rratio 0.25)
       (net 4 "Net-(D1-Pad2)") (pintype "passive"))
@@
     (fp_line (start 0.8 -0.4125) (end 0.8 0.4125) (layer "F.Fab") (width 0.1))
     (pad "1" smd roundrect (at -0.825 0) (size 0.8 0.95) (layers "F.Cu" "F.Paste" "F.Mask") (roundrect_rratio 0.25)
-      (net 67 "Net-(R4-Pad1)") (pintype "passive"))
+      (net 67 "Net-(JP3-Pad1)") (pintype "passive"))
     (pad "2" smd roundrect (at 0.825 0) (size 0.8 0.95) (layers "F.Cu" "F.Paste" "F.Mask") (roundrect_rratio 0.25)
       (net 23 "DIO6") (pintype "passive"))
@@
     (fp_line (start -1.27 3.81) (end -1.27 -0.635) (layer "F.Fab") (width 0.1))
     (pad "1" thru_hole rect (at 0 0) (size 1.7 1.7) (drill 1) (layers *.Cu *.Mask)
-      (net 68 "Net-(R6-Pad1)") (pinfunction "A") (pintype "passive"))
+      (net 68 "Net-(JP4-Pad1)") (pinfunction "A") (pintype "passive"))
     (pad "2" thru_hole oval (at 0 2.54) (size 1.7 1.7) (drill 1) (layers *.Cu *.Mask)
       (net 1 "+5V") (pinfunction "B") (pintype "passive"))
@@
     (fp_line (start -0.8 -0.4125) (end 0.8 -0.4125) (layer "F.Fab") (width 0.1))
     (pad "1" smd roundrect (at -0.825 0) (size 0.8 0.95) (layers "F.Cu" "F.Paste" "F.Mask") (roundrect_rratio 0.25)
-      (net 68 "Net-(R6-Pad1)") (pintype "passive"))
+      (net 68 "Net-(JP4-Pad1)") (pintype "passive"))
     (pad "2" smd roundrect (at 0.825 0) (size 0.8 0.95) (layers "F.Cu" "F.Paste" "F.Mask") (roundrect_rratio 0.25)
       (net 24 "DIO7") (pintype "passive"))

Commit message: update
Parts:
- SW1, SW2: footprint Library:SW_PUSH-12mm_Wuerth-430476085716 -> Library:Omron_B3F-12x12mm
- U2: value HDSP-7501 -> 7segm-symbol; footprint Display_7Segment:HDSP-A151 -> Library:7segm-SA52
- moved SW1 9.52 mm to (84.0, 141.1), turned to 90 degrees
- moved SW2 9.52 mm to (101.8, 141.1), turned to 90 degrees
- moved JP9 7.11 mm to (112.3, 160.9)
- moved U2 4.76 mm to (116.9, 175.9)
Connections:
- U2 pad 1: Net-(JP9-Pad2) -> Net-(R14-Pad2)
- U2 pad 10: Net-(R8-Pad2) -> Net-(R16-Pad2)
- U2 pad 2: Net-(R15-Pad2) -> Net-(R13-Pad2)
- U2 pad 3: Net-(R16-Pad2) -> unconnected-(U2-Pad3)
- U2 pad 4: Net-(R14-Pad2) -> Net-(R11-Pad2)
- U2 pad 5: Net-(R13-Pad2) -> unconnected-(U2-Pad5)
- U2 pad 6: Net-(JP9-Pad2) -> Net-(R9-Pad2)
- U2 pad 7: unconnected-(U2-Pad7) -> Net-(R8-Pad2)
- U2 pad 8: Net-(R11-Pad2) -> Net-(JP9-Pad2)
- U2 pad 9: Net-(R9-Pad2) -> Net-(R15-Pad2)
Routing:
- net Net-(R9-Pad2): track 0.00 -> 23.2 mm
- net Net-(R8-Pad2): track 0.00 -> 18.9 mm
- net Net-(R11-Pad2): track 0.00 -> 18.5 mm
- net Net-(R15-Pad2): track 0.00 -> 13.7 mm
- net Net-(R13-Pad2): track 0.00 -> 13.6 mm
- net Net-(R16-Pad2): track 0.00 -> 8.67 mm
- net Net-(R14-Pad2): track 0.00 -> 8.58 mm
- net Net-(JP9-Pad2): track 0.00 -> 8.23 mm
