File: KiCAD files/myDAQExpansionBoard_v1/myDAQExpansionBoard.kicad_sch (KiCad schematic)
At the start: 64 parts, among them J1 OSTV7XX3151, J2 Conn_01x05_Male, J3 Conn_01x05_Male, J4 Screw_Terminal_01x02, J5 Screw_Terminal_01x02, J6 Screw_Terminal_01x02, J7 Conn_01x08_Male, J8 Screw_Terminal_01x02, J9 Screw_Terminal_01x02, SW1 SW_Push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

Commit message: v2
Parts:
- removed J9: Screw_Terminal_01x02, Connector_PinHeader_2.54mm:PinHeader_1x02_P2.54mm_Vertical, symbol Connector:Screw_Terminal_01x02
- removed SW3, SW4: SW_SPST, Button_Switch_THT:SW_DIP_SPSTx01_Slide_9.78x4.72mm_W7.62mm_P2.54mm, symbol Switch:SW_SPST
- added CD1, CD2: 100n, Capacitor_SMD:C_0603_1608Metric, symbol Device:C
- added SW3, SW4: SW_SPDT, Library:we01014042, symbol Switch:SW_SPDT
- R18: footprint OptoDevice:R_LDR_7x6mm_P5.1mm_Vertical -> OptoDevice:R_LDR_5.1x4.3mm_P3.4mm_Vertical
Connections:
- net +5V: now also SW3.1 (A), SW4.1 (A); no longer JP3.2 (B), JP4.2 (B)
- net DIO4: now also CD1.1
- net DIO5: now also CD2.1
- net DIO6: now also JP3.2 (B); no longer R4.2
- net DIO7: now also JP4.2 (B); no longer R6.2
- net GND: now also J5.1 (Pin_1), J5.2 (Pin_2), U3.3 (IP-), U3.4 (IP-), CD1.2, CD2.2, SW3.3 (C), SW4.3 (C)
- net at JP3.1 (A): now also R4.2; no longer R4.1
- new net: R4.1, SW3.2 (B)
- new net: R6.2, SW4.2 (B)
Other:
- note added: "TO-DO: - smanjiti silkscreen konektora za stepper - dioda za reverse polarity protection - ne treba odvojiti gnd, samo udaljiti analogni od digitalnog dijela - sklopka: dolje napajanje gore GND - ukrasiti legendu korisnim informacijama i oblicima - provjeriti cijelu shemu - tvz logo, jk logo, JLCJLCJLCJLC, gmail adresa - na pločici zaljepiti kaptoj traku ispod shunta DONE: - 2 tipkala i pritezni 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"
- note removed: "TO-DO: - debounce kondenzatori na tipkalima i možda sklopkama - odvojiti analogni i digitalni gnd - spst sklopke zamijeniti footprinte DONE: - 2 tipkala i pritezni otpornici (2 jumpera za pull up) - DIO 4,5 - 2 sklopke i pritezni otpornici (2 jumpera za pull up) - DIO 6,7 - 4 LEDice - DIO 0,1,2,3 - IC za 7.segm zaslon - DIO 0,1,2 - LDR - AIO - LM35 - AI1 - shunt i priključnice - acs712, AI0 - L29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"
- moved on the sheet: JP3, JP4, R4, R6, SW1, SW2
