File: KiCAD files/myDAQExpansionBoard_v2/myDAQExpansionBoard.kicad_pcb (KiCad board)
At the start: 2 copper layers, 100 x 100 mm, 65 parts, among them J1 OSTV7XX3151, J2 Conn_01x05_Male, J3 Conn_01x05_Male, J4 Screw_Terminal_01x02, J5 Screw_Terminal_01x02, J6 Screw_Terminal_01x02, J7 Conn_01x08_Male, J8 Screw_Terminal_01x02, SW1 SW_Push, SW2 SW_Push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

Commit message: update
Parts:
- removed JP12, JP13: Jumper_3_Open, Connector_PinHeader_2.54mm:PinHeader_1x03_P2.54mm_Vertical
- removed JP15, JP6, JP7, JP8: Jumper_2_Open, Connector_PinHeader_2.54mm:PinHeader_1x02_P2.54mm_Vertical
- added R20: 10k, Resistor_SMD:R_0603_1608Metric, F.Cu at (119.2, 112.8)
- added R21: 10k, Resistor_SMD:R_0603_1608Metric, F.Cu at (109.2, 90.5)
- JP14: value Jumper_2_Open -> Jumper_3_Open; footprint Connector_PinHeader_2.54mm:PinHeader_1x02_P2.54mm_Vertical -> Connector_PinHeader_2.54mm:PinHeader_1x03_P2.54mm_Vertical
- moved JP14 28.6 mm to (113.7, 85.8), turned to 90 degrees
- moved JP5 24.8 mm to (80.8, 127.0), turned to 180 degrees
- moved J5 9.70 mm to (129.0, 68.0)
- moved J8 9.70 mm to (129.0, 77.8)
- moved D1 9.34 mm to (50.8, 133.3)
- moved D2 9.34 mm to (58.8, 133.3)
- moved D3 9.34 mm to (66.8, 133.3)
- moved D4 9.34 mm to (74.8, 133.3)
- moved R1 7.60 mm to (50.8, 139.0)
- moved R10 7.60 mm to (74.8, 139.0)
- moved R5 7.60 mm to (58.8, 139.0)
- moved R7 7.60 mm to (66.8, 139.0)
- moved JP9 0.80 mm to (81.6, 85.8)
- moved C1 0.35 mm to (64.7, 99.5)
- moved U1 0.35 mm to (60.9, 90.6)
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Connections:
- D1 pad 1: GND -> Net-(R1-Pad1)
- D1 pad 2: Net-(D1-Pad2) -> DIO0
- D2 pad 1: GND -> Net-(D2-Pad1)
- D2 pad 2: Net-(D2-Pad2) -> DIO1
- D3 pad 1: GND -> Net-(D3-Pad1)
- D3 pad 2: Net-(D3-Pad2) -> DIO2
- D4 pad 1: GND -> Net-(R10-Pad1)
- D4 pad 2: Net-(D4-Pad2) -> DIO3
- JP14 pad 1: Net-(J8-Pad1) -> SHUNT
- JP14 pad 2: SHUNT -> Net-(J8-Pad1)
- JP5 pad 1: DIO0 -> Net-(JP5-Pad1)
- JP5 pad 2: Net-(JP5-Pad2) -> GND
- R1 pad 1: Net-(JP5-Pad2) -> Net-(R1-Pad1)
- R1 pad 2: Net-(D1-Pad2) -> Net-(JP5-Pad1)
- R10 pad 1: Net-(JP8-Pad2) -> Net-(R10-Pad1)
- R10 pad 2: Net-(D4-Pad2) -> Net-(JP5-Pad1)
- R5 pad 1: Net-(JP6-Pad2) -> Net-(D2-Pad1)
- R5 pad 2: Net-(D2-Pad2) -> Net-(JP5-Pad1)
- R7 pad 1: Net-(JP7-Pad2) -> Net-(D3-Pad1)
- R7 pad 2: Net-(D3-Pad2) -> Net-(JP5-Pad1)
Other:
- board text added: "H-MOST"
- board text added: "SHUNT"
