File: KiCAD files/myDAQExpansionBoard_v2/myDAQExpansionBoard.kicad_sch (KiCad schematic)
At the start: 65 parts, among them J1 OSTV7XX3151, J2 Conn_01x05_Male, J3 Conn_01x05_Male, J4 Screw_Terminal_01x02, J5 Screw_Terminal_01x02, J6 Screw_Terminal_01x02, J7 Conn_01x08_Male, J8 Screw_Terminal_01x02, SW1 SW_Push, SW2 SW_Push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

Commit message: update
Parts:
- removed JP12, JP13: Jumper_3_Open, Connector_PinHeader_2.54mm:PinHeader_1x03_P2.54mm_Vertical, symbol Jumper:Jumper_3_Open
- removed JP14, JP15, JP6, JP7, JP8: Jumper_2_Open, Connector_PinHeader_2.54mm:PinHeader_1x02_P2.54mm_Vertical, symbol Jumper:Jumper_2_Open
- added JP14: Jumper_3_Open, Connector_PinHeader_2.54mm:PinHeader_1x03_P2.54mm_Vertical, symbol Jumper:Jumper_3_Open
- added R20, R21: 10k, Resistor_SMD:R_0603_1608Metric, symbol Device:R
Connections:
- net +5V: now also R20.1, R21.1
- net DIO0: now also D1.2 (A); no longer JP5.1 (A)
- net DIO1: now also D2.2 (A)
- net DIO2: now also D3.2 (A)
- net DIO3: now also D4.2 (A)
- net GND: now also JP5.2 (B); no longer D1.1 (K), D2.1 (K), D3.1 (K), D4.1 (K)
- net SHUNT: now also JP14.1 (A)
- net VDD: now also JP14.3 (B)
- net at R7.1: now also D3.1 (K)
- net at R7.2: now also JP5.1 (A), R1.2, R10.2, R5.2; no longer D3.2 (A)
- net at U5.1 (EN1,2): now also R20.2
- net at U5.9 (EN3,4): now also R21.2
- net at R10.1: now also D4.1 (K)
- net at J8.1 (Pin_1), J8.2 (Pin_2): now also JP14.2 (C)
- net at R1.1: now also D1.1 (K); no longer JP5.2 (B)
- net at R5.1: now also D2.1 (K)
Other:
- note added: "TO-DO: - - smanjiti silkscreen konektora za stepper - da li je redosljed izlaza hmosta dobar? - dioda za reverse polarity protection - ne treba odvojiti gnd, samo udaljiti analogni od digitalnog dijela - sklopka: dolje napajanje gore GND - ukrasiti legendu korisnim informacijama i oblicima - provjeriti cijelu shemu - tvz logo, jk logo, JLCJLCJLCJLC, gmail adresa - na pločici zaljepiti kaptoj trak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"
- note removed: "TO-DO: - smanjiti silkscreen konektora za stepper - da li je redosljed izlaza hmosta dobar? - dioda za reverse polarity protection - ne treba odvojiti gnd, samo udaljiti analogni od digitalnog dijela - sklopka: dolje napajanje gore GND - ukrasiti legendu korisnim informacijama i oblicima - provjeriti cijelu shemu - tvz logo, jk logo, JLCJLCJLCJLC, gmail adresa - na pločici zaljepiti kaptoj traku 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"
- moved on the sheet: D1, D2, D3, D4, J8, JP5, R1, R10, R5, R7

Commit message: Update myDAQExpansionBoard.kicad_sch
Other:
- note added: "TO-DO: - potenciometar - smanjiti silkscreen konektora za stepper - da li je redosljed izlaza hmosta dobar? - dioda za reverse polarity protection - ne treba odvojiti gnd, samo udaljiti analogni od digitalnog dijela - sklopka: dolje napajanje gore GND - ukrasiti legendu korisnim informacijama i oblicima - provjeriti cijelu shemu - tvz logo, jk logo, JLCJLCJLCJLC, gmail adresa - na pločici zaljepi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"
- note removed: "TO-DO: - - smanjiti silkscreen konektora za stepper - da li je redosljed izlaza hmosta dobar? - dioda za reverse polarity protection - ne treba odvojiti gnd, samo udaljiti analogni od digitalnog dijela - sklopka: dolje napajanje gore GND - ukrasiti legendu korisnim informacijama i oblicima - provjeriti cijelu shemu - tvz logo, jk logo, JLCJLCJLCJLC, gmail adresa - na pločici zaljepiti kaptoj trak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"
Changed lines of the file:
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@@
+    (stroke (width 0) (type default) (color 0 0 0 0))
+  )
+  (polyline (pts (xy 233.68 15.875) (xy 255.27 15.875))
     (stroke (width 0) (type default) (color 0 0 0 0))
   )
@@
     (stroke (width 0) (type default) (color 0 0 0 0))
   )
+  (polyline (pts (xy 255.27 15.875) (xy 255.27 19.05))
+    (stroke (width 0) (type default) (color 0 0 0 0))
+  )
   (wire (pts (xy 130.175 74.295) (xy 130.175 70.485))
     (stroke (width 0) (type default) (color 0 0 0 0))
   )
+  (polyline (pts (xy 255.27 80.01) (xy 255.27 79.375))
+    (stroke (width 0) (type default) (color 0 0 0 0))
+  )
   (wire (pts (xy 112.395 71.755) (xy 109.22 71.755))
     (stroke (width 0) (type default) (color 0 0 0 0))
@@
     (stroke (width 0) (type default) (color 0 0 0 0))
   )
+  (polyline (pts (xy 233.68 80.01) (xy 255.27 80.01))
+    (stroke (width 0) (type default) (color 0 0 0 0))
+  )
   (wire (pts (xy 236.22 41.275) (xy 236.22 25.4))
     (stroke (width 0) (type default) (color 0 0 0 0))
@@
     (stroke (width 0) (type default) (color 0 0 0 0))
   )
-  (text "TO-DO:\n- \n- smanjiti silkscreen konektora za stepper\n- da li je redosljed izlaza hmosta dobar?\n- dioda za reverse polarity protection\n- ne treba odvojiti gnd, samo udaljiti analogni od digitalnog dijela\n- sklopka: dolje napajanje gore GND\n- ukrasiti legendu korisnim informacijama i oblicima\n- provjeriti cijelu shemu\n- tvz logo, jk logo, JLCJLCJLCJLC, gmail adresa\n- na pločici zaljepiti kaptoj traku ispod shunta\n\nDONE:\n- 2 tipkala i pritezni otpornici (2 jumpera za pull up) - DIO 4,5\n- 2 sklopke i pritezni otpornici (2 jumpera za pull up) - DIO 6,7\n- 4 LEDice - DIO 0,1,2,3\n- IC za 7.segm zaslon - DIO 0,1,2\n- LDR - AIO\n- LM35 - AI1\n- shunt i priključnice\n- acs712, AI0\n- L293D 4 digitalna izlaza, DIP s profi podnožjem\n- staviti 1x05 strip za GND\n- staviti 1x05 strip za +5V"
+  (text "TO-DO:\n- potenciometar\n- smanjiti silkscreen konektora za stepper\n- da li je redosljed izlaza hmosta dobar?\n- dioda za reverse polarity protection\n- ne treba odvojiti gnd, samo udaljiti analogni od digitalnog dijela\n- sklopka: dolje napajanje gore GND\n- ukrasiti legendu korisnim informacijama i oblicima\n- provjeriti cijelu shemu\n- tvz logo, jk logo, JLCJLCJLCJLC, gmail adresa\n- na pločici zaljepiti kaptoj traku ispod shunta\n\nDONE:\n- 2 tipkala i pritezni otpornici (2 jumpera za pull up) - DIO 4,5\n- 2 sklopke i pritezni otpornici (2 jumpera za pull up) - DIO 6,7\n- 4 LEDice - DIO 0,1,2,3\n- IC za 7.segm zaslon - DIO 0,1,2\n- LDR - AIO\n- LM35 - AI1\n- shunt i priključnice\n- acs712, AI0\n- L293D 4 digitalna izlaza, DIP s profi podnožjem\n- staviti 1x05 strip za GND\n- staviti 1x05 strip za +5V"
     (at 302.26 94.615 0)
     (effects (font (size 1.27 1.27)) (justify left bottom))
