File: KiCAD files/myDAQExpansionBoard_v3/myDAQExpansionBoard.kicad_sch (KiCad schematic)
At the start: 61 parts, among them J1 OSTV7XX3151, J2 Conn_01x05_Male, J3 Conn_01x05_Male, J4 Screw_Terminal_01x02, J5 Screw_Terminal_01x01, J6 Screw_Terminal_01x02, J7 Conn_01x08_Male, J8 Screw_Terminal_01x01, SW1 SW_Push, SW2 SW_Push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

Commit message: update
Parts:
- added JP12, JP13: Jumper_3_Open, Connector_PinHeader_2.54mm:PinHeader_1x03_P2.54mm_Vertical, symbol Jumper:Jumper_3_Open
Connections:
- net +5V: now also JP12.3 (B), JP13.3 (B); no longer R20.1, R21.1
- net GND: now also JP12.1 (A), JP13.1 (A)
- new net: JP12.2 (C), R20.1
- new net: JP13.2 (C), R21.1
Changed lines of the file:
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@@
   (junction (at 165.1 125.73) (diameter 0) (color 0 0 0 0)
-  )
-  (junction (at 31.75 130.81) (diameter 0) (color 0 0 0 0)
   )
   (junction (at 236.22 41.275) (diameter 0) (color 0 0 0 0)
@@
     (stroke (width 0) (type default) (color 0 0 0 0))
   )
-  (wire (pts (xy 31.75 124.46) (xy 31.75 130.81))
-    (stroke (width 0) (type default) (color 0 0 0 0))
-  )
   (polyline (pts (xy 220.345 109.855) (xy 223.52 109.855))
     (stroke (width 0) (type default) (color 0 0 0 0))
@@
     (stroke (width 0) (type default) (color 0 0 0 0))
   )
-  (wire (pts (xy 34.29 146.05) (xy 31.75 146.05))
-    (stroke (width 0) (type default) (color 0 0 0 0))
-  )
   (wire (pts (xy 41.91 146.05) (xy 46.355 146.05))
     (stroke (width 0) (type default) (color 0 0 0 0))
@@
     (stroke (width 0) (type default) (color 0 0 0 0))
   )
-  (wire (pts (xy 31.75 130.81) (xy 31.75 146.05))
-    (stroke (width 0) (type default) (color 0 0 0 0))
-  )
   (wire (pts (xy 248.92 112.395) (xy 248.92 114.3))
     (stroke (width 0) (type default) (color 0 0 0 0))
@@
     (stroke (width 0) (type default) (color 0 0 0 0))
   )
-  (wire (pts (xy 33.655 130.81) (xy 31.75 130.81))
-    (stroke (width 0) (type default) (color 0 0 0 0))
-  )
   (wire (pts (xy 135.89 81.915) (xy 128.905 81.915))
     (stroke (width 0) (type default) (color 0 0 0 0))
@@
   )
   (polyline (pts (xy 51.435 15.875) (xy 51.435 57.15))
+    (stroke (width 0) (type default) (color 0 0 0 0))
+  )
+  (wire (pts (xy 28.575 146.05) (xy 34.29 146.05))
     (stroke (width 0) (type default) (color 0 0 0 0))
   )
@@
     (pin "1")
   )
+  (symbol (lib_id "power:+5V") (at 24.765 139.7 0) (unit 1)
+    (in_bom yes) (on_board yes)
+    (property "Reference" "#PWR?" (id 0) (at 24.765 143.51 0)
+      (effects (font (size 1.27 1.27)) hide)
+    )
+    (property "Value" "+5V" (id 1) (at 24.765 136.1242 0))
+    (property "Footprint" "" (id 2) (at 24.765 139.7 0)
+      (effects (font (size 1.27 1.27)) hide)
+    )
+    (property "Datasheet" "" (id 3) (at 24.765 139.7 0)
+      (effects (font (size 1.27 1.27)) hide)
+    )
+    (pin "1")
+  )
   (symbol (lib_id "Device:C") (at 108.585 40.64 90) (unit 1)
     (in_bom yes) (on_board yes) (fields_autoplaced)
@@
     (pin "1")
   )
-  (symbol (lib_id "power:+5V") (at 31.75 124.46 0) (unit 1)
-    (in_bom yes) (on_board yes)
-    (property "Reference" "#PWR033" (id 0) (at 31.75 128.27 0)
-      (effects (font (size 1.27 1.27)) hide)
-    )
-    (property "Value" "+5V" (id 1) (at 31.75 120.8842 0))
-    (property "Footprint" "" (id 2) (at 31.75 124.46 0)
-      (effects (font (size 1.27 1.27)) hide)
-    )
-    (property "Datasheet" "" (id 3) (at 31.75 124.46 0)
+  (symbol (lib_id "power:+5V") (at 29.845 124.46 0) (unit 1)
+    (in_bom yes) (on_board yes)
+    (property "Reference" "#PWR033" (id 0) (at 29.845 128.27 0)
+      (effects (font (size 1.27 1.27)) hide)
+    )
+    (property "Value" "+5V" (id 1) (at 29.845 120.8842 0))
+    (property "Footprint" "" (id 2) (at 29.845 124.46 0)
+      (effects (font (size 1.27 1.27)) hide)
+    )
+    (property "Datasheet" "" (id 3) (at 29.845 124.46 0)
       (effects (font (size 1.27 1.27)) hide)
     )
@@
     (pin "2")
   )
+  (symbol (lib_id "Jumper:Jumper_3_Open") (at 24.765 146.05 90) (unit 1)
+    (in_bom yes) (on_board yes) (fields_autoplaced)
+    (property "Reference" "JP13" (id 0) (at 22.6309 146.4838 90)
+      (effects (font (size 1.27 1.27)) (justify left))
+    )
+    (property "Value" "Jumper_3_Open" (id 1) (at 22.6308 144.3478 90)
+      (effects (font (size 1.27 1.27)) (justify left) hide)
+    )
+    (property "Footprint" "Connector_PinHeader_2.54mm:PinHeader_1x03_P2.54mm_Vertical" (id 2) (at 24.765 146.05 0)
+      (effects (font (size 1.27 1.27)) hide)
+    )
+    (property "Datasheet" "~" (id 3) (at 24.765 146.05 0)
+      (effects (font (size 1.27 1.27)) hide)
+    )
+    (pin "1")
+    (pin "2")
+    (pin "3")
+  )
   (symbol (lib_id "power:+5V") (at 96.52 64.135 0) (unit 1)
     (in_bom yes) (on_board yes)
@@
     )
     (pin "1")
+  )
+  (symbol (lib_id "Jumper:Jumper_3_Open") (at 29.845 130.81 90) (unit 1)
+    (in_bom yes) (on_board yes) (fields_autoplaced)
+    (property "Reference" "JP12" (id 0) (at 27.7109 131.2438 90)
+      (effects (font (size 1.27 1.27)) (justify left))
+    )
+    (property "Value" "Jumper_3_Open" (id 1) (at 27.7108 129.1078 90)
+      (effects (font (size 1.27 1.27)) (justify left) hide)
+    )
+    (property "Footprint" "Connector_PinHeader_2.54mm:PinHeader_1x03_P2.54mm_Vertical" (id 2) (at 29.845 130.81 0)
+      (effects (font (size 1.27 1.27)) hide)
+    )
+    (property "Datasheet" "~" (id 3) (at 29.845 130.81 0)
+      (effects (font (size 1.27 1.27)) hide)
+    )
+    (pin "1")
+    (pin "2")
+    (pin "3")
   )
   (symbol (lib_id "power:GNDA") (at 99.06 124.46 0) (unit 1)
@@
     (pin "1")
   )
+  (symbol (lib_id "power:GND") (at 29.845 137.16 0) (unit 1)
+    (in_bom yes) (on_board yes) (fields_autoplaced)
+    (property "Reference" "#PWR?" (id 0) (at 29.845 143.51 0)
+      (effects (font (size 1.27 1.27)) hide)
+    )
+    (property "Value" "GND" (id 1) (at 29.845 141.6034 0))
+    (property "Footprint" "" (id 2) (at 29.845 137.16 0)
+      (effects (font (size 1.27 1.27)) hide)
+    )
+    (property "Datasheet" "" (id 3) (at 29.845 137.16 0)
+      (effects (font (size 1.27 1.27)) hide)
+    )
+    (pin "1")
+  )
   (symbol (lib_id "power:+5V") (at 59.69 74.93 0) (unit 1)
     (in_bom yes) (on_board yes)
@@
     (pin "1")
     (pin "2")
+  )
+  (symbol (lib_id "power:GND") (at 24.765 152.4 0) (unit 1)
+    (in_bom yes) (on_board yes) (fields_autoplaced)
+    (property "Reference" "#PWR?" (id 0) (at 24.765 158.75 0)
+      (effects (font (size 1.27 1.27)) hide)
+    )
+    (property "Value" "GND" (id 1) (at 24.765 156.8434 0))
+    (property "Footprint" "" (id 2) (at 24.765 152.4 0)
+      (effects (font (size 1.27 1.27)) hide)
+    )
+    (property "Datasheet" "" (id 3) (at 24.765 152.4 0)
+      (effects (font (size 1.27 1.27)) hide)
+    )
+    (pin "1")
   )
   (symbol (lib_id "Device:C") (at 99.06 120.65 0) (unit 1)
@@
       (reference "#PWR0110") (unit 1) (value "GND") (footprint "")
     )
+    (path "/1dcaaf7b-499f-437f-b40c-1ef3977acf50"
+      (reference "#PWR?") (unit 1) (value "+5V") (footprint "")
+    )
+    (path "/9d81ffb6-e253-43e0-84ea-c0744f106382"
+      (reference "#PWR?") (unit 1) (value "GND") (footprint "")
+    )
+    (path "/d4eaed5e-655a-475b-9755-7e9e76c62d55"
+      (reference "#PWR?") (unit 1) (value "GND") (footprint "")
+    )
     (path "/e46c1870-2749-4db8-bfa0-503edc656da7"
       (reference "C1") (unit 1) (value "100n") (footprint "Capacitor_SMD:C_0603_1608Metric")
@@
       (reference "JP11") (unit 1) (value "Jumper_3_Open") (footprint "Connector_PinHeader_2.54mm:PinHeader_1x03_P2.54mm_Vertical")
     )
+    (path "/75a47c1d-830a-4762-aac4-0388ee52ab05"
+      (reference "JP12") (unit 1) (value "Jumper_3_Open") (footprint "Connector_PinHeader_2.54mm:PinHeader_1x03_P2.54mm_Vertical")
+    )
+    (path "/6b52dbbc-5e9d-4d8b-a422-cd9eb7174b37"
+      (reference "JP13") (unit 1) (value "Jumper_3_Open") (footprint "Connector_PinHeader_2.54mm:PinHeader_1x03_P2.54mm_Vertical")
+    )
     (path "/71a1d96c-b1e9-4037-8a91-ce24442bb1fd"

Commit message: update
Connections:
- net +5V: now also JP12.1 (A); no longer JP12.3 (B)
- net GND: now also JP12.3 (B); no longer JP12.1 (A)
- net at U2.3 (CA/CC): now also JP9.2 (C)
- net at U2.8 (CA/CC): no longer JP9.2 (C)
Changed lines of the file:
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@@
   (junction (at 43.815 68.58) (diameter 0) (color 0 0 0 0)
   )
-  (no_connect (at 151.13 92.075))
   (no_connect (at 185.42 153.035))
   (no_connect (at 135.89 89.535))
@@
   (no_connect (at 31.75 91.44))
   (no_connect (at 185.42 160.02))
+  (no_connect (at 151.13 94.615))
   (no_connect (at 161.925 153.035))
   (no_connect (at 161.925 160.02))
@@
     (stroke (width 0) (type default) (color 0 0 0 0))
   )
-  (wire (pts (xy 152.4 94.615) (xy 151.13 94.615))
-    (stroke (width 0) (type default) (color 0 0 0 0))
-  )
   (wire (pts (xy 116.205 81.915) (xy 109.22 81.915))
     (stroke (width 0) (type default) (color 0 0 0 0))
@@
     (stroke (width 0) (type default) (color 0 0 0 0))
   )
-  (wire (pts (xy 152.4 83.185) (xy 152.4 94.615))
+  (wire (pts (xy 152.4 83.185) (xy 152.4 92.075))
     (stroke (width 0) (type default) (color 0 0 0 0))
   )
@@
   )
   (wire (pts (xy 173.355 43.815) (xy 173.355 41.91))
+    (stroke (width 0) (type default) (color 0 0 0 0))
+  )
+  (wire (pts (xy 151.13 92.075) (xy 152.4 92.075))
     (stroke (width 0) (type default) (color 0 0 0 0))
   )
@@
   (symbol (lib_id "power:+5V") (at 24.765 139.7 0) (unit 1)
     (in_bom yes) (on_board yes)
-    (property "Reference" "#PWR?" (id 0) (at 24.765 143.51 0)
+    (property "Reference" "#PWR0111" (id 0) (at 24.765 143.51 0)
       (effects (font (size 1.27 1.27)) hide)
     )
@@
     (pin "1")
   )
-  (symbol (lib_id "Jumper:Jumper_3_Open") (at 29.845 130.81 90) (unit 1)
+  (symbol (lib_id "Jumper:Jumper_3_Open") (at 29.845 130.81 90) (mirror x) (unit 1)
     (in_bom yes) (on_board yes) (fields_autoplaced)
     (property "Reference" "JP12" (id 0) (at 27.7109 131.2438 90)
       (effects (font (size 1.27 1.27)) (justify left))
     )
-    (property "Value" "Jumper_3_Open" (id 1) (at 27.7108 129.1078 90)
+    (property "Value" "Jumper_3_Open" (id 1) (at 27.7108 132.5122 90)
       (effects (font (size 1.27 1.27)) (justify left) hide)
     )
@@
   (symbol (lib_id "power:GND") (at 29.845 137.16 0) (unit 1)
     (in_bom yes) (on_board yes) (fields_autoplaced)
-    (property "Reference" "#PWR?" (id 0) (at 29.845 143.51 0)
+    (property "Reference" "#PWR0112" (id 0) (at 29.845 143.51 0)
       (effects (font (size 1.27 1.27)) hide)
     )
@@
   (symbol (lib_id "power:GND") (at 24.765 152.4 0) (unit 1)
     (in_bom yes) (on_board yes) (fields_autoplaced)
-    (property "Reference" "#PWR?" (id 0) (at 24.765 158.75 0)
+    (property "Reference" "#PWR0113" (id 0) (at 24.765 158.75 0)
       (effects (font (size 1.27 1.27)) hide)
     )
@@
     )
     (path "/1dcaaf7b-499f-437f-b40c-1ef3977acf50"
-      (reference "#PWR?") (unit 1) (value "+5V") (footprint "")
+      (reference "#PWR0111") (unit 1) (value "+5V") (footprint "")
     )
     (path "/9d81ffb6-e253-43e0-84ea-c0744f106382"
-      (reference "#PWR?") (unit 1) (value "GND") (footprint "")
+      (reference "#PWR0112") (unit 1) (value "GND") (footprint "")
     )
     (path "/d4eaed5e-655a-475b-9755-7e9e76c62d55"
-      (reference "#PWR?") (unit 1) (value "GND") (footprint "")
+      (reference "#PWR0113") (unit 1) (value "GND") (footprint "")
     )
     (path "/e46c1870-2749-4db8-bfa0-503edc656da7"

Commit message: update
Parts:
- removed D4: LED, LED_THT:LED_D5.0mm, symbol Device:LED
- removed R10: 1k, Resistor_SMD:R_0603_1608Metric, symbol Device:R
- H1, H2, H3, H4: footprint MountingHole:MountingHole_3.2mm_M3_Pad_Via -> MountingHole:MountingHole_3.2mm_M3; symbol Mechanical:MountingHole_Pad -> Mechanical:MountingHole
Connections:
- net AI0+: now also JP11.2 (C); no longer JP10.2 (C)
- net AI1+: now also JP10.2 (C); no longer JP11.2 (C)
- no-connect marks 9 -> 5
Changed lines of the file:
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@@
   (junction (at 81.915 48.895) (diameter 0) (color 0 0 0 0)
   )
-  (junction (at 236.22 54.61) (diameter 0) (color 0 0 0 0)
-  )
   (junction (at 102.235 48.895) (diameter 0) (color 0 0 0 0)
   )
@@
   (junction (at 43.815 68.58) (diameter 0) (color 0 0 0 0)
   )
-  (no_connect (at 185.42 153.035))
   (no_connect (at 135.89 89.535))
   (no_connect (at 31.75 88.9))
   (no_connect (at 31.75 81.28))
   (no_connect (at 31.75 91.44))
-  (no_connect (at 185.42 160.02))
   (no_connect (at 151.13 94.615))
-  (no_connect (at 161.925 153.035))
-  (no_connect (at 161.925 160.02))
   (wire (pts (xy 43.815 86.36) (xy 43.815 78.74))
     (stroke (width 0) (type default) (color 0 0 0 0))
@@
     (stroke (width 0) (type default) (color 0 0 0 0))
   )
-  (wire (pts (xy 206.375 70.485) (xy 212.725 70.485))
-    (stroke (width 0) (type default) (color 0 0 0 0))
-  )
   (wire (pts (xy 73.025 125.73) (xy 73.025 124.46))
     (stroke (width 0) (type default) (color 0 0 0 0))
@@
     (stroke (width 0) (type default) (color 0 0 0 0))
   )
-  (wire (pts (xy 236.22 54.61) (xy 236.22 70.485))
-    (stroke (width 0) (type default) (color 0 0 0 0))
-  )
   (wire (pts (xy 248.92 124.46) (xy 247.015 124.46))
     (stroke (width 0) (type default) (color 0 0 0 0))
@@
   )
   (polyline (pts (xy 159.385 109.855) (xy 159.385 110.49))
-    (stroke (width 0) (type default) (color 0 0 0 0))
-  )
-  (wire (pts (xy 236.22 70.485) (xy 227.965 70.485))
     (stroke (width 0) (type default) (color 0 0 0 0))
   )
@@
     )
   )
-  (global_label "AI0+" (shape input) (at 151.765 129.54 270) (fields_autoplaced)
+  (global_label "AI0+" (shape input) (at 210.185 129.54 270) (fields_autoplaced)
     (effects (font (size 1.27 1.27)) (justify right))
-    (property "Intersheet References" "${INTERSHEET_REFS}" (id 0) (at 151.8444 136.4283 90)
+    (property "Intersheet References" "${INTERSHEET_REFS}" (id 0) (at 210.2644 136.4283 90)
       (effects (font (size 1.27 1.27)) (justify right) hide)
     )
@@
     )
   )
-  (global_label "AI1+" (shape input) (at 210.185 129.54 270) (fields_autoplaced)
+  (global_label "AI1+" (shape input) (at 151.765 129.54 270) (fields_autoplaced)
     (effects (font (size 1.27 1.27)) (justify right))
-    (property "Intersheet References" "${INTERSHEET_REFS}" (id 0) (at 210.2644 136.4283 90)
+    (property "Intersheet References" "${INTERSHEET_REFS}" (id 0) (at 151.8444 136.4283 90)
       (effects (font (size 1.27 1.27)) (justify right) hide)
     )
@@
     (property "Intersheet References" "${INTERSHEET_REFS}" (id 0) (at 38.5779 50.7206 0)
       (effects (font (size 1.27 1.27)) (justify left) hide)
-    )
-  )
-  (global_label "DIO3" (shape input) (at 206.375 70.485 180) (fields_autoplaced)
-    (effects (font (size 1.27 1.27)) (justify right))
-    (property "Intersheet References" "${INTERSHEET_REFS}" (id 0) (at 199.5471 70.4056 0)
-      (effects (font (size 1.27 1.27)) (justify right) hide)
     )
   )
@@
     (pin "2")
   )
-  (symbol (lib_id "Mechanical:MountingHole_Pad") (at 161.925 150.495 0) (unit 1)
+  (symbol (lib_id "Mechanical:MountingHole") (at 161.925 150.495 0) (unit 1)
     (in_bom yes) (on_board yes) (fields_autoplaced)
     (property "Reference" "H1" (id 0) (at 164.465 148.3903 0)
@@
       (effects (font (size 1.27 1.27)) (justify left))
     )
-    (property "Footprint" "MountingHole:MountingHole_3.2mm_M3_Pad_Via" (id 2) (at 161.925 150.495 0)
+    (property "Footprint" "MountingHole:MountingHole_3.2mm_M3" (id 2) (at 161.925 150.495 0)
       (effects (font (size 1.27 1.27)) hide)
     )
@@
       (effects (font (size 1.27 1.27)) hide)
     )
-    (pin "1")
   )
   (symbol (lib_id "power:+5V") (at 24.765 139.7 0) (unit 1)
@@
     (pin "2")
   )
-  (symbol (lib_id "Mechanical:MountingHole_Pad") (at 185.42 157.48 0) (unit 1)
+  (symbol (lib_id "Mechanical:MountingHole") (at 185.42 157.48 0) (unit 1)
     (in_bom yes) (on_board yes) (fields_autoplaced)
     (property "Reference" "H4" (id 0) (at 187.96 155.3753 0)
@@
       (effects (font (size 1.27 1.27)) (justify left))
     )
-    (property "Footprint" "MountingHole:MountingHole_3.2mm_M3_Pad_Via" (id 2) (at 185.42 157.48 0)
+    (property "Footprint" "MountingHole:MountingHole_3.2mm_M3" (id 2) (at 185.42 157.48 0)
       (effects (font (size 1.27 1.27)) hide)
     )
@@
       (effects (font (size 1.27 1.27)) hide)
     )
-    (pin "1")
   )
   (symbol (lib_id "Connector:Screw_Terminal_01x01") (at 24.765 180.34 180) (unit 1)
@@
     (pin "2")
   )
-  (symbol (lib_id "Mechanical:MountingHole_Pad") (at 161.925 157.48 0) (unit 1)
+  (symbol (lib_id "Mechanical:MountingHole") (at 161.925 157.48 0) (unit 1)
     (in_bom yes) (on_board yes) (fields_autoplaced)
     (property "Reference" "H3" (id 0) (at 164.465 155.3753 0)
@@
       (effects (font (size 1.27 1.27)) (justify left))
     )
-    (property "Footprint" "MountingHole:MountingHole_3.2mm_M3_Pad_Via" (id 2) (at 161.925 157.48 0)
+    (property "Footprint" "MountingHole:MountingHole_3.2mm_M3" (id 2) (at 161.925 157.48 0)
       (effects (font (size 1.27 1.27)) hide)
     )
@@
       (effects (font (size 1.27 1.27)) hide)
     )
-    (pin "1")
   )
   (symbol (lib_id "power:GND") (at 109.855 135.89 0) (unit 1)
@@
     (pin "1")
   )
-  (symbol (lib_id "Mechanical:MountingHole_Pad") (at 185.42 150.495 0) (unit 1)
+  (symbol (lib_id "Mechanical:MountingHole") (at 185.42 150.495 0) (unit 1)
     (in_bom yes) (on_board yes) (fields_autoplaced)
     (property "Reference" "H2" (id 0) (at 187.96 148.3903 0)
@@
       (effects (font (size 1.27 1.27)) (justify left))
     )
-    (property "Footprint" "MountingHole:MountingHole_3.2mm_M3_Pad_Via" (id 2) (at 185.42 150.495 0)
+    (property "Footprint" "MountingHole:MountingHole_3.2mm_M3" (id 2) (at 185.42 150.495 0)
       (effects (font (size 1.27 1.27)) hide)
     )
@@
       (effects (font (size 1.27 1.27)) hide)
     )
-    (pin "1")
   )
   (symbol (lib_id "power:GND") (at 19.05 126.365 0) (unit 1)
@@
     (pin "2")
   )
-  (symbol (lib_id "Device:R") (at 224.155 70.485 90) (unit 1)
-    (in_bom yes) (on_board yes)
-    (property "Reference" "R10" (id 0) (at 224.155 67.945 90))
-    (property "Value" "1k" (id 1) (at 224.155 70.485 90))
-    (property "Footprint" "Resistor_SMD:R_0603_1608Metric" (id 2) (at 224.155 72.263 90)
-      (effects (font (size 1.27 1.27)) hide)
-    )
-    (property "Datasheet" "~" (id 3) (at 224.155 70.485 0)
-      (effects (font (size 1.27 1.27)) hide)
-    )
-    (pin "1")
-    (pin "2")
-  )
   (symbol (lib_id "Device:R") (at 38.1 146.05 90) (unit 1)
     (in_bom yes) (on_board yes)
@@
     )
     (pin "1")
-  )
-  (symbol (lib_id "Device:LED") (at 216.535 70.485 180) (unit 1)
-    (in_bom yes) (on_board yes) (fields_autoplaced)
-    (property "Reference" "D4" (id 0) (at 218.1225 64.6262 0))
-    (property "Value" "LED" (id 1) (at 218.1225 67.1631 0))
-    (property "Footprint" "LED_THT:LED_D5.0mm" (id 2) (at 216.535 70.485 0)
-      (effects (font (size 1.27 1.27)) hide)
-    )
-    (property "Datasheet" "~" (id 3) (at 216.535 70.485 0)
-      (effects (font (size 1.27 1.27)) hide)
-    )
-    (pin "1")
-    (pin "2")
   )
   (symbol (lib_id "power:PWR_FLAG") (at 19.685 33.655 180) (unit 1)
@@
       (reference "D3") (unit 1) (value "LED") (footprint "LED_THT:LED_D5.0mm")
     )
-    (path "/c5de237c-6442-4367-bab1-8253f80b454f"
-      (reference "D4") (unit 1) (value "LED") (footprint "LED_THT:LED_D5.0mm")
-    )
     (path "/1cca44a0-f6b1-45ce-91b2-a8d3ac47bb0c"
-      (reference "H1") (unit 1) (value "MountingHole_Pad") (footprint "MountingHole:MountingHole_3.2mm_M3_Pad_Via")
+      (reference "H1") (unit 1) (value "MountingHole_Pad") (footprint "MountingHole:MountingHole_3.2mm_M3")
     )
     (path "/85d41246-65ff-4aa3-8df5-d28654ae2f51"
-      (reference "H2") (unit 1) (value "MountingHole_Pad") (footprint "MountingHole:MountingHole_3.2mm_M3_Pad_Via")
+      (reference "H2") (unit 1) (value "MountingHole_Pad") (footprint "MountingHole:MountingHole_3.2mm_M3")
     )
     (path "/7ea3b829-301e-4a19-9e92-7f019c96a1b4"
-      (reference "H3") (unit 1) (value "MountingHole_Pad") (footprint "MountingHole:MountingHole_3.2mm_M3_Pad_Via")
+      (reference "H3") (unit 1) (value "MountingHole_Pad") (footprint "MountingHole:MountingHole_3.2mm_M3")
     )
     (path "/6a2f264b-bb2a-489d-9abf-1e8d435dbf88"
-      (reference "H4") (unit 1) (value "MountingHole_Pad") (footprint "MountingHole:MountingHole_3.2mm_M3_Pad_Via")
+      (reference "H4") (unit 1) (value "MountingHole_Pad") (footprint "MountingHole:MountingHole_3.2mm_M3")
     )
     (path "/921d393e-e4ce-4b23-a600-c2b05c546cab"
@@
       (reference "R9") (unit 1) (value "680") (footprint "Resistor_SMD:R_0603_1608Metric")
     )
-    (path "/b86f1d54-499d-48ef-bd66-0eabea12a5e8"
-      (reference "R10") (unit 1) (value "1k") (footprint "Resistor_SMD:R_0603_1608Metric")
-    )
     (path "/7212c595-395e-40b8-bda9-f190b9683d3b"
