File: KiCAD files/myDAQExpansionBoard_v3/myDAQExpansionBoard.kicad_pcb (KiCad board)
At the start: 2 copper layers, 100 x 100 mm, 61 parts, among them J1 OSTV7XX3151, J2 Conn_01x05_Male, J3 Conn_01x05_Male, J4 Screw_Terminal_01x02, J5 Screw_Terminal_01x01, J6 Screw_Terminal_01x02, J7 Conn_01x08_Male, J8 Screw_Terminal_01x01, SW1 SW_Push, SW2 SW_Push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

Commit message: update
Parts:
- added JP12: Jumper_3_Open, Connector_PinHeader_2.54mm:PinHeader_1x03_P2.54mm_Vertical, F.Cu at (81.0, 117.0)
- added JP13: Jumper_3_Open, Connector_PinHeader_2.54mm:PinHeader_1x03_P2.54mm_Vertical, F.Cu at (94.2, 148.0)
- moved J8 104.6 mm to (52.2, 148.8), turned to 0 degrees
- moved R5 101.9 mm to (136.2, 72.8)
- moved R1 100.1 mm to (125.8, 72.8)
- moved D2 95.1 mm to (132.0, 72.8), turned to 180 degrees
- moved R17 94.7 mm to (49.0, 139.8), turned to 90 degrees
- moved D1 93.3 mm to (121.8, 72.8), turned to 180 degrees
- moved R10 83.9 mm to (136.2, 82.0)
- moved R7 82.2 mm to (125.8, 81.8)
- moved J4 79.8 mm to (70.3, 157.6), turned to 0 degrees
- moved J5 77.2 mm to (52.2, 59.8), turned to 0 degrees
- moved D4 76.9 mm to (132.0, 82.0), turned to 180 degrees
- moved D3 75.0 mm to (121.5, 82.0), turned to 180 degrees
- moved J6 73.3 mm to (89.5, 157.6), turned to 0 degrees
- moved JP14 70.3 mm to (65.2, 136.7), turned to 0 degrees
- moved JP5 64.1 mm to (132.8, 89.5), turned to -90 degrees
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Connections:
- R20 pad 1: +5V -> Net-(R20-Pad1)
- R21 pad 1: +5V -> Net-(R21-Pad1)
Routing:
- net +5V: track 0.00 -> 275.6 mm
- net DIO3: track 0.00 -> 167.7 mm, vias 0 -> 2
- net DIO0: track 0.00 -> 148.3 mm, vias 0 -> 4
- net DIO5: track 0.00 -> 115.8 mm
- net DIO4: track 0.00 -> 109.4 mm
- net DIO1: track 0.00 -> 91.7 mm, vias 0 -> 2
- net DIO2: track 0.00 -> 87.7 mm, vias 0 -> 2
- net Net-(JP11-Pad1): track 0.00 -> 65.6 mm
- net DIO7: track 0.00 -> 59.7 mm
- net DIO6: track 0.00 -> 51.8 mm
- net VDD: track 0.00 -> 51.2 mm
- net Net-(JP5-Pad1): track 0.00 -> 49.7 mm
- net Net-(J6-Pad2): track 0.00 -> 46.2 mm
- net Net-(J6-Pad1): track 0.00 -> 36.8 mm
- net Net-(J4-Pad1): track 0.00 -> 31.0 mm
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- added copper zone on F.Cu, net GND
Other:
- board size 100 x 100 mm -> 100 x 117.4 mm

Commit message: update_v3
Parts:
- moved C1 11.5 mm to (81.5, 86.6), turned to 90 degrees
- moved R12 4.70 mm to (69.3, 96.7)
Routing:
- net DIO1: track 91.7 -> 160.9 mm, vias 2 -> 5
- net DIO2: track 87.7 -> 132.9 mm, vias 2 -> 5
- net Net-(R12-Pad2): track 0.00 -> 7.30 mm
- net GND: track 13.7 -> 16.6 mm, vias 8 -> 10
- net unconnected-(J1-Pad1): track 0.00 -> 2.54 mm
- net +5V: track 275.6 -> 277.9 mm
- net Net-(R14-Pad2): track 7.02 -> 5.33 mm

Commit message: update
Parts:
- moved JP9 25.2 mm to (92.2, 107.7)
- moved R12 19.2 mm to (84.2, 108.8), turned to 180 degrees
- moved C1 2.27 mm to (80.0, 84.9), turned to 0 degrees
- moved C3 1.34 mm to (88.3, 125.6)
Connections:
- JP12 pad 1: GND -> +5V
- JP12 pad 3: +5V -> GND
- U2 pad 3: unconnected-(U2-Pad3) -> Net-(JP9-Pad2)
- U2 pad 8: Net-(JP9-Pad2) -> unconnected-(U2-Pad8)
Routing:
- net +5V: track 277.9 -> 357.3 mm
- net Net-(R12-Pad2): track 7.30 -> 25.4 mm
- net DIO3: track 167.7 -> 153.8 mm, vias 2 -> 3
- net Net-(JP9-Pad2): track 6.14 -> 3.86 mm

Commit message: update
Parts:
- removed D4: LED, LED_THT:LED_D5.0mm
- removed R10: 1k, Resistor_SMD:R_0603_1608Metric
- moved JP5 18.3 mm to (135.8, 71.5), turned to 0 degrees
- moved D2 10.1 mm to (124.8, 79.8)
- moved R5 8.89 mm to (130.8, 79.8), turned to 0 degrees
- moved R7 8.00 mm to (130.8, 88.0), turned to 0 degrees
- moved R6 7.75 mm to (128.5, 112.0), turned to 0 degrees
- moved D3 6.82 mm to (124.8, 88.0)
- moved R1 5.15 mm to (130.8, 71.5), turned to 0 degrees
- moved JP12 4.98 mm to (84.9, 120.1)
- moved R20 4.40 mm to (76.4, 125.6)
- moved JP9 3.95 mm to (96.0, 109.0)
- moved R11 3.75 mm to (88.0, 99.8)
- moved R12 3.75 mm to (88.0, 109.0)
- moved R13 3.75 mm to (88.0, 102.8)
- moved R14 3.75 mm to (88.0, 105.8)
- moved R15 3.75 mm to (88.0, 87.8)
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Connections:
- JP10 pad 2: AI0+ -> AI1+
- JP11 pad 2: AI1+ -> AI0+
Routing:
- net DIO1: track 160.9 -> 87.6 mm, vias 5 -> 4
- net DIO3: track 153.8 -> 80.5 mm, vias 3 -> 0
- net Net-(JP11-Pad1): track 65.6 -> 0.00 mm
- net VDD: track 51.2 -> 0.00 mm
- net Net-(J6-Pad2): track 46.2 -> 0.00 mm
- net DIO2: track 132.9 -> 93.8 mm, vias 5 -> 4
- net DIO0: track 148.3 -> 111.0 mm
- net Net-(J6-Pad1): track 36.8 -> 0.00 mm
- net Net-(J4-Pad1): track 31.0 -> 0.00 mm
- net Net-(JP5-Pad1): track 49.7 -> 20.7 mm
- net Net-(J8-Pad1): track 28.9 -> 0.00 mm
- net Net-(R17-Pad2): track 22.7 -> 0.00 mm
- net +5V: track 357.3 -> 334.7 mm
- net Net-(J4-Pad2): track 19.7 -> 0.00 mm
- net SHUNT: track 17.5 -> 0.00 mm
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- added copper zone on F.Cu, net +5V
Other:
- board text added: "LED1"
- board text added: "LED2"
- board text added: "LED3"

Commit message: update
Parts:
- added G***: LOGO, Library:logo, F.Cu at (116.1, 150.2)
- added G***: LOGO, Library:Labview-logo, F.Cu at (176.6, 150.2)
- H1, H2, H3, H4: footprint MountingHole:MountingHole_3.2mm_M3_Pad_Via -> MountingHole:MountingHole_3.2mm_M3
- moved C2 61.5 mm to (130.6, 56.2)
- moved C4 61.5 mm to (130.6, 60.2)
- moved U3 61.5 mm to (125.1, 58.8)
- moved C3 61.5 mm to (149.3, 117.6)
- moved J2 61.4 mm to (183.5, 50.4)
- moved J3 61.4 mm to (183.5, 54.1)
- moved J4 61.4 mm to (131.1, 149.5)
- moved J6 61.4 mm to (150.3, 149.5)
- moved JP10 61.4 mm to (142.3, 50.4)
- moved R11 61.4 mm to (148.8, 91.7)
- moved R12 61.4 mm to (148.8, 100.8)
- moved R13 61.4 mm to (148.8, 94.7)
- moved R14 61.4 mm to (148.8, 97.7)
- moved R15 61.4 mm to (148.8, 79.7)
- moved R16 61.4 mm to (148.8, 82.7)
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Routing:
- net +5V: track 334.7 -> 468.1 mm, vias 0 -> 7
- net DIO2: track 93.8 -> 167.1 mm, vias 4 -> 8
- net DIO1: track 87.6 -> 155.4 mm, vias 4 -> 5
- net Net-(JP11-Pad1): track 0.00 -> 64.0 mm, vias 0 -> 2
- net VDD: track 0.00 -> 62.9 mm
- net DIO3: track 80.5 -> 129.3 mm, vias 0 -> 2
- net Net-(J6-Pad2): track 0.00 -> 43.5 mm
- net DIO0: track 111.0 -> 147.1 mm
- net Net-(J6-Pad1): track 0.00 -> 36.0 mm
- net Net-(J8-Pad1): track 0.00 -> 33.9 mm
- net Net-(J4-Pad1): track 0.00 -> 32.4 mm
- net Net-(J4-Pad2): track 0.00 -> 20.7 mm
- net Net-(JP10-Pad1): track 0.00 -> 19.7 mm
- net SHUNT: track 0.00 -> 19.2 mm
- net Net-(JP12-Pad2): track 0.00 -> 9.36 mm
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- added copper zone on F.Cu, net Net-(R17-Pad2)
Other:
- board text added: "74LS47"
- board text added: "EN"
- board text added: "L293D"
- board text added: "devBoard rev1"

Commit message: update
Routing:
- net DIO1: track 155.4 -> 157.8 mm
- net +5V: vias 7 -> 5
Other:
- board text added: "LED"
- board text added: "SKLOPKE"
- board text added: "TIPKALA"
Changed lines of the file:
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@@
     (property "Sheetname" "")
     (attr through_hole)
-    (fp_text reference "SW4" (at -6.25 0 unlocked) (layer "F.SilkS")
+    (fp_text reference "SW4" (at -4.6 -3.35 unlocked) (layer "F.SilkS")
       (effects (font (size 1 1) (thickness 0.15)))
     )
@@
     (property "Sheetname" "")
     (attr through_hole)
-    (fp_text reference "SW3" (at -6.25 0 unlocked) (layer "F.SilkS")
+    (fp_text reference "SW3" (at -4.6 -3.1 unlocked) (layer "F.SilkS")
       (effects (font (size 1 1) (thickness 0.15)))
     )
@@
       (connect_pads (clearance 0))
       (min_thickness 0.254)
-      (keepout (tracks allowed) (vias allowed) (pads allowed) (copperpour not_allowed) (footprints allowed))
+      (keepout (tracks allowed) (vias allowed) (pads allowed ) (copperpour not_allowed) (footprints allowed))
       (fill (thermal_gap 0.508) (thermal_bridge_width 0.508))
       (polygon
@@
     (effects (font (size 1.5 1.5) (thickness 0.3)))
   )
+  (gr_text "LED" (at 197.25 82.75) (layer "F.SilkS")
+    (effects (font (size 1.5 1.5) (thickness 0.25)))
+  )
   (gr_text "DIO7" (at 176.1 54.65 90) (layer "F.SilkS")
     (effects (font (size 1.5 1.5) (thickness 0.3)))
@@
     (effects (font (size 1.5 1.5) (thickness 0.3)))
   )
+  (gr_text "SKLOPKE" (at 178.5 110.75) (layer "F.SilkS")
+    (effects (font (size 1.5 1.5) (thickness 0.25)))
+  )
   (gr_text "DIO6" (at 173.56 54.65 90) (layer "F.SilkS")
     (effects (font (size 1.5 1.5) (thickness 0.3)))
@@
     (effects (font (size 1.2 1.2) (thickness 0.3)))
   )
+  (gr_text "TIPKALA" (at 172.75 114.5) (layer "F.SilkS")
+    (effects (font (size 1.5 1.5) (thickness 0.25)))
+  )
   (gr_text "DIO1" (at 160.86 54.65 90) (layer "F.SilkS")
     (effects (font (size 1.5 1.5) (thickness 0.3)))
   )
-  (gr_text "L293D" (at 128.1 110.9) (layer "F.SilkS")
+  (gr_text "L293D" (at 126.75 110.9) (layer "F.SilkS")
     (effects (font (size 1.5 1.5) (thickness 0.25)))
   )
@@
   (segment (start 164.55 134.8) (end 165.05 134.8) (width 0.508) (layer "F.Cu") (net 1))
   (segment (start 111.755 98.62) (end 126.32 98.62) (width 0.508) (layer "F.Cu") (net 1))
-  (segment (start 143.1 107.15) (end 145.75 109.8) (width 0.762) (layer "F.Cu") (net 1))
   (segment (start 165.05 134.8) (end 165.6 135.35) (width 0.508) (layer "F.Cu") (net 1))
   (segment (start 183.85 148.15) (end 184.6 148.9) (width 0.762) (layer "F.Cu") (net 1))
@@
   (segment (start 152.95 112.55) (end 152.95 112) (width 0.762) (layer "F.Cu") (net 1))
   (segment (start 156.8425 103.1425) (end 156.8425 103.6575) (width 0.762) (layer "F.Cu") (net 1))
-  (segment (start 130.85 107.15) (end 136.6 107.15) (width 0.762) (layer "F.Cu") (net 1))
   (segment (start 183.1 148.9) (end 167.6 148.9) (width 0.762) (layer "F.Cu") (net 1))
   (segment (start 179.1 120.4) (end 183.85 125.15) (width 0.762) (layer "F.Cu") (net 1))
@@
   (segment (start 199.06 106.44) (end 199.35 106.15) (width 0.762) (layer "F.Cu") (net 1))
   (segment (start 152.95 112.45) (end 153 112.45) (width 0.762) (layer "F.Cu") (net 1))
+  (segment (start 132.5 107.25) (end 143.2 107.25) (width 0.762) (layer "F.Cu") (net 1))
   (segment (start 198.6 119.9) (end 199.35 120.65) (width 0.762) (layer "F.Cu") (net 1))
   (segment (start 126.38 98.62) (end 126.85 98.15) (width 0.508) (layer "F.Cu") (net 1))
@@
   (segment (start 198.39 106.44) (end 198.56 106.44) (width 0.762) (layer "F.Cu") (net 1))
   (segment (start 157.3275 103.6275) (end 156.8425 103.1425) (width 0.762) (layer "F.Cu") (net 1))
-  (segment (start 143.1 107.15) (end 140.1 107.15) (width 0.762) (layer "F.Cu") (net 1))
   (segment (start 193.685 50.4) (end 197.85 50.4) (width 0.762) (layer "F.Cu") (net 1))
   (segment (start 165.05 134.8) (end 165.6 134.25) (width 0.508) (layer "F.Cu") (net 1))
   (segment (start 143.7375 76.0125) (end 144.35 75.4) (width 0.762) (layer "F.Cu") (net 1))
   (segment (start 126.85 98.65) (end 126.85 99.15) (width 0.762) (layer "F.Cu") (net 1))
+  (segment (start 143.2 107.25) (end 145.75 109.8) (width 0.762) (layer "F.Cu") (net 1))
   (segment (start 157 112) (end 157.45 112) (width 0.762) (layer "F.Cu") (net 1))
   (segment (start 126.85 103.15) (end 127.35 103.65) (width 0.762) (layer "F.Cu") (net 1))
@@
   (segment (start 197.85 50.4) (end 199.35 51.9) (width 0.762) (layer "F.Cu") (net 1))
   (via (at 136.35 62.65) (size 0.8) (drill 0.4) (layers "F.Cu" "B.Cu") (net 1))
+  (via (at 132.5 107.25) (size 0.8) (drill 0.4) (layers "F.Cu" "B.Cu") (net 1))
   (via (at 133.35 55.65) (size 0.8) (drill 0.4) (layers "F.Cu" "B.Cu") (net 1))
-  (via (at 136.6 107.15) (size 0.8) (drill 0.4) (layers "F.Cu" "B.Cu") (net 1))
   (via (at 127.35 103.65) (size 0.8) (drill 0.4) (layers "F.Cu" "B.Cu") (net 1))
-  (via (at 130.85 107.15) (size 0.8) (drill 0.4) (layers "F.Cu" "B.Cu") (net 1))
-  (via (at 140.1 107.15) (size 0.8) (drill 0.4) (layers "F.Cu" "B.Cu") (net 1))
   (via (at 164.55 134.8) (size 0.8) (drill 0.4) (layers "F.Cu" "B.Cu") (net 1))
   (segment (start 136.35 62.65) (end 136.35 58.65) (width 0.762) (layer "B.Cu") (net 1))
   (segment (start 155.1 134.82) (end 164.53 134.82) (width 0.508) (layer "B.Cu") (net 1))
   (segment (start 164.53 134.82) (end 164.55 134.8) (width 0.508) (layer "B.Cu") (net 1))
-  (segment (start 130.85 107.15) (end 127.35 103.65) (width 0.762) (layer "B.Cu") (net 1))
-  (segment (start 136.6 107.15) (end 140.1 107.15) (width 0.762) (layer "B.Cu") (net 1))
+  (segment (start 127.35 103.65) (end 127.4 103.65) (width 0.762) (layer "B.Cu") (net 1))
+  (segment (start 131 107.25) (end 132.5 107.25) (width 0.762) (layer "B.Cu") (net 1))
+  (segment (start 127.4 103.65) (end 131 107.25) (width 0.762) (layer "B.Cu") (net 1))
   (segment (start 136.35 58.65) (end 133.35 55.65) (width 0.762) (layer "B.Cu") (net 1))
   (segment (start 129.375 61.025) (end 129.095 60.745) (width 0.508) (layer "F.Cu") (net 2))
@@
   (segment (start 139.85 69.15) (end 136.1175 72.8825) (width 0.508) (layer "F.Cu") (net 11))
   (segment (start 131.35 82.4) (end 131.35 91.15) (width 0.508) (layer "F.Cu") (net 11))
+  (segment (start 137.85 93.4) (end 138.6 94.15) (width 0.508) (layer "F.Cu") (net 11))
   (segment (start 159.725 67.525) (end 159.475 67.775) (width 0.508) (layer "F.Cu") (net 11))
   (segment (start 159.975 67.775) (end 159.475 67.775) (width 0.508) (layer "F.Cu") (net 11))
   (segment (start 135.1 93.4) (end 137.1 93.4) (width 0.254) (layer "F.Cu") (net 11))
+  (segment (start 138.6 94.15) (end 138.6 98.15) (width 0.508) (layer "F.Cu") (net 11))
   (segment (start 159.975 67.775) (end 159.975 67.275) (width 0.508) (layer "F.Cu") (net 11))
   (segment (start 160.1 67.9) (end 159.725 67.525) (width 0.508) (layer "F.Cu") (net 11))
-  (segment (start 138.6 107.15) (end 134.35 111.4) (width 0.508) (layer "F.Cu") (net 11))
-  (segment (start 138.6 94.15) (end 138.6 107.15) (width 0.508) (layer "F.Cu") (net 11))
   (segment (start 156.665 40.78) (end 156.665 43.32) (width 0.762) (layer "F.Cu") (net 11))
   (segment (start 134.325 79.425) (end 131.35 82.4) (width 0.508) (layer "F.Cu") (net 11))
-  (segment (start 137.1 93.4) (end 137.85 93.4) (width 0.508) (layer "F.Cu") (net 11))
   (segment (start 160.1 67.9) (end 159.975 67.775) (width 0.508) (layer "F.Cu") (net 11))
   (segment (start 156.665 44.715) (end 156.665 43.32) (width 0.508) (layer "F.Cu") (net 11))
+  (segment (start 134.1 113.4) (end 134.1 118.9) (width 0.508) (layer "F.Cu") (net 11))
+  (segment (start 131.25 105.5) (end 131.25 110.55) (width 0.508) (layer "F.Cu") (net 11))
   (segment (start 160.86 48.91) (end 156.665 44.715) (width 0.508) (layer "F.Cu") (net 11))
+  (segment (start 137.1 93.4) (end 137.85 93.4) (width 0.508) (layer "F.Cu") (net 11))
   (segment (start 158.1 69.15) (end 139.85 69.15) (width 0.508) (layer "F.Cu") (net 11))
-  (segment (start 134.1 111.65) (end 134.1 118.9) (width 0.508) (layer "F.Cu") (net 11))
   (segment (start 133.6 93.4) (end 135.1 93.4) (width 0.508) (layer "F.Cu") (net 11))
+  (segment (start 131.25 110.55) (end 134.1 113.4) (width 0.508) (layer "F.Cu") (net 11))
   (segment (start 160.86 50.35) (end 160.86 48.91) (width 0.508) (layer "F.Cu") (net 11))
   (segment (start 161.1 68.9) (end 160.1 67.9) (width 0.508) (layer "F.Cu") (net 11))
@@
   (segment (start 160.86 66.39) (end 159.975 67.275) (width 0.508) (layer "F.Cu") (net 11))
   (segment (start 160.86 50.35) (end 160.86 66.39) (width 0.508) (layer "F.Cu") (net 11))
-  (segment (start 137.85 93.4) (end 138.6 94.15) (width 0.508) (layer "F.Cu") (net 11))
-  (segment (start 134.35 111.4) (end 134.1 111.65) (width 0.508) (layer "F.Cu") (net 11))
+  (segment (start 138.6 98.15) (end 131.25 105.5) (width 0.508) (layer "F.Cu") (net 11))
   (via (at 161.1 68.9) (size 0.8) (drill 0.4) (layers "F.Cu" "B.Cu") (net 11))
   (via (at 164.6 71.65) (size 0.8) (drill 0.4) (layers "F.Cu" "B.Cu") (net 11))
@@
   )
   (zone (net 2) (net_name "GND") (layer "B.Cu") (hatch edge 0.508)
-    (connect_pads (clearance 0.508))
+    (connect_pads yes (clearance 0.508))
     (min_thickness 0.254) (filled_areas_thickness no)
     (fill yes (thermal_gap 0.508) (thermal_bridge_width 0.508))
