File: KiCAD files/myDAQExpansionBoard_v4/myDAQExpansionBoard.kicad_pcb (KiCad board)
At the start: 2 copper layers, 0 parts

Commit message: update
Parts:
- added C1: 100n, Capacitor_SMD:C_0603_1608Metric, F.Cu at (118.5, 61.5)
- added C2: 100n, Capacitor_SMD:C_0603_1608Metric, F.Cu at (33.0, 56.2)
- added C3: 100n, Capacitor_SMD:C_0603_1608Metric, F.Cu at (97.2, 73.8)
- added C4: 100n, Capacitor_SMD:C_0603_1608Metric, F.Cu at (30.8, 60.0)
- added C5: 470u, Capacitor_THT:CP_Radial_D12.5mm_P5.00mm, F.Cu at (76.8, 76.3)
- added C6: 1n, Capacitor_SMD:C_0603_1608Metric, F.Cu at (97.2, 76.5)
- added CD1: 1u, Capacitor_SMD:C_0805_2012Metric, F.Cu at (116.1, 109.8)
- added CD2: 1u, Capacitor_SMD:C_0805_2012Metric, F.Cu at (129.5, 110.0)
- added D1: RED, LED_THT:LED_D5.0mm, F.Cu at (125.2, 101.5)
- added D10: 1N4007, Diode_SMD:D_SMA, F.Cu at (39.0, 58.5)
- added D11: 1N4007, Diode_SMD:D_SMA, F.Cu at (49.3, 60.4)
- added D12: 1N4007, Diode_SMD:D_SMA, F.Cu at (47.8, 66.2)
- added D13: LED, LED_SMD:LED_1206_3216Metric, F.Cu at (72.8, 56.0)
- added D14: LED, LED_SMD:LED_1206_3216Metric, F.Cu at (161.0, 44.8)
- added D2: YELLOW, LED_THT:LED_D5.0mm, F.Cu at (134.2, 101.5)
- added D3: GREEN, LED_THT:LED_D5.0mm, F.Cu at (143.2, 101.5)
- added D4: BLUE, LED_THT:LED_D5.0mm, F.Cu at (152.2, 101.5)
- added D5: 1N4007, Diode_SMD:D_SMA, F.Cu at (37.0, 69.0)
- added D6: 1N4007, Diode_SMD:D_SMA, F.Cu at (44.8, 71.5)
- added D7: 1N4007, Diode_SMD:D_SMA, F.Cu at (38.8, 64.2)
- added D8: 1N4007, Diode_SMD:D_SMA, F.Cu at (33.5, 74.8)
- added D9: 1N4007, Diode_SMD:D_SMA, F.Cu at (45.5, 53.5)
- added H1: MountingHole_Pad, MountingHole:MountingHole_3.2mm_M3_ISO7380_Pad, F.Cu at (72.8, 37.2)
- added H2: MountingHole_Pad, MountingHole:MountingHole_3.2mm_M3_ISO7380_Pad, F.Cu at (165.8, 37.2)
- added H3: MountingHole_Pad, MountingHole:MountingHole_3.2mm_M3_ISO7380_Pad, F.Cu at (165.8, 130.2)
- added H4: MountingHole_Pad, MountingHole:MountingHole_3.2mm_M3_ISO7380_Pad, F.Cu at (72.8, 130.2)
- added J1: Conn_01x05_Male, Connector_PinHeader_2.54mm:PinHeader_1x05_P2.54mm_Vertical, F.Cu at (151.7, 49.8)
- added J2: Conn_01x05_Male, Connector_PinHeader_2.54mm:PinHeader_1x05_P2.54mm_Vertical, F.Cu at (151.7, 54.5)
- added J3: Conn_01x08_Male, Connector_PinHeader_2.54mm:PinHeader_1x08_P2.54mm_Vertical, F.Cu at (143.4, 44.8)
- added J4: OSTV7XX3151, Library:OSTV7XX3151, F.Cu at (83.1, 36.8)
- added J5: Screw_Terminal_01x02, TerminalBlock_Phoenix:TerminalBlock_Phoenix_MKDS-1,5-2-5.08_1x02_P5.08mm_Horizontal, F.Cu at (74.4, 97.5)
- added J6: Screw_Terminal_01x02, TerminalBlock_Phoenix:TerminalBlock_Phoenix_MKDS-1,5-2-5.08_1x02_P5.08mm_Horizontal, F.Cu at (74.4, 87.2)
- added J7: Screw_Terminal_01x01, Library:DELTRON 4mm banana socket - red, F.Cu at (80.5, 47.2)
- added J8: Screw_Terminal_01x01, Library:DELTRON 4mm banana socket - black, F.Cu at (80.5, 120.2)
- added JP1: Jumper_2_Open, Library:PinHeader_1x02_P2.54mm_jumper, F.Cu at (156.8, 65.0)
- added JP10: Jumper_2_Open, Library:PinHeader_1x02_P2.54mm_jumper, F.Cu at (110.5, 90.8)
- added JP2: Jumper_2_Open, Library:PinHeader_1x02_P2.54mm_jumper, F.Cu at (146.8, 65.0)
- added JP3: Jumper_2_Open, Library:PinHeader_1x02_P2.54mm_jumper, F.Cu at (151.8, 65.0)
- added JP4: Jumper_2_Open, Library:PinHeader_1x02_P2.54mm_jumper, F.Cu at (161.8, 65.0)
- added JP5: Jumper_2_Open, Library:PinHeader_1x02_P2.54mm_jumper, F.Cu at (152.5, 87.5)
- added JP6: Jumper_3_Open, Library:PinHeader_1x03_P2.54mm_Vertical_jumper, F.Cu at (130.0, 85.8)
- added JP7: Jumper_3_Open, Library:PinHeader_1x03_P2.54mm_Vertical_jumper, F.Cu at (105.3, 44.8)
- added JP8: Jumper_3_Open, Library:PinHeader_1x03_P2.54mm_Vertical_jumper, F.Cu at (111.0, 44.8)
- added JP9: Jumper_2_Open, Library:PinHeader_1x02_P2.54mm_jumper, F.Cu at (110.5, 97.0)
- added R1: 1k, Resistor_SMD:R_0603_1608Metric, F.Cu at (125.2, 94.5)
- added R10: 680, Resistor_SMD:R_0603_1608Metric, F.Cu at (122.2, 73.0)
- added R11: 680, Resistor_SMD:R_0603_1608Metric, F.Cu at (122.2, 76.2)
- added R12: 10k, Resistor_SMD:R_0603_1608Metric, F.Cu at (106.0, 66.0)
- added R13: 680, Resistor_SMD:R_0603_1608Metric, F.Cu at (122.2, 79.5)
- added R14: 680, Resistor_SMD:R_0603_1608Metric, F.Cu at (122.2, 82.8)
- added R15: 680, Resistor_SMD:R_0603_1608Metric, F.Cu at (122.2, 63.2)
- added R16: 680, Resistor_SMD:R_0603_1608Metric, F.Cu at (122.2, 66.5)
- added R17: R_Photo, OptoDevice:R_LDR_5.1x4.3mm_P3.4mm_Vertical, F.Cu at (119.5, 51.8)
- added R18: 10k, Resistor_SMD:R_0603_1608Metric, F.Cu at (116.0, 51.5)
- added R19: 2k7, Resistor_SMD:R_0603_1608Metric, F.Cu at (77.0, 56.0)
- added R2: 10k, Resistor_SMD:R_0603_1608Metric, F.Cu at (156.8, 72.5)
- added R20: 1k, Resistor_SMD:R_0603_1608Metric, F.Cu at (156.2, 44.8)
- added R3: 10k, Resistor_SMD:R_0603_1608Metric, F.Cu at (112.5, 109.8)
- added R4: 10k, Resistor_SMD:R_0603_1608Metric, F.Cu at (126.0, 110.0)
- added R5: 1k, Resistor_SMD:R_0603_1608Metric, F.Cu at (134.2, 94.5)
- added R6: 10k, Resistor_SMD:R_0603_1608Metric, F.Cu at (161.8, 72.5)
- added R7: 1k, Resistor_SMD:R_0603_1608Metric, F.Cu at (143.2, 94.5)
- added R8: 680, Resistor_SMD:R_0603_1608Metric, F.Cu at (122.2, 69.8)
- added R9: 1k, Resistor_SMD:R_0603_1608Metric, F.Cu at (152.2, 94.5)
- added RV1: 10k, Library:Potentiometer_Bourns_3386P_Vertical, F.Cu at (98.5, 61.2)
- added SW1: SW_SPDT, Library:we01014042, F.Cu at (144.2, 121.8)
- added SW2: SW_SPDT, Library:we01014042, F.Cu at (157.2, 121.8)
- added SW3: SW_Push, Library:Omron_B3F-12x12mm, F.Cu at (116.9, 115.5)
- added SW4: SW_Push, Library:Omron_B3F-12x12mm, F.Cu at (130.0, 115.5)
- added U1: 74LS47, Package_DIP:DIP-16_W7.62mm, F.Cu at (110.2, 64.1)
- added U2: 7segm-symbol, Library:7segm-SA52, F.Cu at (132.5, 73.0)
- added U3: ACS712xLCTR-05B, Package_SO:SOIC-8_3.9x4.9mm_P1.27mm, F.Cu at (91.2, 75.8)
- added U4: L298N, Library:TO-220-15_P2.54x2.54mm_StaggerOdd_Lead4.58mm_Vertical, F.Cu at (100.1, 103.4)
Routing:
- net +5V: track 0.00 -> 193.6 mm
- net DIO2: track 0.00 -> 148.6 mm, vias 0 -> 6
- net Net-(CD1-Pad1): track 0.00 -> 124.3 mm
- net DIO0: track 0.00 -> 123.4 mm
- net DIO3: track 0.00 -> 107.2 mm
- net Net-(CD2-Pad1): track 0.00 -> 104.1 mm
- net DIO1: track 0.00 -> 96.4 mm, vias 0 -> 2
- net Net-(R2-Pad1): track 0.00 -> 64.9 mm
- net Net-(R6-Pad2): track 0.00 -> 54.5 mm
- net Net-(D1-Pad1): track 0.00 -> 48.6 mm
- net /OUT3: track 0.00 -> 44.8 mm
- net /OUT2: track 0.00 -> 42.9 mm
- net Net-(JP8-Pad1): track 0.00 -> 41.3 mm
- net DIO7: track 0.00 -> 41.0 mm
- net DIO6: track 0.00 -> 28.1 mm
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Other:
- board outline added: 100 x 100 mm
- board text added: "5V"
- board text added: "CA"
- board text added: "CC"
- board text added: "GND"
- board text added: "POWER"
