File: KiCAD files/myDAQExpansionBoard_v4/myDAQExpansionBoard.kicad_pcb (KiCad board)
At the start: 2 copper layers, 100 x 100 mm, 73 parts, among them J1 Conn_01x05_Male, J2 Conn_01x05_Male, J3 Conn_01x08_Male, J4 OSTV7XX3151, J5 Screw_Terminal_01x02, J6 Screw_Terminal_01x02, J7 Screw_Terminal_01x01, J8 Screw_Terminal_01x01, SW1 SW_SPDT, SW2 SW_SPDT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

Commit message: update
Parts:
- C5: footprint Capacitor_THT:CP_Radial_D12.5mm_P5.00mm -> Capacitor_THT:C_Radial_D10.0mm_H16.0mm_P5.00mm
- moved C4 71.4 mm to (92.8, 95.5), turned to -90 degrees
- moved C2 65.0 mm to (81.2, 99.8), turned to 90 degrees
- moved D11 46.8 mm to (57.2, 106.5), turned to 180 degrees
- moved D10 46.5 mm to (57.2, 101.2), turned to 180 degrees
- moved D12 46.5 mm to (57.2, 111.8), turned to 180 degrees
- moved D9 44.1 mm to (57.2, 96.0), turned to 180 degrees
- moved D8 28.8 mm to (57.2, 91.0)
- moved D7 28.4 mm to (57.2, 85.8)
- moved D5 21.2 mm to (57.2, 75.2)
- moved U4 20.7 mm to (83.9, 90.4), turned to -90 degrees
- moved C5 16.3 mm to (91.5, 83.2), turned to 180 degrees
- moved J6 15.5 mm to (74.4, 102.7)
- moved D6 15.4 mm to (57.2, 80.5)
- moved C3 12.8 mm to (87.2, 65.8)
- moved C6 12.8 mm to (87.2, 68.5)
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Connections:
- RV1 pad 2: Net-(JP7-Pad1) -> Net-(JP8-Pad1)
- U3 pad 7: Net-(JP8-Pad1) -> Net-(JP7-Pad1)
Routing:
- net /OUT3: track 44.8 -> 0.00 mm
- net /OUT2: track 42.9 -> 0.00 mm
- net VDD: track 24.0 -> 0.14 mm
- net /OUT4: track 22.8 -> 0.00 mm
- net /OUT1: track 22.5 -> 0.00 mm
- net DIO2: track 148.6 -> 128.4 mm
- net DIO1: track 96.4 -> 113.9 mm, vias 2 -> 4
- net Net-(JP7-Pad1): track 18.4 -> 35.2 mm
- net DIO0: track 123.4 -> 106.9 mm
- net Net-(JP8-Pad1): track 41.3 -> 28.1 mm
- net Net-(JP9-Pad2): track 13.0 -> 0.00 mm
- net Net-(JP10-Pad2): track 7.92 -> 0.08 mm
- net Net-(CD1-Pad1): track 124.3 -> 119.3 mm
- net Net-(D14-Pad1): track 2.53 -> 6.51 mm
- net Net-(CD2-Pad1): track 104.1 -> 101.8 mm
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- added copper zone on F.Cu, net /IP-
- added copper zone on F.Cu, net VDD

Commit message: Update myDAQExpansionBoard.kicad_pcb
Routing:
- net DIO2: track 128.4 -> 160.3 mm
- net /OUT4: track 0.00 -> 21.5 mm
- net /OUT1: track 0.00 -> 19.6 mm
- net /IP-: track 0.00 -> 16.0 mm
- net /OUT2: track 0.00 -> 11.0 mm
- net /OUT3: track 0.00 -> 10.7 mm
Changed lines of the file:
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@@
   (segment (start 165.9 46.15) (end 165.9 47.3) (width 0.3048) (layer "F.Cu") (net 1))
   (segment (start 162.75 124.75) (end 161.625 125.875) (width 1.27) (layer "F.Cu") (net 1))
-  (segment (start 102.74 93.235) (end 102.75 93.225) (width 0.3048) (layer "F.Cu") (net 1))
   (segment (start 157.25 124.29) (end 160.04 124.29) (width 0.3048) (layer "F.Cu") (net 1))
   (segment (start 161.625 125.875) (end 160.5 127) (width 1.27) (layer "F.Cu") (net 1))
@@
   (segment (start 157.5 132) (end 144.25 132) (width 1.27) (layer "F.Cu") (net 1))
   (segment (start 144.25 132) (end 104.25 132) (width 1.27) (layer "F.Cu") (net 1))
+  (segment (start 89.02 94.165) (end 92.19 94.165) (width 0.3048) (layer "F.Cu") (net 3))
+  (segment (start 92.19 94.165) (end 92.75 94.725) (width 0.3048) (layer "F.Cu") (net 3))
+  (segment (start 91.5 93.475) (end 91.5 83.25) (width 0.3048) (layer "F.Cu") (net 3))
+  (segment (start 92.75 94.725) (end 91.5 93.475) (width 0.3048) (layer "F.Cu") (net 3))
   (via (at 71 68.5) (size 0.8) (drill 0.4) (layers "F.Cu" "B.Cu") (free) (net 3))
   (via (at 74 68.5) (size 0.8) (drill 0.4) (layers "F.Cu" "B.Cu") (free) (net 3))
@@
   (segment (start 126.4875 90.9875) (end 133.5 90.9875) (width 0.3048) (layer "F.Cu") (net 10))
   (segment (start 130.675 47.075) (end 130.675 47.575) (width 0.3048) (layer "F.Cu") (net 10))
+  (segment (start 114.5 98.25) (end 114.5 93.25) (width 0.3048) (layer "F.Cu") (net 10))
   (segment (start 112.21 66) (end 111.545 66.665) (width 0.3048) (layer "F.Cu") (net 10))
   (segment (start 141.4875 90.9875) (end 137 90.9875) (width 0.3048) (layer "F.Cu") (net 10))
   (segment (start 130.675 50.075) (end 130.675 56.325) (width 0.3048) (layer "F.Cu") (net 10))
+  (segment (start 110.965 101.785) (end 114.5 98.25) (width 0.3048) (layer "F.Cu") (net 10))
   (segment (start 116.7625 90.9875) (end 123.9875 90.9875) (width 0.3048) (layer "F.Cu") (net 10))
   (segment (start 111.545 66.665) (end 110.16 66.665) (width 0.3048) (layer "F.Cu") (net 10))
   (segment (start 141.5 90.975) (end 141.4875 90.9875) (width 0.3048) (layer "F.Cu") (net 10))
+  (segment (start 89.02 101.785) (end 110.965 101.785) (width 0.3048) (layer "F.Cu") (net 10))
   (segment (start 130.675 44.75) (end 130.675 47.075) (width 0.3048) (layer "F.Cu") (net 10))
   (segment (start 142.4875 90.9875) (end 143.2375 91.7375) (width 0.3048) (layer "F.Cu") (net 10))
@@
   (segment (start 133.215 57.535) (end 131.25 59.5) (width 0.3048) (layer "F.Cu") (net 11))
   (segment (start 152.2375 92.4875) (end 142.75 83) (width 0.3048) (layer "F.Cu") (net 11))
+  (segment (start 86 113.25) (end 89.02 110.23) (width 0.3048) (layer "F.Cu") (net 12))
+  (segment (start 89.02 110.23) (end 89.02 106.865) (width 0.3048) (layer "F.Cu") (net 12))
+  (segment (start 74.39 107.785) (end 79.855 113.25) (width 0.3048) (layer "F.Cu") (net 12))
+  (segment (start 79.855 113.25) (end 86 113.25) (width 0.3048) (layer "F.Cu") (net 12))
+  (segment (start 81.05 102.705) (end 83.94 105.595) (width 0.3048) (layer "F.Cu") (net 13))
+  (segment (start 74.39 102.705) (end 81.05 102.705) (width 0.3048) (layer "F.Cu") (net 13))
+  (segment (start 83.895 86.5) (end 78 86.5) (width 0.3048) (layer "F.Cu") (net 14))
+  (segment (start 74.445 90.055) (end 74.445 91.5) (width 0.3048) (layer "F.Cu") (net 14))
+  (segment (start 89.02 91.625) (end 83.895 86.5) (width 0.3048) (layer "F.Cu") (net 14))
+  (segment (start 78 86.5) (end 74.445 90.055) (width 0.3048) (layer "F.Cu") (net 14))
+  (segment (start 80.255 96.58) (end 83.94 92.895) (width 0.3048) (layer "F.Cu") (net 15))
+  (segment (start 74.445 96.58) (end 80.255 96.58) (width 0.3048) (layer "F.Cu") (net 15))
   (segment (start 83.375 57.75) (end 83.875 58.25) (width 0.3048) (layer "F.Cu") (net 16))
   (segment (start 86.625 58.25) (end 87.625 57.25) (width 0.3048) (layer "F.Cu") (net 16))

Commit message: update
Parts:
- D10, D11, D12, D5, D6, D7, D8, D9: moved to B.Cu
- moved RV1 28.6 mm to (112.5, 96.0)
- moved D11 26.8 mm to (83.0, 113.8), turned to -90 degrees
- moved D5 26.3 mm to (83.0, 80.8), turned to -90 degrees
- moved D9 25.4 mm to (75.5, 113.8), turned to -90 degrees
- moved D10 25.3 mm to (79.2, 113.8), turned to -90 degrees
- moved D6 22.0 mm to (79.2, 80.8), turned to -90 degrees
- moved D7 18.9 mm to (75.5, 80.8), turned to -90 degrees
- moved JP9 18.3 mm to (99.8, 82.2), turned to 0 degrees
- moved D8 17.8 mm to (71.8, 80.8), turned to -90 degrees
- moved D12 14.6 mm to (71.8, 113.8), turned to -90 degrees
- moved JP10 11.0 mm to (103.5, 82.2), turned to 0 degrees
- moved C4 8.68 mm to (94.5, 87.0), turned to 0 degrees
- moved J6 0.96 mm to (74.7, 101.8)
- moved C5 0.75 mm to (91.5, 82.5)
- moved JP5 0.74 mm to (151.8, 87.5)
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Routing:
- net +5V: track 192.4 -> 449.9 mm, vias 0 -> 10
- net DIO3: track 107.2 -> 191.3 mm, vias 0 -> 2
- net GND: track 0.00 -> 58.4 mm, vias 0 -> 11
- net DIO1: track 113.9 -> 160.6 mm
- net Net-(JP10-Pad2): track 0.08 -> 43.6 mm, vias 0 -> 2
- net /OUT1: track 19.6 -> 58.2 mm
- net /OUT3: track 10.7 -> 44.4 mm
- net /OUT2: track 11.0 -> 42.8 mm
- net /OUT4: track 21.5 -> 52.3 mm
- net Net-(JP8-Pad1): track 28.1 -> 57.4 mm
- net DIO0: track 106.9 -> 132.9 mm, vias 0 -> 2
- net Net-(JP9-Pad2): track 0.00 -> 19.8 mm
- net /IP-: track 16.0 -> 0.00 mm, vias 21 -> 0
- net VDD: track 0.14 -> 10.2 mm
- net DIO6: track 28.1 -> 37.3 mm
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- added copper zone on B.Cu, net /IP-
- added copper zone on B.Cu, net GND
Other:
- board text added: "EXT. POWER"

Commit message: update
Parts:
- RV1: footprint Library:Potentiometer_Bourns_3386P_Vertical -> Library:PTV09A-4225F-B502
- moved RV1 3.73 mm to (110.0, 98.7), turned to 180 degrees
Routing:
- net +5V: track 449.9 -> 483.9 mm, vias 10 -> 12
- net DIO0: track 132.9 -> 130.3 mm
- net DIO1: track 160.6 -> 163.2 mm
- net unconnected-(J4-Pad1): track 0.00 -> 2.54 mm
- net DIO5: track 34.7 -> 37.2 mm
- net AI1+: track 7.95 -> 10.5 mm
- net unconnected-(J4-Pad5): track 0.00 -> 2.54 mm
- net unconnected-(J4-Pad2): track 0.00 -> 2.54 mm
- net DIO7: track 41.0 -> 43.5 mm
- net DIO4: track 30.5 -> 33.0 mm
- net AO0: track 7.97 -> 10.5 mm
- net DIO3: track 191.3 -> 193.9 mm
- net Net-(JP8-Pad1): track 57.4 -> 55.6 mm
- net GND: track 58.4 -> 57.3 mm

Commit message: update
Parts:
- moved D11 22.4 mm to (92.8, 93.6)
Routing:
- net GND: track 57.3 -> 92.7 mm
- net /OUT1: track 58.2 -> 31.5 mm
- net +5V: track 483.9 -> 482.0 mm
Other:
- board text added: "JLCJLCJLCJLC"
Changed lines of the file:
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@@
     (property "Sheetname" "")
     (attr through_hole)
-    (fp_text reference "U1" (at 3.81 -2.33) (layer "F.SilkS")
+    (fp_text reference "U1" (at 3.84 20.125) (layer "F.SilkS")
       (effects (font (size 1 1) (thickness 0.15)))
     )
@@
   )
   (footprint "Diode_SMD:D_SMA" (layer "B.Cu")
-    (at 83 113.75 -90)
+    (at 92.8 93.6 -90)
     (descr "Diode SMA (DO-214AC)")
     (tags "Diode SMA (DO-214AC)")
@@
     (effects (font (size 1.2 1.2) (thickness 0.2)))
   )
+  (gr_text "JLCJLCJLCJLC" (at 114 73.5 90) (layer "F.SilkS")
+    (effects (font (size 1.5 1.5) (thickness 0.3)))
+  )
   (gr_text "GND" (at 164.25 54.5 90) (layer "F.SilkS")
     (effects (font (size 1.2 1.2) (thickness 0.2)))
@@
   (segment (start 86.38 65.845) (end 86.475 65.75) (width 0.3048) (layer "F.Cu") (net 1))
   (segment (start 164.85 48.35) (end 164.85 49.75) (width 0.3048) (layer "F.Cu") (net 1))
+  (segment (start 84.2 113.7) (end 102 113.7) (width 0.508) (layer "F.Cu") (net 1))
   (segment (start 119.55 53.2) (end 118.5 54.25) (width 0.508) (layer "F.Cu") (net 1))
   (segment (start 119.75 132) (end 104.25 132) (width 1.27) (layer "F.Cu") (net 1))
@@
   (segment (start 130.75 88.25) (end 129.96 87.46) (width 0.508) (layer "F.Cu") (net 1))
   (segment (start 87.25 63.75) (end 90.75 63.75) (width 0.508) (layer "F.Cu") (net 1))
-  (segment (start 81.1 113.7) (end 102 113.7) (width 0.508) (layer "F.Cu") (net 1))
   (segment (start 121.75 110) (end 119.75 112) (width 0.508) (layer "F.Cu") (net 1))
   (segment (start 160.5 129) (end 157.5 132) (width 1.27) (layer "F.Cu") (net 1))
@@
   (segment (start 112.5 91.6895) (end 112.5 88) (width 0.508) (layer "F.Cu") (net 1))
   (via (at 90.75 63.75) (size 0.8) (drill 0.4) (layers "F.Cu" "B.Cu") (net 1))
-  (via (at 81.1 113.7) (size 0.8) (drill 0.4) (layers "F.Cu" "B.Cu") (net 1))
   (via (at 102 109.75) (size 0.8) (drill 0.4) (layers "F.Cu" "B.Cu") (net 1))
   (via (at 115.5 61.5) (size 0.8) (drill 0.4) (layers "F.Cu" "B.Cu") (net 1))
@@
   (via (at 81.25 103.75) (size 0.8) (drill 0.4) (layers "F.Cu" "B.Cu") (net 1))
   (via (at 107.5 82.25) (size 0.8) (drill 0.4) (layers "F.Cu" "B.Cu") (net 1))
+  (via (at 84.2 113.7) (size 0.8) (drill 0.4) (layers "F.Cu" "B.Cu") (net 1))
   (segment (start 102 109.75) (end 102 103.75) (width 1.27) (layer "B.Cu") (net 1))
+  (segment (start 81.25 103.75) (end 81.25 110.75) (width 0.508) (layer "B.Cu") (net 1))
   (segment (start 107.475 82.225) (end 107.5 82.25) (width 0.508) (layer "B.Cu") (net 1))
   (segment (start 99 63.75) (end 101 63.75) (width 0.508) (layer "B.Cu") (net 1))
   (segment (start 103.5 82.225) (end 107.475 82.225) (width 0.508) (layer "B.Cu") (net 1))
-  (segment (start 81.1 103.9) (end 81.1 112.4) (width 0.508) (layer "B.Cu") (net 1))
+  (segment (start 81.25 110.75) (end 84.2 113.7) (width 0.508) (layer "B.Cu") (net 1))
   (segment (start 127.25 85.75) (end 123.5 89.5) (width 1.27) (layer "B.Cu") (net 1))
-  (segment (start 81.1 112.4) (end 81.1 113.7) (width 0.508) (layer "B.Cu") (net 1))
-  (segment (start 81.25 103.75) (end 81.1 103.9) (width 0.508) (layer "B.Cu") (net 1))
   (segment (start 129.96 85.75) (end 127.25 85.75) (width 1.27) (layer "B.Cu") (net 1))
   (segment (start 115.5 61.5) (end 109 61.5) (width 0.508) (layer "B.Cu") (net 1))
@@
   (segment (start 109.725 36.8) (end 109.725 39.34) (width 1.27) (layer "B.Cu") (net 2))
   (segment (start 117.345 39.38) (end 117.345 36.84) (width 1.27) (layer "B.Cu") (net 2))
-  (segment (start 117.345 36.84) (end 117.345 35.095) (width 0.508) (layer "B.Cu") (net 2))
+  (segment (start 149.505 34.75) (end 151.635 36.88) (width 0.508) (layer "B.Cu") (net 2))
   (segment (start 109.75 34.75) (end 102 34.75) (width 0.508) (layer "B.Cu") (net 2))
-  (segment (start 117.345 35.095) (end 117 34.75) (width 0.508) (layer "B.Cu") (net 2))
+  (segment (start 117.345 36.84) (end 117.345 34.845) (width 0.508) (layer "B.Cu") (net 2))
   (segment (start 90.675 35.075) (end 90.675 36.8) (width 0.508) (layer "B.Cu") (net 2))
   (segment (start 102.105 34.855) (end 102 34.75) (width 0.508) (layer "B.Cu") (net 2))
   (segment (start 109.725 34.775) (end 109.75 34.75) (width 0.508) (layer "B.Cu") (net 2))
+  (segment (start 117.25 34.75) (end 149.505 34.75) (width 0.508) (layer "B.Cu") (net 2))
   (segment (start 102 34.75) (end 91 34.75) (width 0.508) (layer "B.Cu") (net 2))
   (segment (start 109.725 36.8) (end 109.725 34.775) (width 0.508) (layer "B.Cu") (net 2))
   (segment (start 91 34.75) (end 90.675 35.075) (width 0.508) (layer "B.Cu") (net 2))
+  (segment (start 117.345 34.845) (end 117.25 34.75) (width 0.508) (layer "B.Cu") (net 2))
+  (segment (start 109.75 34.75) (end 117.25 34.75) (width 0.508) (layer "B.Cu") (net 2))
   (segment (start 102.105 36.8) (end 102.105 34.855) (width 0.508) (layer "B.Cu") (net 2))
-  (segment (start 117 34.75) (end 109.75 34.75) (width 0.508) (layer "B.Cu") (net 2))
   (segment (start 90.675 36.8) (end 90.675 39.34) (width 1.27) (layer "B.Cu") (net 2))
   (segment (start 86.36 68.385) (end 86.475 68.5) (width 0.3048) (layer "F.Cu") (net 4))
@@
   (segment (start 85.75 87.25) (end 87.375 88.875) (width 1.27) (layer "F.Cu") (net 14))
   (segment (start 87.375 89.98) (end 87.375 88.875) (width 1.27) (layer "F.Cu") (net 14))
-  (segment (start 92.25 93) (end 90.875 91.625) (width 1.27) (layer "B.Cu") (net 14))
-  (segment (start 90.875 91.625) (end 89.02 91.625) (width 1.27) (layer "B.Cu") (net 14))
-  (segment (start 83 111.75) (end 90 111.75) (width 1.27) (layer "B.Cu") (net 14))
-  (segment (start 90 111.75) (end 92.25 109.5) (width 1.27) (layer "B.Cu") (net 14))
+  (segment (start 92.8 91.6) (end 89.045 91.6) (width 1.27) (layer "B.Cu") (net 14))
   (segment (start 75.5 88) (end 74.695 88.805) (width 1.27) (layer "B.Cu") (net 14))
   (segment (start 74.695 88.805) (end 74.695 91.555) (width 1.27) (layer "B.Cu") (net 14))
-  (segment (start 92.25 109.5) (end 92.25 93) (width 1.27) (layer "B.Cu") (net 14))
+  (segment (start 89.045 91.6) (end 89.02 91.625) (width 1.27) (layer "B.Cu") (net 14))
   (segment (start 75.5 82.75) (end 75.5 88) (width 1.27) (layer "B.Cu") (net 14))
   (segment (start 74.695 96.635) (end 78.115 96.635) (width 1.27) (layer "F.Cu") (net 15))
@@
         (xy 98 133.75)
         (xy 98 41.75)
-        (xy 115.5 41.75)
-        (xy 115.5 33.75)
+        (xy 149.6 41.75)
+        (xy 149.6 33.75)
         (xy 169.25 33.75)
       )

Commit message: update
Changed lines of the file:
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@@
     (connect_pads (clearance 0.354))
     (min_thickness 0.254) (filled_areas_thickness no)
-    (fill yes (thermal_gap 0.508) (thermal_bridge_width 0.508))
+    (fill yes (thermal_gap 0.254) (thermal_bridge_width 0.508))
     (polygon
       (pts
         (xy 169.25 133.75)
         (xy 98 133.75)
-        (xy 98 41.75)
-        (xy 149.6 41.75)
+        (xy 98 41.25)
+        (xy 149.6 41.25)
         (xy 149.6 33.75)
         (xy 169.25 33.75)
@@
         (xy 96.75 133.75)
         (xy 69.25 133.75)
-        (xy 69.25 33.75)
+        (xy 69.25 50.5)
+        (xy 91.5 50.5)
+        (xy 91.5 45.5)
+        (xy 89 43)
+        (xy 89 33.75)
         (xy 92.25 33.75)
-        (xy 92.25 41.75)
-        (xy 96.75 41.75)
+        (xy 92.25 40.5)
+        (xy 93 41.25)
+        (xy 96.75 41.25)
       )
     )
@@
     (connect_pads yes (clearance 0))
     (min_thickness 0.254) (filled_areas_thickness no)
-    (fill yes (thermal_gap 0.508) (thermal_bridge_width 0.508) (smoothing chamfer) (radius 1))
+    (fill yes (thermal_gap 0.508) (thermal_bridge_width 0.508) (smoothing chamfer) (radius 0.2))
     (polygon
       (pts
@@
         (xy 88.5 80)
         (xy 70 80)
-        (xy 70 75.5)
-        (xy 87.75 75.5)
+        (xy 70 77)
+        (xy 89.5 77)
       )
     )
