File: KiCAD files/myDAQExpansionBoard_v4/myDAQExpansionBoard.kicad_sch (KiCad schematic)
At the start: 61 parts, among them J1 OSTV7XX3151, J2 Conn_01x05_Male, J3 Conn_01x05_Male, J4 Screw_Terminal_01x02, J5 Screw_Terminal_01x01, J6 Screw_Terminal_01x02, J7 Conn_01x08_Male, J8 Screw_Terminal_01x01, SW1 SW_Push, SW2 SW_Push, SW3 SW_SPDT, SW4 SW_SPDT, U1 74LS47, U2 7segm-symbol, U3 ACS712xLCTR-05B, U4 LM35-D, U5 L293D

Commit message: update
Parts:
- removed C3: 100n, Capacitor_SMD:C_0603_1608Metric, symbol Device:C
- removed J4, J6: Screw_Terminal_01x02, TerminalBlock_Phoenix:TerminalBlock_Phoenix_MKDS-1,5-2-5.08_1x02_P5.08mm_Horizontal, symbol Connector:Screw_Terminal_01x02
- removed JP12, JP13, JP14: Jumper_3_Open, Connector_PinHeader_2.54mm:PinHeader_1x03_P2.54mm_Vertical, symbol Jumper:Jumper_3_Open
- removed R17: 1R, Library:R_Axial_Power_L60.0mm_W14.0mm_P71.12mm, symbol Device:R
- removed R20, R21: 10k, Resistor_SMD:R_0603_1608Metric, symbol Device:R
- removed U4: LM35-D, Package_SO:SOIC-8_3.9x4.9mm_P1.27mm, symbol Sensor_Temperature:LM35-D
- removed U5: L293D, Package_DIP:DIP-16_W7.62mm, symbol Driver_Motor:L293D
- added C? (x2): 100n, Capacitor_SMD:C_0603_1608Metric, symbol Device:C
- added D?: LED, LED_THT:LED_D5.0mm, symbol Device:LED
- added J? (x2): Screw_Terminal_01x02, symbol Connector:Screw_Terminal_01x02
- added JP? (x2): Jumper_3_Open, Connector_PinHeader_2.54mm:PinHeader_1x03_P2.54mm_Vertical, symbol Jumper:Jumper_3_Open
- added R?: 1k, Resistor_SMD:R_0603_1608Metric, symbol Device:R
- added R? (x2): 10k, Resistor_SMD:R_0603_1608Metric, symbol Device:R
- added RV?: 10k, symbol Device:R_Potentiometer
- added U?: L298N, Package_TO_SOT_THT:TO-220-15_P2.54x2.54mm_StaggerOdd_Lead4.58mm_Vertical, symbol Driver_Motor:L298N
- renumbered C4 to C?, C2 to C?, C1 to C?, CD2 to CD?, CD1 to CD?, D1 to D?, D3 to D?, D2 to D?, H1 to H?, H4 to H?, H3 to H?, H2 to H?, J5 to J?, J3 to J?, J8 to J?, J1 to J?, J2 to J?, J7 to J?, JP10 to JP?, JP3 to JP?, JP5 to JP?, JP4 to JP?, JP2 to JP?, JP1 to JP?, JP9 to JP?, JP11 to JP?, R7 to R?, R2 to R?, R8 to R?, R3 to R?, R1 to R?, R9 to R?, R11 to R?, R18 to R?, R16 to R?, R12 to R?, R13 to R?, R5 to R?, R6 to R?, R15 to R?, R19 to R?, R4 to R?, R14 to R?, SW2 to SW?, SW3 to SW?, SW1 to SW?, SW4 to SW?, U1 to U?, U2 to U?, U3 to U?
Connections:
- net +5V: now also C?.1, JP?.3 (B), JP?.3 (B), RV?.1, U?.9 (Vss)
- net DIO0: now also U?.5 (IN1)
- net DIO1: now also U?.7 (IN2)
- net DIO2: now also U?.10 (IN3)
- net DIO3: now also D?.2 (A), U?.12 (IN4)
- net GND: now also C?.2, C?.2, JP?.1 (A), JP?.1 (A), RV?.3, U?.8 (GND); no longer U?.3 (IP-), U?.4 (IP-)
- net VDD: now also J?.1 (Pin_1), U?.1 (IP+), U?.2 (IP+)
- net at JP?.1 (A), R?.2, R?.2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: now also R?.2
- net at JP?.1 (A): now also RV?.2
- new net: D?.1 (K), R?.1
- new net: JP?.2 (C), R?.1 (x2)
- new net: R?.2, U?.11 (EnB)
- new net: J?.1 (Pin_1), U?.2 (OUT1)
- new net: J?.2 (Pin_2), U?.3 (OUT2)
- new net: R?.2, U?.6 (EnA)
- new net: J?.1 (Pin_1), U?.13 (OUT3)
- new net: J?.2 (Pin_2), U?.14 (OUT4)
- new net I_SENSE: C?.1, U?.3 (IP-), U?.4 (IP-), U?.4 (Vs)
Other:
- note added: "POTENCIOMETAR"
- note removed: "H-MOST"
- note removed: "LM35"
- note removed: "NAPAJANJE"
- note removed: "TO-DO - spojiti priključnice za motor, napajanje za motor dovesti s donje strane - pojašnjenja za sve jumpere - senzor temperature se poklapa - potenciometar s kondenzatorom - hmost kondenzatori - smanjiti silkscreen konektora za stepper - da li je redosljed izlaza hmosta dobar? - dioda za reverse polarity protection - ne treba odvojiti gnd, samo udaljiti analogni od digitalnog dijela - sklopka: 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"
- moved on the sheet: C?, J?, JP?, R?, U?

Commit message: update
Parts:
- added D3: LED, LED_THT:LED_D5.0mm, symbol Device:LED
- added R8: 1k, Resistor_SMD:R_0603_1608Metric, symbol Device:R
- gave numbers to parts that had none: 62
Connections:
- net +5V: now also D3.2 (A)
- net GND: now also R8.2
- new net: D3.1 (K), R8.1
Other:
- note added: "POWER LED"

Commit message: update
Parts:
- removed C3: 100n, Capacitor_SMD:C_0603_1608Metric, symbol Device:C
- removed JP7, JP8: Jumper_3_Open, Connector_PinHeader_2.54mm:PinHeader_1x03_P2.54mm_Vertical, symbol Jumper:Jumper_3_Open
- removed R18: 10k, Resistor_SMD:R_0603_1608Metric, symbol Device:R
- added C4: 100n, Capacitor_SMD:C_0603_1608Metric, symbol Device:C
- added C5: 470u, Capacitor_THT:CP_Radial_D12.5mm_P5.00mm, symbol Device:C_Polarized
- added D10, D11, D12, D5, D6, D7, D8, D9: 1N4007, Library:do214ab, symbol Diode:1N4007
- added D13: LED, LED_SMD:LED_1206_3216Metric, symbol Device:LED
- added JP10, JP9: Jumper_2_Open, Library:PinHeader_1x02_P2.54mm_jumper, symbol Jumper:Jumper_2_Open
- CD1, CD2: value 100n -> 1u; footprint Capacitor_SMD:C_0603_1608Metric -> Capacitor_SMD:C_0805_2012Metric
- D1: value LED -> RED
- D14: renamed from D3; footprint LED_THT:LED_D5.0mm -> LED_SMD:LED_1206_3216Metric
- D2: value LED -> YELLOW
- D3: renamed from D4; value LED -> GREEN
- D4: renamed from D5; value LED -> BLUE
- J5: renamed from J2; footprint (none) -> TerminalBlock_Phoenix:TerminalBlock_Phoenix_MKDS-1,5-2-5.08_1x02_P5.08mm_Horizontal
- J6: renamed from J3; footprint (none) -> TerminalBlock_Phoenix:TerminalBlock_Phoenix_MKDS-1,5-2-5.08_1x02_P5.08mm_Horizontal
- JP1, JP2, JP3, JP4, JP5: footprint Connector_PinHeader_2.54mm:PinHeader_1x02_P2.54mm_Vertical -> Library:PinHeader_1x02_P2.54mm_jumper
- JP6: footprint Connector_PinHeader_2.54mm:PinHeader_1x03_P2.54mm_Vertical -> Library:PinHeader_1x02_P2.54mm_jumper
- JP7: renamed from JP9; footprint Connector_PinHeader_2.54mm:PinHeader_1x03_P2.54mm_Vertical -> Library:PinHeader_1x02_P2.54mm_jumper
- JP8: renamed from JP10; footprint Connector_PinHeader_2.54mm:PinHeader_1x03_P2.54mm_Vertical -> Library:PinHeader_1x02_P2.54mm_jumper
- R19: value 10k -> 2k7
- renumbered C4 to C3, C5 to C6, J4 to J1, J5 to J2, J6 to J3, J1 to J4, R11 to R10, R12 to R11, R13 to R12, R14 to R13, R15 to R14, R16 to R15, R17 to R16, R20 to R17, R21 to R18, R8 to R20, R9 to R8, R10 to R9, U4 to U3, U3 to U4
Connections:
- net +5V: now also JP10.1 (A), JP9.1 (A)
- net GND: now also R19.2, U4.1 (SENSE_A), U4.15 (SENSE_B), C4.2, C5.2, D10.2 (A), D11.2 (A), D12.2 (A), D9.2 (A)
- net VDD: now also D13.2 (A)
- net at R19.1: now also D13.1 (K)
- net at U4.11 (EnB): now also JP10.2 (B); no longer R19.2
- net OUT1: now reaches J5.1 (Pin_1), U4.2 (OUT1)
- net OUT1: now also D11.1 (K), D7.2 (A)
- net OUT2: now reaches J5.2 (Pin_2), U4.3 (OUT2)
- net OUT2: now also D12.1 (K), D8.2 (A)
- net at U4.6 (EnA): now also JP9.2 (B)
- net OUT3: now reaches J6.1 (Pin_1), U4.13 (OUT3)
- net OUT3: now also D10.1 (K), D6.2 (A)
- net OUT4: now reaches J6.2 (Pin_2), U4.14 (OUT4)
- net OUT4: now also D5.2 (A), D9.1 (K)
- net I_SENSE renamed IP-
- net IP-: now also C4.1, C5.1, D5.1 (K), D6.1 (K), D7.1 (K), D8.1 (K)
Other:
- note added: "D5 to D12 = 2 A Fast diodes VF ≤ 1.2 V @ I = 2 A trr ≤ 200 ns SS34"
- note added: "EXTERNAL POWER"
- note added: "L298N"
- note added: "LOGIC POWER LED"
- note removed: "POWER LED"
- moved on the sheet: C2, C3, D14, H1, H2, H3, H4, J1, J2, J3, J5, J6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

Commit message: update
Parts:
- D10, D11, D12, D5, D6, D7, D8, D9: footprint Library:do214ab -> Diode_SMD:D_SMA
- RV1: footprint (none) -> Library:Potentiometer_Bourns_3386P_Vertical
Changed lines of the file:
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@@
       (effects (font (size 1.27 1.27)) (justify left) hide)
     )
-    (property "Footprint" "Library:do214ab" (id 2) (at 249.555 147.955 0)
+    (property "Footprint" "Diode_SMD:D_SMA" (id 2) (at 249.555 147.955 0)
       (effects (font (size 1.27 1.27)) hide)
     )
@@
       (effects (font (size 1.27 1.27)) (justify left) hide)
     )
-    (property "Footprint" "Library:do214ab" (id 2) (at 228.6 127 0)
+    (property "Footprint" "Diode_SMD:D_SMA" (id 2) (at 228.6 127 0)
       (effects (font (size 1.27 1.27)) hide)
     )
@@
       (effects (font (size 1.27 1.27)) (justify left) hide)
     )
-    (property "Footprint" "Library:do214ab" (id 2) (at 249.555 127 0)
+    (property "Footprint" "Diode_SMD:D_SMA" (id 2) (at 249.555 127 0)
       (effects (font (size 1.27 1.27)) hide)
     )
@@
       (effects (font (size 1.27 1.27)) (justify left) hide)
     )
-    (property "Footprint" "Library:do214ab" (id 2) (at 228.6 147.955 0)
+    (property "Footprint" "Diode_SMD:D_SMA" (id 2) (at 228.6 147.955 0)
       (effects (font (size 1.27 1.27)) hide)
     )
@@
       (effects (font (size 1.27 1.27)) (justify left) hide)
     )
-    (property "Footprint" "Library:do214ab" (id 2) (at 235.585 127 0)
+    (property "Footprint" "Diode_SMD:D_SMA" (id 2) (at 235.585 127 0)
       (effects (font (size 1.27 1.27)) hide)
     )
@@
       (effects (font (size 1.27 1.27)) (justify right))
     )
-    (property "Footprint" "" (id 2) (at 107.95 120.015 0)
+    (property "Footprint" "Library:Potentiometer_Bourns_3386P_Vertical" (id 2) (at 107.95 120.015 0)
       (effects (font (size 1.27 1.27)) hide)
     )
@@
       (effects (font (size 1.27 1.27)) (justify left) hide)
     )
-    (property "Footprint" "Library:do214ab" (id 2) (at 242.57 147.955 0)
+    (property "Footprint" "Diode_SMD:D_SMA" (id 2) (at 242.57 147.955 0)
       (effects (font (size 1.27 1.27)) hide)
     )
@@
       (effects (font (size 1.27 1.27)) (justify left) hide)
     )
-    (property "Footprint" "Library:do214ab" (id 2) (at 242.57 127 0)
+    (property "Footprint" "Diode_SMD:D_SMA" (id 2) (at 242.57 127 0)
       (effects (font (size 1.27 1.27)) hide)
     )
@@
       (effects (font (size 1.27 1.27)) (justify left) hide)
     )
-    (property "Footprint" "Library:do214ab" (id 2) (at 235.585 147.955 0)
+    (property "Footprint" "Diode_SMD:D_SMA" (id 2) (at 235.585 147.955 0)
       (effects (font (size 1.27 1.27)) hide)
     )
@@
     )
     (path "/20cd31ae-7493-46e2-b1cb-4b1df99ea6d1"
-      (reference "D5") (unit 1) (value "1N4007") (footprint "Library:do214ab")
+      (reference "D5") (unit 1) (value "1N4007") (footprint "Diode_SMD:D_SMA")
     )
     (path "/7d457770-3ae6-4bba-b199-d7585f460ba2"
-      (reference "D6") (unit 1) (value "1N4007") (footprint "Library:do214ab")
+      (reference "D6") (unit 1) (value "1N4007") (footprint "Diode_SMD:D_SMA")
     )
     (path "/cdc66536-909d-4061-b162-dce4f82e5cd3"
-      (reference "D7") (unit 1) (value "1N4007") (footprint "Library:do214ab")
+      (reference "D7") (unit 1) (value "1N4007") (footprint "Diode_SMD:D_SMA")
     )
     (path "/6eedbe40-3b61-4b26-9ea9-740057121005"
-      (reference "D8") (unit 1) (value "1N4007") (footprint "Library:do214ab")
+      (reference "D8") (unit 1) (value "1N4007") (footprint "Diode_SMD:D_SMA")
     )
     (path "/73b026f9-12ed-4785-b420-64c149f7ca47"
-      (reference "D9") (unit 1) (value "1N4007") (footprint "Library:do214ab")
+      (reference "D9") (unit 1) (value "1N4007") (footprint "Diode_SMD:D_SMA")
     )
     (path "/f7d3a194-7b05-45ac-9a98-e2a775ba02fa"
-      (reference "D10") (unit 1) (value "1N4007") (footprint "Library:do214ab")
+      (reference "D10") (unit 1) (value "1N4007") (footprint "Diode_SMD:D_SMA")
     )
     (path "/bf31004e-2f97-4529-8095-4e31481dcd91"
-      (reference "D11") (unit 1) (value "1N4007") (footprint "Library:do214ab")
+      (reference "D11") (unit 1) (value "1N4007") (footprint "Diode_SMD:D_SMA")
     )
     (path "/19019b8a-90fb-4575-9233-299c1547251b"
-      (reference "D12") (unit 1) (value "1N4007") (footprint "Library:do214ab")
+      (reference "D12") (unit 1) (value "1N4007") (footprint "Diode_SMD:D_SMA")
     )
     (path "/846d44ad-507d-431b-9652-0a18ae445cf0"
@@
     )
     (path "/951d8e55-0983-48e1-a0c4-bac48479355a"
-      (reference "RV1") (unit 1) (value "10k") (footprint "")
+      (reference "RV1") (unit 1) (value "10k") (footprint "Library:Potentiometer_Bourns_3386P_Vertical")
     )
     (path "/7078f9f8-f76c-4524-96a7-1f5a2c6a03e5"

Commit message: Update myDAQExpansionBoard.kicad_sch
Other:
- note added: "D5 to D12 = 2 A Fast diodes VF ≤ 1.2 V @ I = 2 A trr ≤ 200 ns 1N4007 SMD"
- note removed: "D5 to D12 = 2 A Fast diodes VF ≤ 1.2 V @ I = 2 A trr ≤ 200 ns SS34"
Changed lines of the file:
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@@
     (effects (font (size 1.27 1.27)) (justify left bottom))
   )
-  (text "D5 to D12 = 2 A Fast diodes VF ≤ 1.2 V @ I = 2 A\ntrr ≤ 200 ns\n\nSS34"
+  (text "D5 to D12 = 2 A Fast diodes VF ≤ 1.2 V @ I = 2 A\ntrr ≤ 200 ns\n\n1N4007 SMD"
     (at 219.71 113.03 0)
     (effects (font (size 1.27 1.27)) (justify left bottom))

Commit message: update
Parts:
- removed H1, H2, H3, H4: MountingHole_Pad, MountingHole:MountingHole_3.2mm_M3, symbol Mechanical:MountingHole
- added H1, H2, H3, H4: MountingHole_Pad, MountingHole:MountingHole_3.2mm_M3_ISO7380_Pad, symbol Mechanical:MountingHole_Pad
- JP6, JP7, JP8: footprint Library:PinHeader_1x02_P2.54mm_jumper -> Library:PinHeader_1x03_P2.54mm_Vertical_jumper
- U4: footprint Package_TO_SOT_THT:TO-220-15_P2.54x2.54mm_StaggerOdd_Lead4.58mm_Vertical -> Library:TO-220-15_P2.54x2.54mm_StaggerOdd_Lead4.58mm_Vertical
Connections:
- net +5V: now also R3.1, R4.1; no longer JP2.2 (B), JP3.2 (B)
- net DIO0: now also R1.1; no longer D1.2 (A)
- net DIO1: now also R5.1; no longer D2.2 (A)
- net DIO2: now also R7.1; no longer D3.2 (A)
- net DIO3: now also R9.1; no longer D4.2 (A)
- net DIO4: now also JP2.2 (B); no longer CD1.1, R3.2, SW3.1
- net DIO5: now also JP3.2 (B); no longer CD2.1, R4.2, SW4.1
- net at D3.1 (K): now also D1.1 (K), D2.1 (K), D4.1 (K), JP5.1 (A); no longer R7.1
- net at JP2.1 (A): now also CD1.1, R3.2, SW3.1; no longer R3.1
- net at JP3.1 (A): now also CD2.1, R4.2, SW4.1; no longer R4.1
- new net: D3.2 (A), R7.2
- new net: D1.2 (A), R1.2
- new net: D4.2 (A), R9.2
- new net: D2.2 (A), R5.2
- no-connect marks 5 -> 9
Other:
- note added: "- pin headeri mogu biti u različitim bojama"
- moved on the sheet: CD1, CD2, JP2, JP3, JP5, R1, R3, R4, R5, R7, R9, SW3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

Commit message: update
Parts:
- C5: footprint Capacitor_THT:CP_Radial_D12.5mm_P5.00mm -> Capacitor_THT:C_Radial_D10.0mm_H16.0mm_P5.00mm
Connections:
- net at JP8.1 (A): now also RV1.2; no longer U3.7 (VIOUT)
- net at JP7.1 (A): now also U3.7 (VIOUT); no longer RV1.2
Other:
- note removed: "POTENCIOMETAR"
- moved on the sheet: JP7, JP8, R17, R18, RV1

Commit message: update
Other:
- note added: "-provjeriti gnd oko hmosta - pin headeri mogu biti u različitim bojama"
- note removed: "- pin headeri mogu biti u različitim bojama"
Changed lines of the file:
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@@
     (effects (font (size 1.27 1.27)) (justify left bottom))
   )
-  (text "- pin headeri mogu biti u različitim bojama" (at 309.88 86.36 0)
+  (text "-provjeriti gnd oko hmosta\n- pin headeri mogu biti u različitim bojama"
+    (at 309.88 86.36 0)
     (effects (font (size 1.27 1.27)) (justify left bottom))
   )
