File: KiCAD files/myDAQExpansionBoard_v4/myDAQExpansionBoard.kicad_sch (KiCad schematic)
At the start: 73 parts, among them J1 Conn_01x05_Male, J2 Conn_01x05_Male, J3 Conn_01x08_Male, J4 OSTV7XX3151, J5 Screw_Terminal_01x02, J6 Screw_Terminal_01x02, J7 Screw_Terminal_01x01, J8 Screw_Terminal_01x01, SW1 SW_SPDT, SW2 SW_SPDT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

Commit message: update
Parts:
- RV1: footprint Library:Potentiometer_Bourns_3386P_Vertical -> Library:PTV09A-4225F-B502
Changed lines of the file:
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@@
       (effects (font (size 1.27 1.27)) (justify right))
     )
-    (property "Footprint" "Library:Potentiometer_Bourns_3386P_Vertical" (id 2) (at 97.409 125.857 0)
+    (property "Footprint" "Library:PTV09A-4225F-B502" (id 2) (at 97.409 125.857 0)
       (effects (font (size 1.27 1.27)) hide)
     )
@@
     )
     (path "/951d8e55-0983-48e1-a0c4-bac48479355a"
-      (reference "RV1") (unit 1) (value "10k") (footprint "Library:Potentiometer_Bourns_3386P_Vertical")
+      (reference "RV1") (unit 1) (value "10k") (footprint "Library:PTV09A-4225F-B502")
     )
     (path "/7078f9f8-f76c-4524-96a7-1f5a2c6a03e5"

Commit message: Update myDAQExpansionBoard.kicad_sch
Other:
- note added: "- uljepšati shemu - JLCJLCJLCJLC - provjeriti gnd oko hmosta - 3d model hladnjaka - isprintati i provjeriti layout - isprintati i provjeriti vodiče - github qr - jk logo - TVZ logo - pin headeri mogu biti u različitim bojama"
- note removed: "-provjeriti gnd oko hmosta - pin headeri mogu biti u različitim bojama"
Changed lines of the file:
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@@
     (effects (font (size 1.27 1.27)) (justify left bottom))
   )
-  (text "-provjeriti gnd oko hmosta\n- pin headeri mogu biti u različitim bojama"
+  (text "- uljepšati shemu\n- JLCJLCJLCJLC\n- provjeriti gnd oko hmosta\n- 3d model hladnjaka\n- isprintati i provjeriti layout\n- isprintati i provjeriti vodiče\n- github qr\n- jk logo\n- TVZ logo\n- pin headeri mogu biti u različitim bojama"
     (at 309.88 86.36 0)
     (effects (font (size 1.27 1.27)) (justify left bottom))

Commit message: update
Other:
- note added: "- uljepšati shemu - dodati legendu, pojasniti priključnice i jumpere, grupirati elemente ako treba - silkscreen preklapanje, optimizirati konektore za motor - 3d model hladnjaka - isprintati i provjeriti layout - isprintati i provjeriti vodiče - github qr - jk logo - TVZ logo - pin headeri mogu biti u različitim bojama"
- note removed: "- uljepšati shemu - JLCJLCJLCJLC - provjeriti gnd oko hmosta - 3d model hladnjaka - isprintati i provjeriti layout - isprintati i provjeriti vodiče - github qr - jk logo - TVZ logo - pin headeri mogu biti u različitim bojama"
Changed lines of the file:
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@@
     (effects (font (size 1.27 1.27)) (justify left bottom))
   )
-  (text "- uljepšati shemu\n- JLCJLCJLCJLC\n- provjeriti gnd oko hmosta\n- 3d model hladnjaka\n- isprintati i provjeriti layout\n- isprintati i provjeriti vodiče\n- github qr\n- jk logo\n- TVZ logo\n- pin headeri mogu biti u različitim bojama"
+  (text "- uljepšati shemu\n- dodati legendu, pojasniti priključnice i jumpere, grupirati elemente ako treba\n- silkscreen preklapanje, optimizirati konektore za motor\n- 3d model hladnjaka\n- isprintati i provjeriti layout\n- isprintati i provjeriti vodiče\n- github qr\n- jk logo\n- TVZ logo\n- pin headeri mogu biti u različitim bojama"
     (at 309.88 86.36 0)
     (effects (font (size 1.27 1.27)) (justify left bottom))

Commit message: update
Other:
- note added: "- dodati legendu, pojasniti priključnice i jumpere, grupirati elemente ako treba - silkscreen preklapanje, optimizirati konektore za motor - 3d model hladnjaka - isprintati i provjeriti layout - isprintati i provjeriti vodiče - github qr - jk logo - TVZ logo - LabVIEW logo - pin headeri mogu biti u različitim bojama"
- note added: "5V LED INDIKATOR"
- note added: "5V i GND KONEKTORI"
- note added: "7SEGM + IC SN74LS74"
- note added: "DODATNO NAPAJANJE I LED INDIKATOR"
- note added: "GND i AGND su spojeni jednim tanjim vodičem"
- note added: "HALL SENZOR"
- note added: "MON. RUPE"
- note added: "POT"
- note added: "POWER FLAGovi"
- note added: "myDAQ KONEKTOR"
- note removed: "- uljepšati shemu - dodati legendu, pojasniti priključnice i jumpere, grupirati elemente ako treba - silkscreen preklapanje, optimizirati konektore za motor - 3d model hladnjaka - isprintati i provjeriti layout - isprintati i provjeriti vodiče - github qr - jk logo - TVZ logo - pin headeri mogu biti u različitim bojama"
- note removed: "7SEGM"
- note removed: "ACS712"
- note removed: "EXTERNAL POWER"
- note removed: "LOGIC POWER LED"
- moved on the sheet: C1, C2, C3, C4, C5, C6, CD1, CD2, D1, D10, D11, D12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
