File: KiCAD files/myDAQExpansionBoard_v4.1/myDAQExpansionBoard.kicad_sch (KiCad schematic)
At the start: 73 parts, among them J1 Conn_01x05_Male, J2 Conn_01x05_Male, J3 Conn_01x08_Male, J4 OSTV7XX3151, J5 Screw_Terminal_01x02, J6 Screw_Terminal_01x02, J7 Screw_Terminal_01x01, J8 Screw_Terminal_01x01, SW1 SW_SPDT, SW2 SW_SPDT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

Commit message: update
Other:
- note added: "- vodiči 14 mils - dodati legendu, pojasniti priključnice i jumpere, grupirati elemente ako treba - odvojiti AGND - silkscreen preklapanje, optimizirati konektore za motor - 3d model hladnjaka i footprint - isprintati i provjeriti layout - isprintati i provjeriti vodiče - github qr - jk logo - TVZ logo - LabVIEW logo MONTAŽA: - pin headeri mogu biti u različitim bojama"
- note removed: "- dodati legendu, pojasniti priključnice i jumpere, grupirati elemente ako treba - odvojiti AGND i gnd visokog napona - silkscreen preklapanje, optimizirati konektore za motor - 3d model hladnjaka - isprintati i provjeriti layout - isprintati i provjeriti vodiče - github qr - jk logo - TVZ logo - LabVIEW logo - pin headeri mogu biti u različitim bojama"
Changed lines of the file:
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@@
     (effects (font (size 2 2)) (justify left bottom))
   )
-  (text "- dodati legendu, pojasniti priključnice i jumpere, grupirati elemente ako treba\n- odvojiti AGND i gnd visokog napona\n- silkscreen preklapanje, optimizirati konektore za motor\n- 3d model hladnjaka\n- isprintati i provjeriti layout\n- isprintati i provjeriti vodiče\n- github qr\n- jk logo\n- TVZ logo\n- LabVIEW logo\n- pin headeri mogu biti u različitim bojama"
+  (text "- vodiči 14 mils\n- dodati legendu, pojasniti priključnice i jumpere, grupirati elemente ako treba\n- odvojiti AGND\n- silkscreen preklapanje, optimizirati konektore za motor\n- 3d model hladnjaka i footprint\n- isprintati i provjeriti layout\n- isprintati i provjeriti vodiče\n- github qr\n- jk logo\n- TVZ logo\n- LabVIEW logo\n\n\nMONTAŽA:\n- pin headeri mogu biti u različitim bojama"
     (at 13.462 176.784 0)
     (effects (font (size 1.27 1.27)) (justify left bottom))

Commit message: update
Parts:
- RV1: footprint Library:PTV09A-4225F-B502 -> Library:Potentiometer_Bourns_3386P_Vertical
Connections:
- net +5V: now also RV1.3; no longer RV1.1
- net GND: now also RV1.1; no longer RV1.3
Other:
- note added: "- dodati legendu, pojasniti priključnice i jumpere, grupirati elemente ako treba - odvojiti AGND - silkscreen preklapanje, optimizirati konektore za motor - 3d model hladnjaka i footprint - isprintati i provjeriti layout - isprintati i provjeriti vodiče - github qr s donje strane - jk logo - TVZ logo - LabVIEW logo - ime pločice i revizija - opensource hardware logo MONTAŽA: - pin headeri mogu bi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"
- note removed: "- vodiči 14 mils - dodati legendu, pojasniti priključnice i jumpere, grupirati elemente ako treba - odvojiti AGND - silkscreen preklapanje, optimizirati konektore za motor - 3d model hladnjaka i footprint - isprintati i provjeriti layout - isprintati i provjeriti vodiče - github qr - jk logo - TVZ logo - LabVIEW logo MONTAŽA: - pin headeri mogu biti u različitim bojama"
Changed lines of the file:
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@@
     (effects (font (size 2 2)) (justify left bottom))
   )
-  (text "- vodiči 14 mils\n- dodati legendu, pojasniti priključnice i jumpere, grupirati elemente ako treba\n- odvojiti AGND\n- silkscreen preklapanje, optimizirati konektore za motor\n- 3d model hladnjaka i footprint\n- isprintati i provjeriti layout\n- isprintati i provjeriti vodiče\n- github qr\n- jk logo\n- TVZ logo\n- LabVIEW logo\n\n\nMONTAŽA:\n- pin headeri mogu biti u različitim bojama"
-    (at 13.462 176.784 0)
+  (text "- dodati legendu, pojasniti priključnice i jumpere, grupirati elemente ako treba\n- odvojiti AGND\n- silkscreen preklapanje, optimizirati konektore za motor\n- 3d model hladnjaka i footprint\n- isprintati i provjeriti layout\n- isprintati i provjeriti vodiče\n- github qr s donje strane\n- jk logo\n- TVZ logo\n- LabVIEW logo\n- ime pločice i revizija\n- opensource hardware logo\n\nMONTAŽA:\n- pin headeri mogu biti u različitim bojama"
+    (at 12.954 187.198 0)
     (effects (font (size 1.27 1.27)) (justify left bottom))
   )
@@
     (pin "1")
   )
-  (symbol (lib_id "Device:R_Potentiometer") (at 56.134 83.82 0) (unit 1)
+  (symbol (lib_id "Device:R_Potentiometer") (at 56.134 83.82 0) (mirror x) (unit 1)
     (in_bom yes) (on_board yes) (fields_autoplaced)
     (property "Reference" "RV1" (id 0) (at 54.3561 82.9853 0)
@@
       (effects (font (size 1.27 1.27)) (justify right))
     )
-    (property "Footprint" "Library:PTV09A-4225F-B502" (id 2) (at 56.134 83.82 0)
+    (property "Footprint" "Library:Potentiometer_Bourns_3386P_Vertical" (id 2) (at 56.134 83.82 0)
       (effects (font (size 1.27 1.27)) hide)
     )
@@
     )
     (path "/951d8e55-0983-48e1-a0c4-bac48479355a"
-      (reference "RV1") (unit 1) (value "10k") (footprint "Library:PTV09A-4225F-B502")
+      (reference "RV1") (unit 1) (value "10k") (footprint "Library:Potentiometer_Bourns_3386P_Vertical")
     )
     (path "/7078f9f8-f76c-4524-96a7-1f5a2c6a03e5"

Commit message: update
Other:
- note added: "- dodati legendu, pojasniti priključnice i jumpere, grupirati elemente ako treba - odvojiti AGND - silkscreen preklapanje, optimizirati konektore za motor - 3d model hladnjaka i footprint - isprintati i provjeriti layout - isprintati i provjeriti vodiče - github qr s donje strane - jk logo - TVZ logo - LabVIEW logo - ime pločice i revizija - opensource hardware logo - moj mail MONTAŽA: - pin head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"
- note removed: "- dodati legendu, pojasniti priključnice i jumpere, grupirati elemente ako treba - odvojiti AGND - silkscreen preklapanje, optimizirati konektore za motor - 3d model hladnjaka i footprint - isprintati i provjeriti layout - isprintati i provjeriti vodiče - github qr s donje strane - jk logo - TVZ logo - LabVIEW logo - ime pločice i revizija - opensource hardware logo MONTAŽA: - pin headeri mogu bi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"
Changed lines of the file:
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@@
     (effects (font (size 2 2)) (justify left bottom))
   )
-  (text "- dodati legendu, pojasniti priključnice i jumpere, grupirati elemente ako treba\n- odvojiti AGND\n- silkscreen preklapanje, optimizirati konektore za motor\n- 3d model hladnjaka i footprint\n- isprintati i provjeriti layout\n- isprintati i provjeriti vodiče\n- github qr s donje strane\n- jk logo\n- TVZ logo\n- LabVIEW logo\n- ime pločice i revizija\n- opensource hardware logo\n\nMONTAŽA:\n- pin headeri mogu biti u različitim bojama"
-    (at 12.954 187.198 0)
+  (text "- dodati legendu, pojasniti priključnice i jumpere, grupirati elemente ako treba\n- odvojiti AGND\n- silkscreen preklapanje, optimizirati konektore za motor\n- 3d model hladnjaka i footprint\n- isprintati i provjeriti layout\n- isprintati i provjeriti vodiče\n- github qr s donje strane\n- jk logo\n- TVZ logo\n- LabVIEW logo\n- ime pločice i revizija\n- opensource hardware logo\n- moj mail\n\nMONTAŽA:\n- pin headeri mogu biti u različitim bojama\n- jumperi moraju biti oni koji imaju ručkicu + u bojama"
+    (at 12.954 190.246 0)
     (effects (font (size 1.27 1.27)) (justify left bottom))
   )

Commit message: update
Parts:
- U4: footprint Library:TO-220-15_P2.54x2.54mm_StaggerOdd_Lead4.58mm_Vertical -> Library:L298n
Other:
- note added: "- 3d model hladnjaka i footprint - provjeriti orjentaciju potenciometra - pitati lučana za mišljenje za potenciometar - l298n footprint s hladnjakom - dodati legendu, pojasniti priključnice i jumpere, grupirati elemente ako treba - odvojiti AGND - silkscreen preklapanje, optimizirati konektore za motor - isprintati i provjeriti layout - isprintati i provjeriti vodiče - github qr s donje strane - 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"
- note removed: "- dodati legendu, pojasniti priključnice i jumpere, grupirati elemente ako treba - odvojiti AGND - silkscreen preklapanje, optimizirati konektore za motor - 3d model hladnjaka i footprint - isprintati i provjeriti layout - isprintati i provjeriti vodiče - github qr s donje strane - jk logo - TVZ logo - LabVIEW logo - ime pločice i revizija - opensource hardware logo - moj mail MONTAŽA: - pin head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"
Changed lines of the file:
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@@
     (effects (font (size 2 2)) (justify left bottom))
   )
-  (text "- dodati legendu, pojasniti priključnice i jumpere, grupirati elemente ako treba\n- odvojiti AGND\n- silkscreen preklapanje, optimizirati konektore za motor\n- 3d model hladnjaka i footprint\n- isprintati i provjeriti layout\n- isprintati i provjeriti vodiče\n- github qr s donje strane\n- jk logo\n- TVZ logo\n- LabVIEW logo\n- ime pločice i revizija\n- opensource hardware logo\n- moj mail\n\nMONTAŽA:\n- pin headeri mogu biti u različitim bojama\n- jumperi moraju biti oni koji imaju ručkicu + u bojama"
-    (at 12.954 190.246 0)
+  (text "- 3d model hladnjaka i footprint\n- provjeriti orjentaciju potenciometra\n- pitati lučana za mišljenje za potenciometar\n- l298n footprint s hladnjakom\n- dodati legendu, pojasniti priključnice i jumpere, grupirati elemente ako treba\n- odvojiti AGND\n- silkscreen preklapanje, optimizirati konektore za motor\n- isprintati i provjeriti layout\n- isprintati i provjeriti vodiče\n- github qr s donje strane\n- jk logo\n- LabVIEW logo\n\nMONTAŽA:\n- pin headeri mogu biti u različitim bojama\n- jumperi moraju biti oni koji imaju ručkicu + u bojama"
+    (at 12.7 192.786 0)
     (effects (font (size 1.27 1.27)) (justify left bottom))
   )
@@
       (effects (font (size 1.27 1.27)) (justify left))
     )
-    (property "Footprint" "Library:TO-220-15_P2.54x2.54mm_StaggerOdd_Lead4.58mm_Vertical" (id 2) (at 133.096 162.179 0)
+    (property "Footprint" "Library:L298n" (id 2) (at 133.096 162.179 0)
       (effects (font (size 1.27 1.27)) (justify left) hide)
     )
@@
     )
     (path "/dfb5f089-6957-4ffa-aef1-b0b311b19342"
-      (reference "U4") (unit 1) (value "L298N") (footprint "Library:TO-220-15_P2.54x2.54mm_StaggerOdd_Lead4.58mm_Vertical")
-    )
-  )
+      (reference "U4") (unit 1) (value "L298N") (footprint "Library:L298n")
+    )
+  )

Commit message: update
Other:
- note added: "- l298n footprint s hladnjakom - provjeriti orjentaciju potenciometra - pitati lučana za mišljenje za potenciometa - odvojiti AGND - silkscreen preklapanje, optimizirati konektore za motor - isprintati i provjeriti layout - isprintati i provjeriti vodiče - github qr s donje strane - jk logo - LabVIEW logo MONTAŽA: - pin headeri mogu biti u različitim bojama - jumperi moraju biti oni koji imaju ru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"
- note removed: "- 3d model hladnjaka i footprint - provjeriti orjentaciju potenciometra - pitati lučana za mišljenje za potenciometar - l298n footprint s hladnjakom - dodati legendu, pojasniti priključnice i jumpere, grupirati elemente ako treba - odvojiti AGND - silkscreen preklapanje, optimizirati konektore za motor - isprintati i provjeriti layout - isprintati i provjeriti vodiče - github qr s donje strane - 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"
Changed lines of the file:
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@@
     (effects (font (size 2 2)) (justify left bottom))
   )
-  (text "- 3d model hladnjaka i footprint\n- provjeriti orjentaciju potenciometra\n- pitati lučana za mišljenje za potenciometar\n- l298n footprint s hladnjakom\n- dodati legendu, pojasniti priključnice i jumpere, grupirati elemente ako treba\n- odvojiti AGND\n- silkscreen preklapanje, optimizirati konektore za motor\n- isprintati i provjeriti layout\n- isprintati i provjeriti vodiče\n- github qr s donje strane\n- jk logo\n- LabVIEW logo\n\nMONTAŽA:\n- pin headeri mogu biti u različitim bojama\n- jumperi moraju biti oni koji imaju ručkicu + u bojama"
+  (text "- l298n footprint s hladnjakom\n- provjeriti orjentaciju potenciometra\n- pitati lučana za mišljenje za potenciometa\n- odvojiti AGND\n- silkscreen preklapanje, optimizirati konektore za motor\n- isprintati i provjeriti layout\n- isprintati i provjeriti vodiče\n- github qr s donje strane\n- jk logo\n- LabVIEW logo\n\nMONTAŽA:\n- pin headeri mogu biti u različitim bojama\n- jumperi moraju biti oni koji imaju ručkicu + u bojama"
     (at 12.7 192.786 0)
     (effects (font (size 1.27 1.27)) (justify left bottom))
