File: KiCAD files/myDAQExpansionBoard_v4.1/_autosave-myDAQExpansionBoard.kicad_sch (KiCad schematic)
At the start: 71 parts, among them J1 Conn_01x05_Male, J2 Conn_01x05_Male, J3 Conn_01x08_Male, J4 OSTV7XX3151, J5 Screw_Terminal_01x02, J6 Screw_Terminal_01x02, J7 Screw_Terminal_01x01, J8 Screw_Terminal_01x01, SW1 SW_SPDT, SW2 SW_SPDT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

Commit message: update
Other:
- note added: "- github qr s donje strane MONTAŽA: - pin headeri mogu biti u različitim bojama - jumperi moraju biti oni koji imaju ručkicu + u bojama"
- note removed: "- provjeriti debljinu GNDa - provjeriti debljinu napajanja za motor - odvojiti AGND - isprintati i provjeriti vodiče - github qr s donje strane MONTAŽA: - pin headeri mogu biti u različitim bojama - jumperi moraju biti oni koji imaju ručkicu + u bojama"
Changed lines of the file:
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@@
     (effects (font (size 2 2)) (justify left bottom))
   )
-  (text "- provjeriti debljinu GNDa\n- provjeriti debljinu napajanja za motor\n- odvojiti AGND\n- isprintati i provjeriti vodiče\n- github qr s donje strane\n\nMONTAŽA:\n- pin headeri mogu biti u različitim bojama\n- jumperi moraju biti oni koji imaju ručkicu + u bojama"
+  (text "- github qr s donje strane\n\nMONTAŽA:\n- pin headeri mogu biti u različitim bojama\n- jumperi moraju biti oni koji imaju ručkicu + u bojama"
     (at 17.145 177.165 0)
     (effects (font (size 1.27 1.27)) (justify left bottom))
