File: KiCAD files/myDAQExpansionBoard_v4.1/myDAQExpansionBoard.kicad_pcb (KiCad board)
At the start: 2 copper layers, 100 x 100 mm, 73 parts, among them J1 Conn_01x05_Male, J2 Conn_01x05_Male, J3 Conn_01x08_Male, J4 OSTV7XX3151, J5 Screw_Terminal_01x02, J6 Screw_Terminal_01x02, J7 Screw_Terminal_01x01, J8 Screw_Terminal_01x01, SW1 SW_SPDT, SW2 SW_SPDT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

Commit message: update
Parts:
- moved D9 28.7 mm to (48.6, 103.4)
- moved D10 28.7 mm to (52.5, 103.4)
- moved D11 28.7 mm to (66.0, 83.2)
- moved D12 28.7 mm to (45.0, 103.4)
- moved D5 28.7 mm to (56.2, 70.4)
- moved D6 28.7 mm to (52.5, 70.4)
- moved D7 28.7 mm to (48.7, 70.4)
- moved D8 28.7 mm to (45.0, 70.4)
- moved J5 28.6 mm to (74.7, 63.0)
- moved C2 18.7 mm to (70.8, 84.2)
- moved U4 18.7 mm to (73.4, 74.9)
- moved C5 17.7 mm to (86.5, 65.5), turned to 0 degrees
- moved C4 14.4 mm to (82.2, 79.4), turned to -90 degrees
- moved R19 10.8 mm to (77.0, 54.5), turned to 0 degrees
- moved C3 10.7 mm to (89.5, 55.2)
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Routing:
- net /OUT4: track 52.3 -> 16.1 mm
- net +5V: track 482.0 -> 449.8 mm, vias 12 -> 6
- net /OUT3: track 44.4 -> 14.1 mm
- net /OUT2: track 42.8 -> 13.7 mm
- net /OUT1: track 31.5 -> 18.9 mm
- net Net-(JP10-Pad2): track 43.6 -> 31.4 mm
- net Net-(R11-Pad2): track 15.3 -> 4.97 mm
- net Net-(JP7-Pad1): track 35.2 -> 25.1 mm
- net VDD: track 10.0 -> 0.00 mm
- net Net-(R11-Pad1): track 3.84 -> 13.9 mm
- net DIO0: track 130.3 -> 120.4 mm
- net Net-(R10-Pad1): track 4.14 -> 13.9 mm
- net Net-(R8-Pad1): track 4.43 -> 13.9 mm
- net Net-(R10-Pad2): track 20.5 -> 11.9 mm
- net DIO3: track 193.9 -> 186.1 mm
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- removed copper zone on B.Cu, net /IP-
- removed copper zone on F.Cu, net /IP-
- removed copper zone on F.Cu, net VDD

Commit message: update
Parts:
- RV1: footprint Library:PTV09A-4225F-B502 -> Library:Potentiometer_Bourns_3386P_Vertical
- moved JP5 57.2 mm to (95.8, 99.0), turned to 0 degrees
- moved RV1 41.8 mm to (151.8, 99.7), turned to -90 degrees
- moved JP10 24.6 mm to (88.2, 101.5), turned to 180 degrees
- moved JP9 20.8 mm to (92.0, 101.5), turned to 180 degrees
- moved D2 19.3 mm to (115.0, 101.5)
- moved D3 19.3 mm to (124.0, 101.5)
- moved R5 19.3 mm to (115.0, 94.5)
- moved R7 19.3 mm to (124.0, 94.5)
- moved D1 19.2 mm to (106.0, 101.5)
- moved D4 19.2 mm to (133.0, 101.5)
- moved R1 19.2 mm to (106.0, 94.5)
- moved R9 19.2 mm to (133.0, 94.5)
- moved R8 10.2 mm to (122.5, 69.8)
- moved R10 10.0 mm to (122.5, 73.0)
- moved R11 9.98 mm to (122.5, 76.2)
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Connections:
- RV1 pad 1: +5V -> GND
- RV1 pad 3: GND -> +5V
Routing:
- net Net-(JP8-Pad1): track 55.6 -> 106.1 mm, vias 0 -> 4
- net Net-(JP10-Pad2): track 31.4 -> 0.00 mm, vias 2 -> 0
- net DIO0: track 120.4 -> 89.7 mm
- net GND: track 90.8 -> 116.6 mm
- net +5V: track 449.8 -> 428.9 mm, vias 6 -> 8
- net /OUT1: track 18.9 -> 0.04 mm
- net /OUT4: track 16.1 -> 0.00 mm
- net /OUT3: track 14.1 -> 0.00 mm
- net Net-(JP9-Pad2): track 14.0 -> 0.00 mm
- net /OUT2: track 13.7 -> 0.00 mm
- net Net-(D1-Pad1): track 49.3 -> 38.3 mm
- net Net-(R11-Pad2): track 4.97 -> 14.7 mm
- net Net-(R11-Pad1): track 13.9 -> 4.13 mm
- net Net-(R10-Pad1): track 13.9 -> 4.43 mm
- net Net-(R8-Pad1): track 13.9 -> 5.16 mm
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Other:
- board text added: "OUT1"
- board text added: "OUT2"
- board text added: "OUT3"
- board text added: "OUT4"
- board text added: "POT"
- board text added: "S1"
- board text added: "S2"
- board text added: "T1"
- board text added: "T2"

Commit message: update
Parts:
- added G***: LOGO, Library:tvz, F.Cu at (163.5, 114.2)
- moved D1 0.25 mm to (105.7, 101.5)
- moved D2 0.25 mm to (114.7, 101.5)
- moved D3 0.25 mm to (123.7, 101.5)
- moved D4 0.25 mm to (132.7, 101.5)
- moved R1 0.25 mm to (105.7, 94.5)
- moved R5 0.25 mm to (114.7, 94.5)
- moved R7 0.25 mm to (123.7, 94.5)
- moved R9 0.25 mm to (132.7, 94.5)
Routing:
- net DIO3: track 179.5 -> 154.1 mm
- net DIO2: track 161.7 -> 141.7 mm
- net DIO1: track 151.8 -> 140.1 mm
Other:
- board text added: "AO0"
- board text added: "DIO0"
- board text added: "DIO1"
- board text added: "DIO2"
- board text added: "DIO3"
- board text added: "DIO4"
- board text added: "DIO5"
- board text added: "DIO6"
- board text added: "DIO7"
- board text added: "I_SENS"
- board text added: "LDR"
- board text added: "myDAQExpansionBoard v1rev1"

Commit message: update
Parts:
- removed the G*** at (163.5, 114.2)
- added G***: LOGO, Library:tvz2, F.Cu at (95.8, 86.8)
- U4: footprint Library:TO-220-15_P2.54x2.54mm_StaggerOdd_Lead4.58mm_Vertical -> Library:L298n
- moved JP10 5.49 mm to (88.2, 107.0)
- moved JP5 5.49 mm to (95.8, 104.5)
- moved JP9 5.49 mm to (92.0, 107.0)
Routing:
- net Net-(D1-Pad1): track 38.0 -> 39.3 mm
Other:
- board text added: "josip.kordek@gmail.com"

Commit message: update
Parts:
- added G***: LOGO, Library:Labview-logo, F.Cu at (165.2, 101.0)

Commit message: update
Parts:
- removed D13: LED, LED_SMD:LED_1206_3216Metric
- removed the G*** at (165.2, 101.0)
- removed R19: 2k7, Resistor_SMD:R_0603_1608Metric
- RV1: footprint Library:Potentiometer_Bourns_3386P_Vertical -> Library:PTV09A-4225F-B502
- moved G*** 67.8 mm to (163.0, 95.0)
- moved D12 56.1 mm to (73.8, 55.2), turned to 90 degrees
- moved D6 43.7 mm to (85.2, 99.2), turned to 180 degrees
- moved D8 40.3 mm to (85.2, 68.5), turned to 180 degrees
- moved D7 37.5 mm to (85.2, 78.8), turned to 180 degrees
- moved D9 34.4 mm to (82.0, 111.9)
- moved D5 34.4 mm to (85.2, 88.8), turned to 180 degrees
- moved D11 32.2 mm to (82.0, 55.2), turned to 90 degrees
- moved JP9 26.4 mm to (97.5, 81.2), turned to -90 degrees
- moved D10 22.9 mm to (73.8, 111.9)
- moved JP10 18.9 mm to (97.5, 90.5), turned to -90 degrees
- moved R20 4.26 mm to (167.0, 44.5)
- moved JP5 2.97 mm to (96.2, 101.5), turned to 180 degrees
- moved D14 2.77 mm to (163.2, 44.5)
- moved C4 1.54 mm to (82.2, 77.9), turned to 90 degrees
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Routing:
- net +5V: track 428.9 -> 531.5 mm, vias 8 -> 14
- net Net-(JP10-Pad2): track 0.00 -> 60.5 mm, vias 0 -> 2
- net DIO3: track 154.1 -> 213.6 mm
- net DIO2: track 141.7 -> 197.4 mm
- net DIO1: track 140.1 -> 192.4 mm
- net /OUT4: track 0.00 -> 33.2 mm
- net /OUT1: track 0.04 -> 32.3 mm
- net /OUT2: track 0.00 -> 31.4 mm
- net /OUT3: track 0.00 -> 30.9 mm
- net DIO0: track 89.8 -> 118.3 mm
- net Net-(JP9-Pad2): track 0.00 -> 16.5 mm
- net Net-(JP8-Pad1): track 105.8 -> 98.5 mm
- net /IP-: track 3.73 -> 0.00 mm
- net GND: track 116.6 -> 119.6 mm
- net Net-(D1-Pad1): track 39.3 -> 36.5 mm
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- added copper zone on B.Cu, net /IP-
- added copper zone on F.Cu, net /IP-
- added copper zone on F.Cu, net VDD
Other:
- board text added: "+"
- board text added: "-"
- board text added: "1"
- board text added: "2"
- board text added: "3"
- board text added: "4"
- board text added: "OUTPUT"
- board text removed: "EXT. POWER"
- board text removed: "OUT1"
- board text removed: "OUT2"
- board text removed: "OUT3"
- board text removed: "OUT4"

Commit message: update
Parts:
- added G***: LOGO, Library:qrcode, B.Cu at (154.2, 76.2)
Other:
- board text added: "Git:"
