File: KiCADFiles/myDAQExpansionBoard/myDAQExpansionBoard.kicad_sch (KiCad schematic)
At the start: 73 parts, among them J1 Conn_01x05_Male, J2 Conn_01x05_Male, J3 Conn_01x08_Male, J4 OSTV7XX3151, J5 Screw_Terminal_01x02, J6 Screw_Terminal_01x02, J7 Screw_Terminal_01x01, J8 Screw_Terminal_01x01, SW1 SW_SPDT, SW2 SW_SPDT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

Commit message: Initial release
Other:
- note removed: "BILJEŠKE: - BOM se nalazi u bom folderu, datoteka se zove myDAQExpansionBoard.xlsx"
Changed lines of the file:
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@@
   (title_block
     (title "myDAQExpansionBoard")
-    (date "2022-07-24")
+    (date "2023-03-28")
     (rev "1")
     (company "TVZ")
@@
     (effects (font (size 2 2)) (justify left bottom))
   )
-  (text "BILJEŠKE:\n\n- BOM se nalazi u bom folderu, datoteka se zove myDAQExpansionBoard.xlsx"
-    (at 15.24 185.42 0)
-    (effects (font (size 2.54 2.54)) (justify left bottom))
-  )
   (text "MON. RUPE" (at 14.986 88.9 0)
